File: circuits/Drive/Power.kicad_sch (KiCad schematic)
At the start: 76 parts, among them IC1 DCDC_MPM3620A, J1 Conn_01x02_Male, J10 Conn_01x02_Male, J11 Conn_01x02_Male, J12 Conn_01x02_Male, J13 Conn_01x02_Male, J14 Conn_01x02_Male, J15 Conn_01x02_Male, J9 Conn_01x02_Male, Q16 SSM6J808R, Q17 SSM6J808R, Q18 SSM3J332R, Q19 S8550, Q2 BSS138, Q20 SSM3J332R, Q21 S8550, Q23 S8550, Q24 SSM3J332R, Q25 S8550, Q3 SSM3J332R, Q4 BSS138, SW1 SW_SPDT_White, U1 AZ1117CH-3.3

Commit message: Driveほぼ完成
Parts:
- removed C10, C7, C9: 470uF, Capacitor_SMD:C_Elec_8x10.2, symbol Device:C_Polarized
- removed J1: Conn_01x02_Male, Connector_AMASS:AMASS_XT30PW-M_1x02_P2.50mm_Horizontal, symbol Connector:Conn_01x02_Male
- removed U1: AZ1117CH-3.3, Package_TO_SOT_SMD:SOT-223-3_TabPin2, symbol Regulator_Linear:AMS1117CD-3.3
- added C23, C25, C26, C32, C33, C37, C38, C39: 470uF, symbol Device:C_Polarized
- added C40: 10uF, Capacitor_SMD:C_0805_2012Metric, symbol Device:C
- added J14: Conn_01x02_Male, Connector_Molex:Molex_SPOX_5267-02A_1x02_P2.50mm_Vertical, symbol Connector:Conn_01x02_Male
- added J6: USB_C_Receptacle_USB2.0, Connector_USB:USB_C_Receptacle_G-Switch_GT-USB-7010ASV, symbol Connector:USB_C_Receptacle_USB2.0
- added R64, R65: 5.1k, Resistor_SMD:R_0402_1005Metric, symbol Device:R
- C6: footprint Capacitor_SMD:C_Elec_8x10.2 -> (none)
Connections:
- net +3.3V: now also C26.1
- net +5V: now also C25.1
- net +BATT: now also C32.1, C33.1, C37.1, C38.1, C39.1, J14.2 (Pin_2)
- net GND: now also C23.2, C25.2, C26.2, C32.2, C33.2, C37.2, C38.2, C39.2, C40.1, J14.1 (Pin_1), J6.A1 (GND), J6.A12 (GND), J6.B1 (GND), J6.B12 (GND), J6.S1 (SHIELD), R64.1, R65.1
- net VBUS: now also C40.2, J6.A4 (VBUS), J6.A9 (VBUS), J6.B4 (VBUS), J6.B9 (VBUS)
- net VCC: now also C23.1
- new net: J6.B5 (CC2), R64.2
- new net: J6.A5 (CC1), R65.2
- no-connect marks 5 -> 11
Other:
- note added: "USB-C"
- note added: "三端子を新しく選定したのにする"
- moved on the sheet: C1, C2, C23, C3, C4, C5, C6, C8, D1, D2, D3, D4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
