File: circuits/Drive/Mouse.kicad_sch (KiCad schematic)
At the start: 3 parts, among them U10 Sensor_OpticalFlowSensor_PIM4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

Commit message: Driveほぼ完成
Parts:
- removed JP16: SolderJumper_2_Open, Jumper:SolderJumper-2_P1.3mm_Open_TrianglePad1.0x1.5mm, symbol Jumper:SolderJumper_2_Open
- added Q16: BSS138, Package_TO_SOT_SMD:SOT-23, symbol Device:Q_NMOS_GSD
- added R63: 10k, Resistor_SMD:R_0402_1005Metric, symbol Device:R
- U10: value Sensor_OpticalFlowSensor_PIM453 -> Sensor_OpticalFlowSensor_PIM573
Connections:
- net GNDD: now also Q16.2 (S), R63.2
- net Mouse_INT: now also Q16.1 (G), R63.1
- net at U10.6 (INT): now also Q16.3 (D)
Changed lines of the file:
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@@
 (kicad_sch (version 20230121) (generator eeschema)
   (paper "A4")
+  (junction (at 142.24 106.68) (diameter 0) (color 0 0 0 0)
+  )
+  (junction (at 154.94 116.84) (diameter 0) (color 0 0 0 0)
+  )
   (junction (at 152.4 88.9) (diameter 0) (color 0 0 0 0)
   )
-  (wire (pts (xy 152.4 104.14) (xy 152.4 106.68))
+  (junction (at 149.86 116.84) (diameter 0) (color 0 0 0 0)
+  )
+  (wire (pts (xy 154.94 104.14) (xy 154.94 116.84))
+    (stroke (width 0) (type default))
+  )
+  (wire (pts (xy 154.94 116.84) (xy 154.94 119.38))
+    (stroke (width 0) (type default))
+  )
+  (wire (pts (xy 149.86 116.84) (xy 154.94 116.84))
     (stroke (width 0) (type default))
   )
@@
     (stroke (width 0) (type default))
   )
+  (wire (pts (xy 149.86 111.76) (xy 149.86 116.84))
+    (stroke (width 0) (type default))
+  )
   (polyline (pts (xy 118.11 66.04) (xy 185.42 66.04))
     (stroke (width 0.5) (type default))
@@
     (stroke (width 0.5) (type default))
   )
-  (wire (pts (xy 151.13 101.6) (xy 154.94 101.6))
+  (wire (pts (xy 149.86 116.84) (xy 142.24 116.84))
     (stroke (width 0) (type default))
   )
@@
     (stroke (width 0.5) (type default))
   )
-  (wire (pts (xy 152.4 104.14) (xy 154.94 104.14))
+  (wire (pts (xy 149.86 101.6) (xy 154.94 101.6))
     (stroke (width 0) (type default))
   )
@@
     (stroke (width 0) (type default))
   )
-  (wire (pts (xy 142.24 101.6) (xy 143.51 101.6))
-    (stroke (width 0) (type default))
-  )
   (wire (pts (xy 152.4 88.9) (xy 151.13 88.9))
     (stroke (width 0) (type default))
@@
     (stroke (width 0.5) (type default))
   )
+  (wire (pts (xy 142.24 116.84) (xy 142.24 115.57))
+    (stroke (width 0) (type default))
+  )
+  (wire (pts (xy 142.24 106.68) (xy 142.24 107.95))
+    (stroke (width 0) (type default))
+  )
   (wire (pts (xy 152.4 93.98) (xy 154.94 93.98))
+    (stroke (width 0) (type default))
+  )
+  (wire (pts (xy 139.7 106.68) (xy 142.24 106.68))
     (stroke (width 0) (type default))
   )
@@
     (effects (font (size 2.54 2.54) (thickness 0.254) bold) (justify left bottom))
   )
-  (hierarchical_label "Mouse_INT" (shape input) (at 142.24 101.6 180) (fields_autoplaced)
+  (hierarchical_label "Mouse_INT" (shape input) (at 139.7 106.68 180) (fields_autoplaced)
     (effects (font (size 1.27 1.27) bold) (justify right))
   )
@@
     (effects (font (size 1.27 1.27)) (justify right))
   )
-  (symbol (lib_id "power:GNDD") (at 152.4 106.68 0) (unit 1)
+  (symbol (lib_id "Device:R") (at 142.24 111.76 0) (mirror y) (unit 1)
+    (in_bom yes) (on_board yes) (dnp no)
+    (property "Reference" "R63" (at 140.97 110.49 0)
+      (effects (font (size 1.27 1.27)) (justify left))
+    )
+    (property "Value" "10k" (at 140.97 113.03 0)
+      (effects (font (size 1.27 1.27)) (justify left))
+    )
+    (property "Footprint" "Resistor_SMD:R_0402_1005Metric" (at 144.018 111.76 90)
+      (effects (font (size 1.27 1.27)) hide)
+    )
+    (property "Datasheet" "~" (at 142.24 111.76 0)
+      (effects (font (size 1.27 1.27)) hide)
+    )
+    (pin "1")
+    (pin "2")
+    (instances
+      (project "Drive"
+        (path "/bf4fa0f7-7e40-4646-9c11-e04533c904d6/eede7486-c694-4c67-81d8-d20707e697df"
+          (reference "R63") (unit 1)
+        )
+      )
+    )
+  )
+  (symbol (lib_name "Q_NMOS_GSD_1") (lib_id "Device:Q_NMOS_GSD") (at 147.32 106.68 0) (unit 1)
+    (in_bom yes) (on_board yes) (dnp no)
+    (property "Reference" "Q16" (at 139.7 101.6 0)
+      (effects (font (size 1.27 1.27)) (justify left))
+    )
+    (property "Value" "BSS138" (at 139.7 104.14 0)
+      (effects (font (size 1.27 1.27)) (justify left))
+    )
+    (property "Footprint" "Package_TO_SOT_SMD:SOT-23" (at 152.4 104.14 0)
+      (effects (font (size 1.27 1.27)) hide)
+    )
+    (property "Datasheet" "~" (at 147.32 106.68 0)
+      (effects (font (size 1.27 1.27)) hide)
+    )
+    (pin "1")
+    (pin "2")
+    (pin "3")
+    (instances
+      (project "Drive"
+        (path "/bf4fa0f7-7e40-4646-9c11-e04533c904d6/eede7486-c694-4c67-81d8-d20707e697df"
+          (reference "Q16") (unit 1)
+        )
+      )
+    )
+  )
+  (symbol (lib_id "power:GNDD") (at 154.94 119.38 0) (unit 1)
     (in_bom yes) (on_board yes) (dnp no) (fields_autoplaced)
-    (property "Reference" "#PWR0137" (at 152.4 113.03 0)
-      (effects (font (size 1.27 1.27)) hide)
-    )
-    (property "Value" "GNDD" (at 152.4 110.49 0)
+    (property "Reference" "#PWR0137" (at 154.94 125.73 0)
+      (effects (font (size 1.27 1.27)) hide)
+    )
+    (property "Value" "GNDD" (at 154.94 123.19 0)
       (effects (font (size 1.27 1.27)))
     )
-    (property "Footprint" "" (at 152.4 106.68 0)
-      (effects (font (size 1.27 1.27)) hide)
-    )
-    (property "Datasheet" "" (at 152.4 106.68 0)
+    (property "Footprint" "" (at 154.94 119.38 0)
+      (effects (font (size 1.27 1.27)) hide)
+    )
+    (property "Datasheet" "" (at 154.94 119.38 0)
       (effects (font (size 1.27 1.27)) hide)
     )
@@
         (path "/aa9d7141-7530-418f-853d-a56ee68433fb/dd025a71-f40c-48d2-8202-a120d14a823c"
           (reference "#PWR0137") (unit 1)
+        )
+      )
+      (project "Drive"
+        (path "/bf4fa0f7-7e40-4646-9c11-e04533c904d6/eede7486-c694-4c67-81d8-d20707e697df"
+          (reference "#PWR0107") (unit 1)
         )
       )
@@
         )
       )
+      (project "Drive"
+        (path "/bf4fa0f7-7e40-4646-9c11-e04533c904d6/eede7486-c694-4c67-81d8-d20707e697df"
+          (reference "#PWR0106") (unit 1)
+        )
+      )
     )
   )
@@
         )
       )
-    )
-  )
-  (symbol (lib_id "Jumper:SolderJumper_2_Open") (at 147.32 101.6 0) (mirror x) (unit 1)
-    (in_bom yes) (on_board yes) (dnp no)
-    (property "Reference" "JP16" (at 139.7 106.68 0)
-      (effects (font (size 1.27 1.27)))
-    )
-    (property "Value" "SolderJumper_2_Open" (at 139.7 104.14 0)
-      (effects (font (size 1.27 1.27)))
-    )
-    (property "Footprint" "Jumper:SolderJumper-2_P1.3mm_Open_TrianglePad1.0x1.5mm" (at 147.32 101.6 0)
-      (effects (font (size 1.27 1.27)) hide)
-    )
-    (property "Datasheet" "~" (at 147.32 101.6 0)
-      (effects (font (size 1.27 1.27)) hide)
-    )
-    (pin "2")
-    (pin "1")
-    (instances
-      (project "Main"
-        (path "/aa9d7141-7530-418f-853d-a56ee68433fb/dd025a71-f40c-48d2-8202-a120d14a823c"
-          (reference "JP16") (unit 1)
+      (project "Drive"
+        (path "/bf4fa0f7-7e40-4646-9c11-e04533c904d6/eede7486-c694-4c67-81d8-d20707e697df"
+          (reference "#PWR0105") (unit 1)
         )
       )
@@
         )
       )
+      (project "Drive"
+        (path "/bf4fa0f7-7e40-4646-9c11-e04533c904d6/eede7486-c694-4c67-81d8-d20707e697df"
+          (reference "C34") (unit 1)
+        )
+      )
     )
   )
   (symbol (lib_id "MyLibrary:Sensor_OpticalFlowSensor_PIM453") (at 167.64 93.98 0) (unit 1)
     (in_bom yes) (on_board yes) (dnp no)
-    (property "Reference" "U10" (at 137.16 114.3 0)
-      (effects (font (size 1.27 1.27)) (justify left))
-    )
-    (property "Value" "Sensor_OpticalFlowSensor_PIM453" (at 137.16 116.84 0)
+    (property "Reference" "U10" (at 144.78 76.2 0)
+      (effects (font (size 1.27 1.27)) (justify left))
+    )
+    (property "Value" "Sensor_OpticalFlowSensor_PIM573" (at 144.78 78.74 0)
       (effects (font (size 1.27 1.27)) (justify left))
     )
@@
           (reference "U10") (unit 1)
         )
+      )
+      (project "Drive"
+        (path "/bf4fa0f7-7e40-4646-9c11-e04533c904d6/eede7486-c694-4c67-81d8-d20707e697df"
+          (reference "U10") (unit 1)
+        )

Commit message: 無線&UI完成？
Other:
- note added: "配置時は裏向きになるのでフットプリント注意 表面につくけど裏向きになる"
Changed lines of the file:
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@@
     (effects (font (size 2.54 2.54) (thickness 0.254) bold) (justify left bottom))
+  )
+  (text "配置時は裏向きになるのでフットプリント注意\n表面につくけど裏向きになる" (at 119.38 142.24 0)
+    (effects (font (size 2.54 2.54)) (justify left bottom))
   )
   (hierarchical_label "Mouse_INT" (shape input) (at 139.7 106.68 180) (fields_autoplaced)

Commit message: ラズパイ基板とか
Parts:
- removed Q16: BSS138, Package_TO_SOT_SMD:SOT-23, symbol Device:Q_NMOS_GSD
- removed R63: 10k, Resistor_SMD:R_0402_1005Metric, symbol Device:R
Connections:
- net INT: now reaches U10.6 (INT)
Other:
- moved on the sheet: C26, U10

Commit message: シンボル・フットプリントMyLib->TomoshibiLib置き換え
Parts:
- U10: footprint MyLibrary:Sensor_OpticalFlowSensor_PIM453 -> TomoshibiLibrary:Sensor_OpticalFlowSensor_PIM453; symbol MyLibrary:Sensor_OpticalFlowSensor_PIM453 -> TomoshibiLibrary:Sensor_OpticalFlowSensor_PIM453
Changed lines of the file:
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@@
     )
   )
-  (symbol (lib_id "MyLibrary:Sensor_OpticalFlowSensor_PIM453") (at 154.94 93.98 0) (unit 1)
+  (symbol (lib_id "TomoshibiLibrary:Sensor_OpticalFlowSensor_PIM453") (at 154.94 93.98 0) (unit 1)
     (in_bom yes) (on_board yes) (dnp no)
     (property "Reference" "U10" (at 132.08 76.2 0)
@@
       (effects (font (size 1.27 1.27)) (justify left))
     )
-    (property "Footprint" "MyLibrary:Sensor_OpticalFlowSensor_PIM453" (at 158.75 105.41 0)
+    (property "Footprint" "TomoshibiLibrary:Sensor_OpticalFlowSensor_PIM453" (at 158.75 105.41 0)
       (effects (font (size 1.27 1.27)) (justify left) hide)
     )
