File: circuits/Drive/RS485_MD.kicad_sch (KiCad schematic)
At the start: 18 parts, among them J11 Conn_01x06_MountingPin, J12 Conn_01x06_MountingPin, Q14 S8550, U5 MAX3485, U6 MAX3485

Commit message: 無線&UI完成？
Parts:
- removed J11, J12: Conn_01x06_MountingPin, Connector_Molex:Molex_PicoBlade_53261-0671_1x06-1MP_P1.25mm_Horizontal, symbol Connector_Generic_MountingPin:Conn_01x06_MountingPin
- added J8, J9: Conn_01x05_MountingPin, Connector_Molex:Molex_PicoBlade_53261-0571_1x05-1MP_P1.25mm_Horizontal, symbol Connector_Generic_MountingPin:Conn_01x05_MountingPin
Connections:
- net GNDD: now also J8.1 (Pin_1), J8.MP (MountPin), J9.1 (Pin_1), J9.MP (MountPin)
- net RS485MD_RA: now also J8.4 (Pin_4), J9.4 (Pin_4)
- net RS485MD_RB: now also J8.5 (Pin_5), J9.5 (Pin_5)
- net RS485MD_TA: now also J8.2 (Pin_2), J9.2 (Pin_2)
- net RS485MD_TB: now also J8.3 (Pin_3), J9.3 (Pin_3)

Commit message: 更新
Parts:
- JP4, JP5: footprint Connector_PinHeader_2.54mm:PinHeader_1x02_P2.54mm_Vertical -> Jumper:SolderJumper-2_P1.3mm_Open_RoundedPad1.0x1.5mm
Changed lines of the file:
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@@
       (effects (font (size 1.27 1.27)))
     )
-    (property "Footprint" "Connector_PinHeader_2.54mm:PinHeader_1x02_P2.54mm_Vertical" (at 162.56 60.96 0)
+    (property "Footprint" "Jumper:SolderJumper-2_P1.3mm_Open_RoundedPad1.0x1.5mm" (at 162.56 60.96 0)
       (effects (font (size 1.27 1.27)) hide)
     )
@@
       (effects (font (size 1.27 1.27)))
     )
-    (property "Footprint" "Connector_PinHeader_2.54mm:PinHeader_1x02_P2.54mm_Vertical" (at 162.56 121.92 0)
-      (effects (font (size 1.27 1.27)) hide)
-    )
+    (property "Footprint" "Jumper:SolderJumper-2_P1.3mm_Open_RoundedPad1.0x1.5mm" (at 162.56 121.92 0)
+      (effects (font (size 1.27 1.27)) hide)
+    )
