File: circuits/Drive/UI.kicad_sch (KiCad schematic)
At the start: 11 parts, among them SW2 SW_SPST, SW3 SW_SPDT, SW8 SW_SPDT

Commit message: Driveほぼ完成
Parts:
- removed C25: 0.1uF, Capacitor_SMD:C_0402_1005Metric, symbol Device:C
- removed R61, R62: 10k, Resistor_SMD:R_0402_1005Metric, symbol Device:R
- removed SW2: SW_SPST, Button_Switch_SMD:SW_SPST_Omron_B3FS-100xP, symbol Switch:SW_SPST
- removed SW8: SW_SPDT, MyLibrary:SW_Slide_3P_SPDT, symbol Switch:SW_SPDT
- added R54, R55, R57, R58: 10k, Resistor_SMD:R_0402_1005Metric, symbol Device:R
- added SW3: SW_DIP_x04, Button_Switch_SMD:SW_DIP_SPSTx04_Slide_Copal_CHS-04B_W7.62mm_P1.27mm, symbol Switch:SW_DIP_x04
Connections:
- net +3.3V: now also SW3.5, SW3.6, SW3.7, SW3.8
- net GNDD: now also R54.1, R55.1, R57.1, R58.1
- new net DIP_SW0: R54.2, SW3.1
- new net DIP_SW1: R55.2, SW3.2
- new net DIP_SW2: R57.2, SW3.3
- new net DIP_SW3: R58.2, SW3.4
- no-connect marks 2 -> 1
Other:
- note added: "DIPスイッチ"
- note removed: "タクトスイッチ"
- moved on the sheet: R63, SW3

Commit message: ラズパイ基板とか
Parts:
- R59, R60: value 2k -> 1k
Connections:
- net DIP_SW0 renamed DIPSW0
- net DIP_SW1 renamed DIPSW1
- net DIP_SW2 renamed DIPSW2
- net DIP_SW3 renamed DIPSW3
- net Slide_SW0 renamed SlideSW0
Changed lines of the file:
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@@
     (effects (font (size 2.54 2.54)) (justify left bottom))
   )
-  (hierarchical_label "Slide_SW0" (shape input) (at 132.08 78.74 0) (fields_autoplaced)
+  (hierarchical_label "SlideSW0" (shape input) (at 132.08 78.74 0) (fields_autoplaced)
+    (effects (font (size 1.27 1.27)) (justify left))
+  )
+  (hierarchical_label "DIPSW2" (shape input) (at 144.78 116.84 0) (fields_autoplaced)
     (effects (font (size 1.27 1.27)) (justify left))
   )
@@
     (effects (font (size 1.27 1.27)) (justify right))
   )
-  (hierarchical_label "DIP_SW3" (shape input) (at 144.78 119.38 0) (fields_autoplaced)
+  (hierarchical_label "DIPSW1" (shape input) (at 144.78 114.3 0) (fields_autoplaced)
     (effects (font (size 1.27 1.27)) (justify left))
   )
@@
     (effects (font (size 1.27 1.27)) (justify right))
   )
-  (hierarchical_label "DIP_SW0" (shape input) (at 144.78 111.76 0) (fields_autoplaced)
-    (effects (font (size 1.27 1.27)) (justify left))
-  )
-  (hierarchical_label "DIP_SW1" (shape input) (at 144.78 114.3 0) (fields_autoplaced)
-    (effects (font (size 1.27 1.27)) (justify left))
-  )
-  (hierarchical_label "DIP_SW2" (shape input) (at 144.78 116.84 0) (fields_autoplaced)
+  (hierarchical_label "DIPSW0" (shape input) (at 144.78 111.76 0) (fields_autoplaced)
+    (effects (font (size 1.27 1.27)) (justify left))
+  )
+  (hierarchical_label "DIPSW3" (shape input) (at 144.78 119.38 0) (fields_autoplaced)
     (effects (font (size 1.27 1.27)) (justify left))
   )
@@
       (effects (font (size 1.27 1.27)))
     )
-    (property "Value" "2k" (at 124.46 60.96 90)
+    (property "Value" "1k" (at 124.46 60.96 90)
       (effects (font (size 1.27 1.27)))
     )
@@
       (effects (font (size 1.27 1.27)))
     )
-    (property "Value" "2k" (at 124.46 50.8 90)
-      (effects (font (size 1.27 1.27)))
-    )
+    (property "Value" "1k" (at 124.46 50.8 90)
+      (effects (font (size 1.27 1.27)))
+    )

Commit message: PDFプロット
Parts:
- added D12: LightGreen, LED_SMD:LED_0603_1608Metric_Pad1.05x0.95mm_HandSolder, symbol Device:LED
- added D13: Red, LED_SMD:LED_0603_1608Metric_Pad1.05x0.95mm_HandSolder, symbol Device:LED
- added D14: Yellow, LED_SMD:LED_0603_1608Metric_Pad1.05x0.95mm_HandSolder, symbol Device:LED
- added Q18: BSS138, Package_TO_SOT_SMD:SOT-23, symbol Device:Q_NMOS_GSD
- added R63, R66, R67: 1k, Resistor_SMD:R_0402_1005Metric, symbol Device:R
- added R69: 10k, Resistor_SMD:R_0402_1005Metric, symbol Device:R
- D10, D11: value Red -> Blue
- renumbered R60 to R52, R59 to R53, R63 to R56, SW3 to SW4
Connections:
- net +3.3V: now also R66.1
- net DIPSW0: no longer R54.2
- net DIPSW1: no longer SW3.2
- net DIPSW2: no longer SW3.3
- net DIPSW3: no longer SW3.4
- net GNDD: now also D12.1 (K), D13.1 (K), D14.1 (K), Q18.2 (S), R69.2
- net LED0 renamed LED_B0
- net LED1 renamed LED_B1
- new net: D13.2 (A), Q18.3 (D), R66.2
- new net: R54.2, SW3.4
- new net: D14.2 (A), R67.1
- new net: SW3.2, SW3.3
- new net: D12.2 (A), R63.1
- new net LED_LG0: R63.2
- new net LED_Y0: R67.2
- new net LED_nR0: Q18.1 (G), R69.1
Other:
- note added: "Error"
- note added: "Indicator"
- note added: "Running"
- note added: "not Running"

Commit message: panelフットプリント配置
Connections:
- net DIPSW0: now also R54.2
- net DIPSW1: now also SW3.2
- net DIPSW2: now also SW3.3
- net DIPSW3: now also SW3.4
Changed lines of the file:
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@@
   (junction (at 106.68 116.84) (diameter 0) (color 0 0 0 0)
   )
+  (junction (at 127 111.76) (diameter 0) (color 0 0 0 0)
+  )
   (junction (at 106.68 114.3) (diameter 0) (color 0 0 0 0)
   )
@@
   )
   (junction (at 129.54 86.36) (diameter 0) (color 0 0 0 0)
-  )
-  (junction (at 142.24 132.08) (diameter 0) (color 0 0 0 0)
   )
   (junction (at 142.24 119.38) (diameter 0) (color 0 0 0 0)
@@
     (stroke (width 0) (type default))
   )
+  (wire (pts (xy 124.46 119.38) (xy 142.24 119.38))
+    (stroke (width 0) (type default))
+  )
   (wire (pts (xy 142.24 129.54) (xy 137.16 129.54))
     (stroke (width 0) (type default))
@@
     (stroke (width 0) (type default))
   )
-  (wire (pts (xy 124.46 114.3) (xy 127 114.3))
-    (stroke (width 0) (type default))
-  )
-  (wire (pts (xy 142.24 132.08) (xy 147.32 132.08))
-    (stroke (width 0) (type default))
-  )
   (wire (pts (xy 195.58 111.76) (xy 199.39 111.76))
     (stroke (width 0) (type default))
@@
     (stroke (width 0) (type default))
   )
-  (wire (pts (xy 124.46 111.76) (xy 144.78 111.76))
+  (wire (pts (xy 124.46 111.76) (xy 127 111.76))
     (stroke (width 0) (type default))
   )
@@
     (stroke (width 0) (type default))
   )
-  (wire (pts (xy 129.54 119.38) (xy 142.24 119.38))
-    (stroke (width 0) (type default))
-  )
   (wire (pts (xy 207.01 111.76) (xy 209.55 111.76))
     (stroke (width 0) (type default))
@@
     (stroke (width 0) (type default))
   )
-  (wire (pts (xy 142.24 129.54) (xy 147.32 129.54))
-    (stroke (width 0) (type default))
-  )
   (wire (pts (xy 127 86.36) (xy 129.54 86.36))
     (stroke (width 0) (type default))
@@
     (stroke (width 0) (type default))
   )
-  (wire (pts (xy 129.54 114.3) (xy 132.08 114.3))
+  (wire (pts (xy 124.46 114.3) (xy 132.08 114.3))
     (stroke (width 0) (type default))
   )
@@
     (stroke (width 0) (type default))
   )
-  (wire (pts (xy 127 120.65) (xy 127 119.38))
+  (wire (pts (xy 127 111.76) (xy 144.78 111.76))
+    (stroke (width 0) (type default))
+  )
+  (wire (pts (xy 127 111.76) (xy 127 120.65))
     (stroke (width 0) (type default))
   )
@@
     (stroke (width 0) (type default))
   )
-  (wire (pts (xy 129.54 116.84) (xy 137.16 116.84))
-    (stroke (width 0) (type default))
-  )
   (polyline (pts (xy 96.52 139.7) (xy 160.02 139.7))
     (stroke (width 0.5) (type solid))
@@
     (stroke (width 0) (type default))
   )
-  (wire (pts (xy 127 114.3) (xy 127 116.84))
-    (stroke (width 0) (type default))
-  )
   (wire (pts (xy 132.08 129.54) (xy 137.16 129.54))
     (stroke (width 0) (type default))
@@
     (stroke (width 0) (type default))
   )
-  (wire (pts (xy 124.46 116.84) (xy 127 116.84))
+  (wire (pts (xy 124.46 116.84) (xy 137.16 116.84))
     (stroke (width 0) (type default))
   )
@@
     (stroke (width 0) (type default))
   )
-  (wire (pts (xy 124.46 119.38) (xy 127 119.38))
-    (stroke (width 0) (type default))
-  )

Commit message: シンボル・フットプリントMyLib->TomoshibiLib置き換え
Parts:
- SW4: footprint MyLibrary:SW_Slide_3P_SPDT -> TomoshibiLibrary:SW_Slide_3P_SPDT
Changed lines of the file:
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@@
       (effects (font (size 1.27 1.27)) (justify left))
     )
-    (property "Footprint" "MyLibrary:SW_Slide_3P_SPDT" (at 121.92 83.82 0)
+    (property "Footprint" "TomoshibiLibrary:SW_Slide_3P_SPDT" (at 121.92 83.82 0)
       (effects (font (size 1.27 1.27)) hide)
     )

Commit message: 更新
Parts:
- removed Q18: BSS138, Package_TO_SOT_SMD:SOT-23, symbol Device:Q_NMOS_GSD
- added H3, H4: MountingHole_Pad, TestPoint:TestPoint_Pad_1.5x1.5mm, symbol Mechanical:MountingHole_Pad
- added Q18: 2N7002, Package_TO_SOT_SMD:SOT-23, symbol Transistor_FET:2N7002
- SW4: footprint TomoshibiLibrary:SW_Slide_3P_SPDT -> TomoshibiLibrary:SW_Slide_SPDT_SSSS213202
Connections:
- net GNDD: now also Q18.2 (S)
- net LED_B0: now also H3.1
- net LED_B1: now also H4.1
- net LED_nR0: now also Q18.1 (G)
- net at D13.2 (A), R66.2: now also Q18.3 (D)
Changed lines of the file:
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@@
   (junction (at 137.16 129.54) (diameter 0) (color 0 0 0 0)
   )
+  (junction (at 106.68 116.84) (diameter 0) (color 0 0 0 0)
+  )
+  (junction (at 127 111.76) (diameter 0) (color 0 0 0 0)
+  )
+  (junction (at 106.68 114.3) (diameter 0) (color 0 0 0 0)
+  )
+  (junction (at 215.9 78.74) (diameter 0) (color 0 0 0 0)
+  )
+  (junction (at 132.08 114.3) (diameter 0) (color 0 0 0 0)
+  )
+  (junction (at 132.08 129.54) (diameter 0) (color 0 0 0 0)
+  )
+  (junction (at 119.38 48.26) (diameter 0) (color 0 0 0 0)
+  )
+  (junction (at 119.38 58.42) (diameter 0) (color 0 0 0 0)
+  )
   (junction (at 200.66 83.82) (diameter 0) (color 0 0 0 0)
-  )
-  (junction (at 106.68 116.84) (diameter 0) (color 0 0 0 0)
-  )
-  (junction (at 127 111.76) (diameter 0) (color 0 0 0 0)
-  )
-  (junction (at 106.68 114.3) (diameter 0) (color 0 0 0 0)
-  )
-  (junction (at 215.9 78.74) (diameter 0) (color 0 0 0 0)
-  )
-  (junction (at 132.08 114.3) (diameter 0) (color 0 0 0 0)
-  )
-  (junction (at 132.08 129.54) (diameter 0) (color 0 0 0 0)
   )
   (junction (at 137.16 116.84) (diameter 0) (color 0 0 0 0)
@@
     (stroke (width 0) (type default))
   )
+  (wire (pts (xy 119.38 58.42) (xy 120.65 58.42))
+    (stroke (width 0) (type default))
+  )
   (wire (pts (xy 132.08 129.54) (xy 127 129.54))
     (stroke (width 0) (type default))
@@
     (stroke (width 0) (type default))
   )
+  (wire (pts (xy 119.38 48.26) (xy 120.65 48.26))
+    (stroke (width 0) (type default))
+  )
   (wire (pts (xy 106.68 111.76) (xy 109.22 111.76))
     (stroke (width 0) (type default))
@@
     (stroke (width 0.5) (type solid))
   )
-  (wire (pts (xy 116.84 58.42) (xy 120.65 58.42))
+  (wire (pts (xy 116.84 58.42) (xy 119.38 58.42))
     (stroke (width 0) (type default))
   )
@@
     (stroke (width 0) (type default))
   )
-  (wire (pts (xy 116.84 48.26) (xy 120.65 48.26))
+  (wire (pts (xy 116.84 48.26) (xy 119.38 48.26))
     (stroke (width 0) (type default))
   )
@@
     )
   )
-  (symbol (lib_name "Q_NMOS_GSD_1") (lib_id "Device:Q_NMOS_GSD") (at 205.74 83.82 0) (unit 1)
-    (in_bom yes) (on_board yes) (dnp no)
-    (property "Reference" "Q18" (at 203.2 88.9 0)
-      (effects (font (size 1.27 1.27)) (justify left))
-    )
-    (property "Value" "BSS138" (at 203.2 91.44 0)
-      (effects (font (size 1.27 1.27)) (justify left))
-    )
-    (property "Footprint" "Package_TO_SOT_SMD:SOT-23" (at 210.82 81.28 0)
-      (effects (font (size 1.27 1.27)) hide)
-    )
-    (property "Datasheet" "~" (at 205.74 83.82 0)
-      (effects (font (size 1.27 1.27)) hide)
-    )
-    (pin "1")
-    (pin "2")
-    (pin "3")
-    (instances
-      (project "Drive"
-        (path "/bf4fa0f7-7e40-4646-9c11-e04533c904d6/dba30bfe-4311-47ce-87e3-759a65c4e558"
-          (reference "Q18") (unit 1)
+  (symbol (lib_id "Mechanical:MountingHole_Pad") (at 119.38 45.72 0) (mirror y) (unit 1)
+    (in_bom yes) (on_board yes) (dnp no)
+    (property "Reference" "H3" (at 104.14 43.18 0)
+      (effects (font (size 1.27 1.27)) (justify right))
+    )
+    (property "Value" "MountingHole_Pad" (at 104.14 40.64 0)
+      (effects (font (size 1.27 1.27)) (justify right))
+    )
+    (property "Footprint" "TestPoint:TestPoint_Pad_1.5x1.5mm" (at 119.38 45.72 0)
+      (effects (font (size 1.27 1.27)) hide)
+    )
+    (property "Datasheet" "~" (at 119.38 45.72 0)
+      (effects (font (size 1.27 1.27)) hide)
+    )
+    (pin "1")
+    (instances
+      (project "Drive"
+        (path "/bf4fa0f7-7e40-4646-9c11-e04533c904d6/dba30bfe-4311-47ce-87e3-759a65c4e558"
+          (reference "H3") (unit 1)
         )
       )
@@
         (path "/bf4fa0f7-7e40-4646-9c11-e04533c904d6/dba30bfe-4311-47ce-87e3-759a65c4e558"
           (reference "R54") (unit 1)
+        )
+      )
+    )
+  )
+  (symbol (lib_id "Transistor_FET:2N7002") (at 205.74 83.82 0) (unit 1)
+    (in_bom yes) (on_board yes) (dnp no)
+    (property "Reference" "Q18" (at 198.12 76.2 0)
+      (effects (font (size 1.27 1.27)) (justify left))
+    )
+    (property "Value" "2N7002" (at 198.12 78.74 0)
+      (effects (font (size 1.27 1.27)) (justify left))
+    )
+    (property "Footprint" "Package_TO_SOT_SMD:SOT-23" (at 210.82 85.725 0)
+      (effects (font (size 1.27 1.27) italic) (justify left) hide)
+    )
+    (property "Datasheet" "https://www.onsemi.com/pub/Collateral/NDS7002A-D.PDF" (at 210.82 87.63 0)
+      (effects (font (size 1.27 1.27)) (justify left) hide)
+    )
+    (pin "3")
+    (pin "1")
+    (pin "2")
+    (instances
+      (project "Drive"
+        (path "/bf4fa0f7-7e40-4646-9c11-e04533c904d6/dba30bfe-4311-47ce-87e3-759a65c4e558"
+          (reference "Q18") (unit 1)
         )
       )
@@
       (effects (font (size 1.27 1.27)) (justify left))
     )
-    (property "Footprint" "TomoshibiLibrary:SW_Slide_3P_SPDT" (at 121.92 83.82 0)
+    (property "Footprint" "TomoshibiLibrary:SW_Slide_SPDT_SSSS213202" (at 121.92 83.82 0)
       (effects (font (size 1.27 1.27)) hide)
     )
@@
         )
       )
+    )
+  )
+  (symbol (lib_id "Mechanical:MountingHole_Pad") (at 119.38 55.88 0) (mirror y) (unit 1)
+    (in_bom yes) (on_board yes) (dnp no)
+    (property "Reference" "H4" (at 104.14 53.34 0)
+      (effects (font (size 1.27 1.27)) (justify right))
+    )
+    (property "Value" "MountingHole_Pad" (at 104.14 50.8 0)
+      (effects (font (size 1.27 1.27)) (justify right))
+    )
+    (property "Footprint" "TestPoint:TestPoint_Pad_1.5x1.5mm" (at 119.38 55.88 0)
+      (effects (font (size 1.27 1.27)) hide)
+    )
+    (property "Datasheet" "~" (at 119.38 55.88 0)
+      (effects (font (size 1.27 1.27)) hide)
+    )
+    (pin "1")
+    (instances
+      (project "Drive"
+        (path "/bf4fa0f7-7e40-4646-9c11-e04533c904d6/dba30bfe-4311-47ce-87e3-759a65c4e558"
+          (reference "H4") (unit 1)
+        )
+      )
