File: circuits/Drive/Drive.kicad_pcb (KiCad board)
At the start: 2 copper layers, 170 parts, among them IC1 DCDC_MPM3620A, J1 Conn_01x14_Pin, J10 Conn_01x06_MountingPin, J13 Conn_01x06_MountingPin, J2 Conn_01x02_Male, J3 Conn_01x02_Male, J4 Conn_01x02_Male, J5 Conn_01x02_Male, J6 USB_C_Receptacle_USB2.0, J7 Conn_01x02_Male, J8 Conn_01x05_MountingPin, J9 Conn_01x05_MountingPin, Q1 SSM3J332R, Q10 S8550, Q11 SSM3J332R, Q12 S8550, Q13 S8550, Q14 S8550, Q15 BSS138, Q16 BSS138, Q17 S8550, Q18 BSS138, Q2 S8550, Q3 SSM3J332R, Q4 S8550, Q5 BSS138, Q6 SSM3J332R, Q7 SSM6J808R, Q8 BSS138, Q9 SSM6J808R, SW1 SW_SPST, SW2 SW_SPDT_White, SW3 SW_DIP_x04, SW4 SW_SPDT, U1 AZ1117CH-3.3, U10 Sensor_OpticalFlowSensor_PIM5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, U11 MAX3485, U12 MAX3485, U2 STM32F446RETx, U3 MAX3485, U4 MAX3485, U5 MAX3485, U6 MAX3485, U7 BNO055, Y2 16MHz

Commit message: 更新
Parts:
- removed IC1: DCDC_MPM3620A, TomoshibiLibrary:DCDC_MPM3620A
- removed J6: USB_C_Receptacle_USB2.0, Connector_USB:USB_C_Receptacle_G-Switch_GT-USB-7010ASV
- removed R2: 10k, Resistor_SMD:R_0402_1005Metric
- removed R5: 200k, Resistor_SMD:R_0402_1005Metric
- added C12: 4.7uF, Capacitor_SMD:C_0603_1608Metric, B.Cu at (-11.6, 16.9)
- added C13: 1uF, Capacitor_SMD:C_0402_1005Metric, B.Cu at (-11.0, 18.1)
- added C14: 2.2uF, Capacitor_SMD:C_0402_1005Metric, B.Cu at (4.66, 11.4)
- added C15: 2.2uF, Capacitor_SMD:C_0402_1005Metric, B.Cu at (8.28, 26.2)
- added C22: 47uF, Capacitor_SMD:CP_Elec_6.3x5.4, F.Cu at (1.42, -18.8)
- added C23: 47uF, Capacitor_SMD:CP_Elec_6.3x5.4, F.Cu at (-6.37, -17.6)
- added C25: 22uF, Capacitor_SMD:C_0805_2012Metric, B.Cu at (16.4, -7.50)
- added C26: 22uF, Capacitor_SMD:C_0805_2012Metric, B.Cu at (17.9, 6.53)
- added C32: 100uF, TomoshibiLibrary:Capacitor_Alum_Radial_5.0x11.0mm_Horizontal, F.Cu at (30.0, -0.14)
- added C33: 100uF, TomoshibiLibrary:Capacitor_Alum_Radial_5.0x11.0mm_Horizontal, F.Cu at (-30.0, 0.14)
- added C37: 47uF, Capacitor_SMD:CP_Elec_6.3x5.4, F.Cu at (12.5, -55.2)
- added C38: 47uF, Capacitor_SMD:CP_Elec_6.3x5.4, F.Cu at (-14.2, -18.9)
- added C41: 22uF, Capacitor_SMD:C_0805_2012Metric, B.Cu at (-3.40, -17.8)
- added H1: MountingHole_Pad, MountingHole:MountingHole_3.2mm_M3_Pad_Via, F.Cu at (-9.55, -68.7)
- added H2: MountingHole_Pad, MountingHole:MountingHole_3.2mm_M3_Pad_Via, F.Cu at (9.54, -68.7)
- added H3: MountingHole_Pad, TestPoint:TestPoint_Pad_1.5x1.5mm, F.Cu at (-3.82, 29.5)
- added H4: MountingHole_Pad, TestPoint:TestPoint_Pad_1.5x1.5mm, F.Cu at (3.06, 28.0)
- added J11: Conn_01x02_Pin, Connector_Molex:Molex_SPOX_5268-02A_1x02_P2.50mm_Horizontal, B.Cu at (2.91, 37.2)
- added SW5: SW_SPST, Button_Switch_THT:SW_PUSH_1P1T_6x3.5mm_H4.3_APEM_MJTP1243, B.Cu at (-3.25, -71.6)
- added U8: STM32H723VGTx, Package_QFP:LQFP-100_14x14mm_P0.5mm, B.Cu at (-1.40, 21.6)
- C1, C10, C16, C17, C18, C19, C2, C20, C21, C24, C27, C28, C29, C3, C30, C31, C34, C35, C36, C4, C40, C5, C6, C7, C8, D1, D2, D3, D4, D5, D6, J1, J8, J9, Q1, Q10, Q11, Q12, Q13, Q14, Q17, Q2, Q3, Q4, Q6, R1, R13, R14, R15, R16, R17, R18, R19, R20, R21, R22, R23, R24, R25, R26, R27, R28, R29, R3, R30, R31, R32, R33, R34, R35, R36, R37, R38, R39, R4, R40, R41, R42, R43, R44, R45, R46, R47, R48, R49, R50, R51, R52, R53, R54, R55, R56, R57, R58, R59, R6, R60, R61, R62, R63, R64, R65, R66, R67, R68, R69, R7, R71, R72, R73, R74, R75, R76, R77, R78, R79, R8, R9, U1, U10, U11, U12, U3, U4, U5, U6, Y2: moved to B.Cu
- C11: value 4.7uF -> 1uF; footprint Capacitor_SMD:C_0603_1608Metric -> Capacitor_SMD:C_0402_1005Metric; moved to B.Cu
- C9: value 1uF -> 0.1uF; moved to B.Cu
- J10, J13: footprint Connector_Molex:Molex_PicoBlade_53261-0671_1x06-1MP_P1.25mm_Horizontal -> Connector_Molex:Molex_PicoBlade_53398-0671_1x06-1MP_P1.25mm_Vertical
- J2, J3, J4, J5: value Conn_01x02_Male -> Conn_01x02_Pin; footprint Connector_Molex:Molex_SPOX_5267-02A_1x02_P2.50mm_Vertical -> Connector_Molex:Molex_SPOX_5268-02A_1x02_P2.50mm_Horizontal; moved to B.Cu
- J7: value Conn_01x02_Male -> USB_C_Receptacle_PowerOnly_6P; footprint Connector_Molex:Molex_SPOX_5267-02A_1x02_P2.50mm_Vertical -> Connector_USB:USB_C_Receptacle_GCT_USB4125-xx-x_6P_TopMnt_Horizontal
- JP4, JP5: footprint Connector_PinHeader_2.54mm:PinHeader_1x02_P2.54mm_Vertical -> Jumper:SolderJumper-2_P1.3mm_Open_RoundedPad1.0x1.5mm; moved to B.Cu
- L1: value 22uH -> 1uH; footprint TomoshibiLibrary:Inductor_CDPH4D19F -> Inductor_SMD:L_0603_1608Metric; moved to B.Cu
- Q15, Q16, Q18, Q5, Q8: value BSS138 -> 2N7002; moved to B.Cu
- R10: value 100k -> 10k; moved to B.Cu
- R11: value 12k -> 20k; moved to B.Cu
- R12: value 2.2k -> 5.1k; moved to B.Cu
- SW4: footprint TomoshibiLibrary:SW_Slide_3P_SPDT -> TomoshibiLibrary:SW_Slide_SPDT_SSSS213202
- U2: value STM32F446RETx -> DCDC_TPSM336x5; footprint Package_QFP:LQFP-64_10x10mm_P0.5mm -> TomoshibiLibrary:DCDC_TPSM336x5; moved to B.Cu
- moved SW2 199.6 mm to (-41.3, 3.24), turned to -135 degrees
- moved L1 186.6 mm to (-6.05, -21.2), turned to -90 degrees
- moved Q7 184.1 mm to (-8.40, -24.4)
- moved Q9 183.0 mm to (-4.80, -24.4), turned to -90 degrees
- moved R68 168.9 mm to (5.45, -70.5)
- moved C10 165.6 mm to (5.20, -72.0), turned to -90 degrees
- moved J9 163.1 mm to (-44.5, 0.00), turned to 90 degrees
- moved C30 151.8 mm to (-20.7, 3.50), turned to 90 degrees
- moved J1 146.7 mm to (-0.30, 41.8), turned to -135 degrees
- moved U6 144.7 mm to (-16.4, 6.47), turned to 180 degrees
- moved JP5 144.2 mm to (-21.4, 7.97), turned to 90 degrees
- moved C29 141.5 mm to (-19.6, 16.2), turned to -90 degrees
- moved Q14 137.7 mm to (-12.0, 12.6), turned to 90 degrees
- moved R43 137.7 mm to (-11.6, 15.3), turned to 180 degrees
- moved R51 137.3 mm to (-21.1, 5.85)
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Connections:
- C11 pad 1: Net-(U2-VCAP_1) -> Net-(U2-RT)
- C9 pad 1: GND -> +3.3V
- C9 pad 2: +3.3V -> GND
- Q15 pad 1: Main->RST_BNO -> Main->INT_Mouse
- Q15 pad 3: RST_BNO -> INT_Mouse
- Q16 pad 1: Main->INT_Mouse -> Main->RST_BNO
- Q16 pad 3: INT_Mouse -> RST_BNO
- R10 pad 1: /Power/PG -> Net-(U2-RT)
- R10 pad 2: Net-(IC1-VCC) -> /Power/PG
- R11 pad 1: Net-(IC1-FB) -> Net-(U2-FB)
- R12 pad 2: Net-(IC1-FB) -> Net-(U2-FB)
- R20 pad 1: Net-(SW2-A) -> Net-(SW2-C)
- R64 pad 2: Net-(J6-CC2) -> Net-(J7-CC2)
- R65 pad 2: Net-(J6-CC1) -> Net-(J7-CC1)
- SW2 pad 1: Net-(SW2-A) -> unconnected-(SW2-A-Pad1)
- SW2 pad 3: unconnected-(SW2-C-Pad3) -> Net-(SW2-C)
- U2 pad 1: +3.3V -> /Power/PG
- U2 pad 10: unconnected-(U2-PC2-Pad10) -> GND
- U2 pad 11: unconnected-(U2-PC3-Pad11) -> Net-(U2-RT)
- U2 pad 2: unconnected-(U2-PC13-Pad2) -> VCC
- U2 pad 3: unconnected-(U2-PC14-Pad3) -> VCC
- U2 pad 4: unconnected-(U2-PC15-Pad4) -> /Power/Vout
- U2 pad 5: HSE_IN -> unconnected-(U2-SW-Pad5)
- U2 pad 6: HSE_OUT -> unconnected-(U2-SW-Pad6)
- U2 pad 7: NRST -> unconnected-(U2-BOOT-Pad7)
- U2 pad 8: unconnected-(U2-PC0-Pad8) -> Net-(U2-RT)
- U2 pad 9: unconnected-(U2-PC1-Pad9) -> Net-(U2-FB)
Routing:
- net +3.3V: track 0.00 -> 362.9 mm, vias 0 -> 24
- net SHDN/BOOT: track 0.00 -> 133.3 mm
- net GND: track 0.00 -> 115.9 mm, vias 0 -> 3
- net /RS485_MD/RS485MD_TB: track 0.00 -> 113.9 mm, vias 0 -> 3
- net /RS485_MD/RS485MD_TA: track 0.00 -> 112.2 mm, vias 0 -> 3
- net /RS485_MD/RS485MD_RA: track 0.00 -> 107.2 mm, vias 0 -> 3
- net /RS485_MD/RS485MD_RB: track 0.00 -> 105.4 mm, vias 0 -> 3
- net +5V: track 0.00 -> 85.7 mm, vias 0 -> 10
- net SlideSW0: track 0.00 -> 64.3 mm, vias 0 -> 2
- net Net-(Q1-G): track 0.00 -> 62.4 mm, vias 0 -> 3
- net /Power/S-S: track 0.00 -> 61.1 mm, vias 0 -> 4
- net Net-(Q9-G): track 0.00 -> 58.8 mm, vias 0 -> 3
- net DIPSW3: track 0.00 -> 51.3 mm, vias 0 -> 2
- net DIPSW0: track 0.00 -> 51.0 mm, vias 0 -> 2
- net DIPSW2: track 0.00 -> 50.8 mm, vias 0 -> 2
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- added copper zone on B.Cu, net +3.3V
- added copper zone on B.Cu, net +5V
- added copper zone on F.Cu, net +BATT
- added copper zone on F.Cu, net /Power/S-S
- added copper zone on B.Cu, net /Power/VSYS
- added copper zone on B.Cu, net /Power/Vout
- added copper zone on B.Cu, net GND
- added copper zone on F.Cu, net GND
- added copper zone on B.Cu, net Net-(D5-K)
- added copper zone on B.Cu, net VBUS
- added copper zone on F.Cu, net VBUS
- added copper zone on B.Cu, net VCC
- added copper zone on B.Cu, net VDD
- added copper zone on F.Cu, net VDD
Other:
- board outline added: 102.2 x 125.7 mm
- board text added: "BNOのピン名"

Commit message: raspi基板回路図
Parts:
- D1: moved to F.Cu
- SW2: footprint TomoshibiLibrary:SW_Slide_SPDT_White -> TomoshibiLibrary:SW_Slide_SPDT_IS-1235-G
- moved D1 15.0 mm to (3.91, 40.7), turned to 135 degrees
- moved R62 9.23 mm to (-1.49, 38.6), turned to 0 degrees
- moved R20 2.98 mm to (-35.8, 10.2)
- moved R21 2.50 mm to (-34.6, 9.30), turned to 180 degrees
- moved Q8 1.86 mm to (-33.6, 11.8)
- moved R12 1.51 mm to (-11.3, -14.2), turned to 0 degrees
- moved R22 1.00 mm to (-36.5, 10.9)
- moved SW1 0.71 mm to (6.43, 39.3)
- moved R11 0.23 mm to (-10.4, -15.2)
- moved C11 0.20 mm to (-9.90, -13.8)
- moved R10 0.10 mm to (-9.90, -18.3)
- moved D7 0.08 mm to (34.8, -9.65)
- moved D9 0.07 mm to (32.5, -11.8)
- moved R29 0.06 mm to (-15.3, -15.9)
- moved R30 0.06 mm to (-16.4, -14.9)
Connections:
- net CSx_Mouse renamed CS2_Mouse
- net MISOx renamed MISO2
- net MOSIx renamed MOSI2
- net MainRXx_RS485MDTX renamed MainRX2_RS485MDTX
- net MainRXx_RS485RingXTX renamed MainRX1_RS485RingXTX
- net MainRXx_RS485RingYTX renamed MainRX4_RS485RingYTX
- net MainTXx_RS485MDRX renamed MainTX2_RS485MDRX
- net MainTXx_RS485RingXRX renamed MainTX1_RS485RingXRX
- net MainTXx_RS485RingYRX renamed MainTX4_RS485RingYRX
- net SCLKx renamed SCLK2
- net SCLx renamed SCL4
- net SDAx renamed SDA4
Routing:
- net GND: track 115.9 -> 33.5 mm, vias 3 -> 810
- net (no net): track 35.0 -> 0.00 mm, vias 5 -> 0
- net +3.3V: track 362.9 -> 351.1 mm, vias 24 -> 21
- net +BATT: track 44.6 -> 38.9 mm, vias 8 -> 21
- net Net-(Q9-G): track 58.8 -> 55.5 mm
- net NRST: track 40.4 -> 41.6 mm
- net /RS485_MD/RS485MD_TB: track 113.9 -> 115.0 mm
- net /RS485_MD/RS485MD_TA: track 112.2 -> 113.3 mm
- net Net-(D1-K): track 10.9 -> 9.85 mm
- net Net-(Q8-D): track 2.35 -> 2.90 mm

Commit message: 発注_第一弾
Drive, 1stLayer_Power, 2ndLayer_3rdLayer
を発注
Parts:
- removed TP1, TP2: TestPoint, TestPoint:TestPoint_THTPad_D2.0mm_Drill1.0mm
- moved R72 170.9 mm to (133.8, 142.9)
- moved R78 170.8 mm to (140.5, 148.5)
- moved R75 170.8 mm to (141.8, 148.5)
- moved R74 170.7 mm to (141.7, 149.8)
- moved R69 170.7 mm to (131.2, 147.1)
- moved R62 170.7 mm to (125.6, 152.6)
- moved C2 170.7 mm to (132.5, 147.6)
- moved C13 170.7 mm to (116.0, 132.1)
- moved C36 170.7 mm to (145.2, 146.1)
- moved D12 170.7 mm to (124.3, 145.3)
- moved H4 170.7 mm to (130.1, 142.0)
- moved R46 170.7 mm to (112.0, 131.6)
- moved R52 170.7 mm to (126.5, 144.8)
- moved R66 170.7 mm to (129.9, 148.1)
- moved R67 170.7 mm to (124.0, 145.8)
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- renumbered J13 to J11, J11 to J6
Routing:
- net +BATT: track 38.9 -> 27.2 mm, vias 21 -> 40
- net GND: track 33.5 -> 42.7 mm, vias 810 -> 843
- net VCC: vias 0 -> 11
- added copper zone on B.Cu, net +BATT
- added copper zone on F.Cu, net VCC
Other:
- board text added: "+3V3"
- board text added: "+5V"
- board text added: "B0"
- board text added: "B1"
- board text added: "Designed by @cat_nekonekone"
- board text added: "GND"
- board text added: "IND"
- board text added: "JLCJLCJLCJLC"
- board text added: "LG0"
- board text added: "MD"
- board text added: "NRST"
- board text added: "PWR"
- board text added: "R0"
- board text added: "RING"
- board text added: "Tomoshibi"
- board text added: "Y0"
- board text added: "燈"
- board text removed: "BNOのピン名"
