File: circuits/Wireless/2ndLayer/RS485_RingNW.kicad_sch (KiCad schematic)
At the start: 30 parts, among them J13 Conn_01x06_MountingPin, J8 Conn_01x06_MountingPin, Q17 S8550, Q5 S8550, U11 MAX3485, U12 MAX3485, U14 MAX3485, U16 MAX3485

Commit message: 無線&UI完成？
Parts:
- added JP1, JP2, JP3, JP4: Jumper_2_Open, Connector_PinHeader_2.54mm:PinHeader_1x02_P2.54mm_Vertical, symbol Jumper:Jumper_2_Open
- renumbered C21 to C30, C22 to C31, C35 to C32, C36 to C33, J8 to J10, J13 to J11, Q5 to Q14, Q17 to Q15, R71 to R42, R78 to R43, R77 to R44, R87 to R45, R88 to R46, R79 to R47, R80 to R48, R90 to R49, R89 to R50, R71 to R51, R72 to R52, R73 to R53, R74 to R54, R75 to R55, R76 to R56, R77 to R57, R78 to R58, R79 to R59, U16 to U3, U14 to U4, U11 to U5, U12 to U6
Connections:
- net MainRX_RS485RingX_TX renamed MainRX_RS485X_TX
- net MainRX_RS485RingY_TX renamed MainRX_RS485Y_TX
- net MainTX_RS485RingX_RX renamed MainTX_RS485X_RX
- net MainTX_RS485RingY_RX renamed MainTX_RS485Y_RX
- net RS485RingX_RA renamed RS485X_RA
- net RS485X_RA: now also JP2.1 (A); no longer R50.1
- net RS485RingX_RB renamed RS485X_RB
- net RS485RingX_TA renamed RS485X_TA
- net RS485X_TA: now also JP1.1 (A); no longer R49.1
- net RS485RingX_TB renamed RS485X_TB
- net RS485RingY_RA renamed RS485Y_RA
- net RS485Y_RA: now also JP4.1 (A); no longer R59.1
- net RS485RingY_RB renamed RS485Y_RB
- net RS485RingY_TA renamed RS485Y_TA
- net RS485Y_TA: now also JP3.1 (A); no longer R58.1
- net RS485RingY_TB renamed RS485Y_TB
- new net: JP3.2 (B), R58.1
- new net: JP1.2 (B), R49.1
- new net: JP2.2 (B), R50.1
- new net: JP4.2 (B), R59.1
Other:
- moved on the sheet: R49, R50, R58, R59

Commit message: ラズパイ基板とか
Parts:
- removed C30, C31, C32, C33: 0.1uF, Capacitor_SMD:C_0402_1005Metric, symbol Device:C
- removed JP1, JP2, JP3, JP4: Jumper_2_Open, Connector_PinHeader_2.54mm:PinHeader_1x02_P2.54mm_Vertical, symbol Jumper:Jumper_2_Open
- removed Q15: S8550, Package_TO_SOT_SMD:SOT-23, symbol Device:Q_PNP_BEC
- removed R57: 2.2k, Resistor_SMD:R_0402_1005Metric, symbol Device:R
- removed R58, R59: 120, Resistor_SMD:R_0402_1005Metric, symbol Device:R
- added C11, C18, C20, C23: 0.1uF, Capacitor_SMD:C_0402_1005Metric, symbol Device:C
- added Q13: S8550, Package_TO_SOT_SMD:SOT-23, symbol Device:Q_PNP_BEC
- added R36: 10k, Resistor_SMD:R_0402_1005Metric, symbol Device:R
- added R4: 7.5k, Resistor_SMD:R_0603_1608Metric, symbol Device:R
- added R5: 20k, Resistor_SMD:R_0402_1005Metric, symbol Device:R
- R42, R51: value 7.5k -> 2.2k; footprint Resistor_SMD:R_0603_1608Metric -> Resistor_SMD:R_0402_1005Metric
- R43, R52: value 20k -> 2.2k
- R44, R53: value 10k -> 2.2k
- R46, R47, R55, R56: value 2.2k -> 120
- R48: value 2.2k -> 7.5k; footprint Resistor_SMD:R_0402_1005Metric -> Resistor_SMD:R_0603_1608Metric
- R49: value 120 -> 20k
- R50: value 120 -> 10k
Connections:
- net +3.3V: now also R42.1, R44.1, R51.1, R53.1, C11.1, C18.1, C20.1, C23.1, Q13.2 (E); no longer R45.1, R47.1, R54.1, R56.1
- net GNDD: now also R45.2, R49.2, R50.2, R54.2, C11.2, C18.2, C20.2, C23.2, R36.2, R5.2; no longer R44.2, R46.2, R48.2, R53.2, R55.2
- net MainTX_RS485X_RX: now also R4.2; no longer R42.2
- net MainTX_RS485Y_RX: now also R48.2; no longer R51.2
- net RS485X_RA: now also R44.2, R47.1; no longer R47.2
- net RS485X_RB: now also R45.1, R47.2; no longer R48.1, R50.2
- net RS485X_TA: now also R42.2, R46.1; no longer R45.2
- net RS485X_TB: now also R43.1, R46.2; no longer R46.1, R49.2
- net RS485Y_RA: now also R53.2, R56.1; no longer R56.2
- net RS485Y_RB: now also R54.1, R56.2
- net RS485Y_TA: now also R51.2, R55.1; no longer R54.2
- net RS485Y_TB: now also R52.1, R55.2; no longer R55.1
- net at Q14.1 (B): now also R48.1; no longer R42.1
- net at U3.2 (~{RE}), U3.3 (DE): now also Q13.3 (C), R5.1; no longer Q14.3 (C), R43.1
- net at U4.2 (~{RE}), U4.3 (DE): now also R36.1; no longer R44.1
- net at R49.1: now also Q14.3 (C), U5.2 (~{RE}), U5.3 (DE)
- net at R50.1: now also U6.2 (~{RE}), U6.3 (DE)
- new net: Q13.1 (B), R4.1
