File: circuits/Wireless/2ndLayer/TweLite.kicad_sch (KiCad schematic)
At the start: 12 parts, among them SW3 SW_SPST, SW4 SW_SPST, U2 TWE-L-WX

Commit message: ラズパイ基板とか
Parts:
- R39, R40: value 2k -> 1k
Connections:
- net Twe_LED0 renamed LED0
- net Twe_LED1 renamed LED1
- net Twe_PRG renamed PRG
- net Twe_RST renamed nRST
- net Twe_SET renamed SET
Other:
- moved on the sheet: D10, D11, R39, R40

Commit message: PDFプロット
Parts:
- D10, D11: value Red -> Blue
Changed lines of the file:
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@@
       (effects (font (size 1.27 1.27)))
     )
-    (property "Value" "Red" (at 101.6 119.38 0)
+    (property "Value" "Blue" (at 101.6 119.38 0)
       (effects (font (size 1.27 1.27)))
     )
@@
       (effects (font (size 1.27 1.27)))
     )
-    (property "Value" "Red" (at 101.6 129.54 0)
-      (effects (font (size 1.27 1.27)))
-    )
+    (property "Value" "Blue" (at 101.6 129.54 0)
+      (effects (font (size 1.27 1.27)))
+    )
