File: circuits/Wireless/2ndLayer/Power.kicad_sch (KiCad schematic)
At the start: 81 parts, among them IC1 DCDC_MPM3620A, J10 Conn_01x02_Male, J11 Conn_01x02_Male, J12 Conn_01x02_Male, J13 Conn_01x02_Male, J6 USB_C_Receptacle_USB2.0, J9 Conn_01x02_Male, Q16 SSM6J808R, Q17 SSM6J808R, Q18 SSM3J332R, Q19 S8550, Q2 BSS138, Q20 SSM3J332R, Q21 S8550, Q23 S8550, Q24 SSM3J332R, Q25 S8550, Q3 SSM3J332R, Q4 BSS138, SW1 SW_SPDT_White

Commit message: 無線&UI完成？
Parts:
- removed C32, C33, C37, C38, C39: 470uF, symbol Device:C_Polarized
- removed C40: 10uF, Capacitor_SMD:C_0805_2012Metric, symbol Device:C
- removed J10, J11, J12, J13, J9: Conn_01x02_Male, Connector_Molex:Molex_SPOX_5267-02A_1x02_P2.50mm_Vertical, symbol Connector:Conn_01x02_Male
- removed J6: USB_C_Receptacle_USB2.0, Connector_USB:USB_C_Receptacle_G-Switch_GT-USB-7010ASV, symbol Connector:USB_C_Receptacle_USB2.0
- removed R64, R65: 5.1k, Resistor_SMD:R_0402_1005Metric, symbol Device:R
- renumbered C1 to C12, C23 to C13, C2 to C14, C3 to C15, C4 to C16, C5 to C17, C6 to C19, C23 to C21, C8 to C22, C25 to C24, D1 to D2, D8 to D3, D2 to D4, D3 to D5, D4 to D6, D9 to D7, D5 to D8, D6 to D9, Q18 to Q1, Q23 to Q10, Q24 to Q11, Q25 to Q12, Q19 to Q2, Q20 to Q3, Q21 to Q4, Q2 to Q5, Q3 to Q6, Q17 to Q7, Q4 to Q8, Q16 to Q9, R93 to R10, R94 to R11, R4 to R12, R5 to R13, R6 to R14, R95 to R15, R8 to R16, R96 to R17, R7 to R18, R10 to R19, R9 to R20, R11 to R21, R1 to R22, R12 to R23, R2 to R24, R99 to R25, R13 to R26, R100 to R27, R14 to R28, R15 to R29, R16 to R30, R17 to R31, R18 to R32, R19 to R33, R20 to R34, R65 to R35, R76 to R6, R3 to R7, R91 to R8, R92 to R9, SW1 to SW2, TP3 to TP1, TP1 to TP2, TP2 to TP3
Connections:
- no-connect marks 11 -> 5
Other:
- note removed: "Conn to EachBoard"
- note removed: "Conn to Power"
- note removed: "USB-C"

Commit message: ラズパイ基板とか
Parts:
- R33, R34, R35: value 2k -> 1k
Changed lines of the file:
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@@
       (effects (font (size 1.27 1.27)))
     )
-    (property "Value" "2k" (at 335.28 210.82 90)
+    (property "Value" "1k" (at 335.28 210.82 90)
       (effects (font (size 1.27 1.27)))
     )
@@
       (effects (font (size 1.27 1.27)))
     )
-    (property "Value" "2k" (at 335.28 198.12 90)
+    (property "Value" "1k" (at 335.28 198.12 90)
       (effects (font (size 1.27 1.27)))
     )
@@
       (effects (font (size 1.27 1.27)))
     )
-    (property "Value" "2k" (at 335.28 223.52 90)
-      (effects (font (size 1.27 1.27)))
-    )
+    (property "Value" "1k" (at 335.28 223.52 90)
+      (effects (font (size 1.27 1.27)))
+    )

Commit message: PDFプロット
Parts:
- added U7: AZ1084CD-3.3, Package_TO_SOT_SMD:TO-252-2, symbol Regulator_Linear:AMS1117CD-3.3
Connections:
- net +3.3V: now also U7.2 (VO)
- net +5V: now also U7.3 (VI)
- net GND: now also U7.1 (GND)
Changed lines of the file:
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@@
     (stroke (width 0) (type default))
   )
-  (polyline (pts (xy 93.98 182.88) (xy 93.98 30.48))
+  (polyline (pts (xy 93.98 246.38) (xy 93.98 30.48))
     (stroke (width 0.5) (type solid))
   )
@@
     (stroke (width 0) (type default))
   )
-  (polyline (pts (xy 43.18 246.38) (xy 43.18 182.88))
-    (stroke (width 0.5) (type default))
-  )
   (wire (pts (xy 238.76 147.32) (xy 238.76 160.02))
     (stroke (width 0) (type default))
@@
     (stroke (width 0) (type default))
   )
-  (polyline (pts (xy 43.18 182.88) (xy 93.98 182.88))
-    (stroke (width 0.5) (type default))
-  )
   (polyline (pts (xy 205.74 116.84) (xy 205.74 182.88))
     (stroke (width 0) (type dash))
@@
     (stroke (width 0) (type default))
   )
-  (polyline (pts (xy 93.98 246.38) (xy 43.18 246.38))
-    (stroke (width 0.5) (type default))
-  )
   (wire (pts (xy 109.22 170.18) (xy 132.08 170.18))
     (stroke (width 0) (type default))
@@
   (wire (pts (xy 349.25 195.58) (xy 353.06 195.58))
     (stroke (width 0) (type default))
-  )
-  (polyline (pts (xy 93.98 182.88) (xy 93.98 246.38))
-    (stroke (width 0) (type dash))
   )
   (wire (pts (xy 193.04 71.12) (xy 193.04 74.93))
@@
         )
       )
+    )
+  )
+  (symbol (lib_id "Regulator_Linear:AMS1117CD-3.3") (at 236.22 213.36 0) (unit 1)
+    (in_bom yes) (on_board yes) (dnp no) (fields_autoplaced)
+    (property "Reference" "U7" (at 236.22 207.01 0)
+      (effects (font (size 1.27 1.27)))
+    )
+    (property "Value" "AZ1084CD-3.3" (at 236.22 209.55 0)
+      (effects (font (size 1.27 1.27)))
+    )
+    (property "Footprint" "Package_TO_SOT_SMD:TO-252-2" (at 236.22 208.28 0)
+      (effects (font (size 1.27 1.27)) hide)
+    )
+    (property "Datasheet" "http://www.advanced-monolithic.com/pdf/ds1117.pdf" (at 238.76 219.71 0)
+      (effects (font (size 1.27 1.27)) hide)
+    )
+    (pin "1")
+    (pin "2")
+    (pin "3")
+    (instances
+      (project "2ndLayer"
+        (path "/5cc21ad3-a17c-4615-8f1b-99935a785699/3369f809-2737-4dac-a1dc-b9b69997c920"
+          (reference "U7") (unit 1)
+        )
+      )

Commit message: panelフットプリント配置
Parts:
- U7: value AZ1084CD-3.3 -> AZ1117CH-3.3; footprint Package_TO_SOT_SMD:TO-252-2 -> Package_TO_SOT_SMD:SOT-223-3_TabPin2
Changed lines of the file:
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@@
-    )
-  )
-  (symbol (lib_id "Regulator_Linear:AMS1117CD-3.3") (at 236.22 213.36 0) (unit 1)
-    (in_bom yes) (on_board yes) (dnp no) (fields_autoplaced)
-    (property "Reference" "U7" (at 236.22 207.01 0)
-      (effects (font (size 1.27 1.27)))
-    )
-    (property "Value" "AZ1084CD-3.3" (at 236.22 209.55 0)
-      (effects (font (size 1.27 1.27)))
-    )
-    (property "Footprint" "Package_TO_SOT_SMD:TO-252-2" (at 236.22 208.28 0)
-      (effects (font (size 1.27 1.27)) hide)
-    )
-    (property "Datasheet" "http://www.advanced-monolithic.com/pdf/ds1117.pdf" (at 238.76 219.71 0)
-      (effects (font (size 1.27 1.27)) hide)
-    )
-    (pin "1")
-    (pin "2")
-    (pin "3")
-    (instances
-      (project "2ndLayer"
-        (path "/5cc21ad3-a17c-4615-8f1b-99935a785699/3369f809-2737-4dac-a1dc-b9b69997c920"
-          (reference "U7") (unit 1)
-        )
-      )
     )
   )
@@
         )
       )
+    )
+  )
+  (symbol (lib_id "Regulator_Linear:AMS1117CD-3.3") (at 236.22 213.36 0) (unit 1)
+    (in_bom yes) (on_board yes) (dnp no) (fields_autoplaced)
+    (property "Reference" "U7" (at 236.22 207.01 0)
+      (effects (font (size 1.27 1.27)))
+    )
+    (property "Value" "AZ1117CH-3.3" (at 236.22 209.55 0)
+      (effects (font (size 1.27 1.27)))
+    )
+    (property "Footprint" "Package_TO_SOT_SMD:SOT-223-3_TabPin2" (at 236.22 208.28 0)
+      (effects (font (size 1.27 1.27)) hide)
+    )
+    (property "Datasheet" "http://www.advanced-monolithic.com/pdf/ds1117.pdf" (at 238.76 219.71 0)
+      (effects (font (size 1.27 1.27)) hide)
+    )
+    (pin "1")
+    (pin "2")
+    (pin "3")
+    (instances
+      (project "2ndLayer"
+        (path "/5cc21ad3-a17c-4615-8f1b-99935a785699/3369f809-2737-4dac-a1dc-b9b69997c920"
+          (reference "U7") (unit 1)
+        )
+      )

Commit message: シンボル・フットプリントMyLib->TomoshibiLib置き換え
Parts:
- IC1: footprint MyLibrary:DCDC_MPM3620A -> TomoshibiLibrary:DCDC_MPM3620A; symbol MyLibrary:DCDC_MPM3620A -> TomoshibiLibrary:DCDC_MPM3620A
- L1: footprint MyLibrary:Inductor_CDPH4D19F -> TomoshibiLibrary:Inductor_CDPH4D19F
- Q7, Q9: footprint MyLibrary:Package_TSOP6F -> TomoshibiLibrary:Package_TSOP6F
- SW2: footprint MyLibrary:SW_Slide_SPDT_White -> TomoshibiLibrary:SW_Slide_SPDT_White
Changed lines of the file:
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@@
       (effects (font (size 1.27 1.27)))
     )
-    (property "Footprint" "MyLibrary:Inductor_CDPH4D19F" (at 246.38 71.12 0)
+    (property "Footprint" "TomoshibiLibrary:Inductor_CDPH4D19F" (at 246.38 71.12 0)
       (effects (font (size 1.27 1.27)) hide)
     )
@@
     )
   )
-  (symbol (lib_id "MyLibrary:DCDC_MPM3620A") (at 119.38 137.16 0) (unit 1)
+  (symbol (lib_id "TomoshibiLibrary:DCDC_MPM3620A") (at 119.38 137.16 0) (unit 1)
     (in_bom yes) (on_board yes) (dnp no)
     (property "Reference" "IC1" (at 134.62 133.35 0)
@@
       (effects (font (size 1.27 1.27)))
     )
-    (property "Footprint" "MyLibrary:DCDC_MPM3620A" (at 148.59 232.08 0)
+    (property "Footprint" "TomoshibiLibrary:DCDC_MPM3620A" (at 104.14 100.66 0)
       (effects (font (size 1.27 1.27)) (justify left top) hide)
     )
-    (property "Datasheet" "http://www.monolithicpower.com/DesktopModules/DocumentManage/API/Document/getDocument?id=3961" (at 148.59 332.08 0)
+    (property "Datasheet" "http://www.monolithicpower.com/DesktopModules/DocumentManage/API/Document/getDocument?id=3961" (at 104.14 200.66 0)
       (effects (font (size 1.27 1.27)) (justify left top) hide)
     )
@@
       (effects (font (size 1.27 1.27)))
     )
-    (property "Footprint" "MyLibrary:SW_Slide_SPDT_White" (at 203.2 40.64 0)
+    (property "Footprint" "TomoshibiLibrary:SW_Slide_SPDT_White" (at 203.2 40.64 0)
       (effects (font (size 1.27 1.27)) hide)
     )
@@
       (effects (font (size 1.27 1.27)))
     )
-    (property "Footprint" "MyLibrary:Package_TSOP6F" (at 213.36 68.58 0)
+    (property "Footprint" "TomoshibiLibrary:Package_TSOP6F" (at 213.36 68.58 0)
       (effects (font (size 1.27 1.27)) (justify left) hide)
     )
@@
       (effects (font (size 1.27 1.27)))
     )
-    (property "Footprint" "MyLibrary:Package_TSOP6F" (at 187.96 68.58 0)
+    (property "Footprint" "TomoshibiLibrary:Package_TSOP6F" (at 187.96 68.58 0)
       (effects (font (size 1.27 1.27)) (justify left) hide)
     )
