File: circuits/Panel/NeoPixel.kicad_sch (KiCad schematic)
At the start: 1200 parts

Commit message: シンボル・フットプリントMyLib->TomoshibiLib置き換え
Parts:
- D1, D10, D100, D1000, D1001, D1002, D1003, D1004, D1005, D1006, D1007, D1008, D1009, D101, D1010, D1011, D1012, D1013, D1014, D1015, D1016, D1017, D1018, D1019, D102, D1020, D1021, D1022, D1023, D1024, D1025, D1026, D1027, D1028, D1029, D103, D1030, D1031, D1032, D1033, D1034, D1035, D1036, D1037, D1038, D1039, D104, D1040, D1041, D1042, D1043, D1044, D1045, D1046, D1047, D1048, D1049, D105, D1050, D1051, D1052, D1053, D1054, D1055, D1056, D1057, D1058, D1059, D106, D1060, D1061, D1062, D1063, D1064, D1065, D1066, D1067, D1068, D1069, D107, D1070, D1071, D1072, D1073, D1074, D1075, D1076, D1077, D1078, D1079, D108, D1080, D1081, D1082, D1083, D1084, D1085, D1086, D1087, D1088, D1089, D109, D1090, D1091, D1092, D1093, D1094, D1095, D1096, D1097, D1098, D1099, D11, D110, D1100, D1101, D1102, D1103, D1104, D1105, D1106, D1107, D1108, D1109, D111, D1110, D1111, D1112, D1113, D1114, D1115, D1116, D1117, D1118, D1119, D112, D1120, D1121, D1122, D1123, D1124, D1125, D1126, D1127, D1128, D1129, D113, D1130, D1131, D1132, D1133, D1134, D1135, D1136, D1137, D1138, D1139, D114, D1140, D1141, D1142, D1143, D1144, D1145, D1146, D1147, D1148, D1149, D115, D1150, D1151, D1152, D1153, D1154, D1155, D1156, D1157, D1158, D1159, D116, D1160, D1161, D1162, D1163, D1164, D1165, D1166, D1167, D1168, D1169, D117, D1170, D1171, D1172, D1173, D1174, D1175, D1176, D1177, D1178, D1179, D118, D1180, D1181, D1182, D1183, D1184, D1185, D1186, D1187, D1188, D1189, D119, D1190, D1191, D1192, D1193, D1194, D1195, D1196, D1197, D1198, D1199, D12, D120, D1200, D121, D122, D123, D124, D125, D126, D127, D128, D129, D13, D130, D131, D132, D133, D134, D135, D136, D137, D138, D139, D14, D140, D141, D142, D143, D144, D145, D146, D147, D148, D149, D15, D150, D151, D152, D153, D154, D155, D156, D157, D158, D159, D16, D160, D161, D162, D163, D164, D165, D166, D167, D168, D169, D17, D170, D171, D172, D173, D174, D175, D176, D177, D178, D179, D18, D180, D181, D182, D183, D184, D185, D186, D187, D188, D189, D19, D190, D191, D192, D193, D194, D195, D196, D197, D198, D199, D2, D20, D200, D201, D202, D203, D204, D205, D206, D207, D208, D209, D21, D210, D211, D212, D213, D214, D215, D216, D217, D218, D219, D22, D220, D221, D222, D223, D224, D225, D226, D227, D228, D229, D23, D230, D231, D232, D233, D234, D235, D236, D237, D238, D239, D24, D240, D241, D242, D243, D244, D245, D246, D247, D248, D249, D25, D250, D251, D252, D253, D254, D255, D256, D257, D258, D259, D26, D260, D261, D262, D263, D264, D265, D266, D267, D268, D269, D27, D270, D271, D272, D273, D274, D275, D276, D277, D278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: footprint MyLibrary:NeoPixel_WS2812C-2020-V1_ValueOnly -> TomoshibiLibrary:NeoPixel_WS2812C-2020-V1_ValueOnly; symbol NeoPixel:WS2812C-2020-V1 -> TomoshibiLibrary:NeoPixel_WS2812C-2020-V1
Connections:
- net DIN0: no longer D1001.3 (DIN), D201.3 (DIN), D401.3 (DIN), D601.3 (DIN), D801.3 (DIN)
- net DOUT0: no longer D1000.1 (DOUT), D1200.1 (DOUT), D400.1 (DOUT), D600.1 (DOUT), D800.1 (DOUT)
- new net DIN1: D201.3 (DIN)
- new net DIN2: D401.3 (DIN)
- new net DIN3: D601.3 (DIN)
- new net DIN4: D801.3 (DIN)
- new net DIN5: D1001.3 (DIN)
- new net DOUT1: D400.1 (DOUT)
- new net DOUT2: D600.1 (DOUT)
- new net DOUT3: D800.1 (DOUT)
- new net DOUT4: D1000.1 (DOUT)
- new net DOUT5: D1200.1 (DOUT)
