File: circuits/Panel/Pass_con.kicad_sch (KiCad schematic)
At the start: 1200 parts

Commit message: シンボル・フットプリントMyLib->TomoshibiLib置き換え
Parts:
- C1, C10, C100, C1000, C1001, C1002, C1003, C1004, C1005, C1006, C1007, C1008, C1009, C101, C1010, C1011, C1012, C1013, C1014, C1015, C1016, C1017, C1018, C1019, C102, C1020, C1021, C1022, C1023, C1024, C1025, C1026, C1027, C1028, C1029, C103, C1030, C1031, C1032, C1033, C1034, C1035, C1036, C1037, C1038, C1039, C104, C1040, C1041, C1042, C1043, C1044, C1045, C1046, C1047, C1048, C1049, C105, C1050, C1051, C1052, C1053, C1054, C1055, C1056, C1057, C1058, C1059, C106, C1060, C1061, C1062, C1063, C1064, C1065, C1066, C1067, C1068, C1069, C107, C1070, C1071, C1072, C1073, C1074, C1075, C1076, C1077, C1078, C1079, C108, C1080, C1081, C1082, C1083, C1084, C1085, C1086, C1087, C1088, C1089, C109, C1090, C1091, C1092, C1093, C1094, C1095, C1096, C1097, C1098, C1099, C11, C110, C1100, C1101, C1102, C1103, C1104, C1105, C1106, C1107, C1108, C1109, C111, C1110, C1111, C1112, C1113, C1114, C1115, C1116, C1117, C1118, C1119, C112, C1120, C1121, C1122, C1123, C1124, C1125, C1126, C1127, C1128, C1129, C113, C1130, C1131, C1132, C1133, C1134, C1135, C1136, C1137, C1138, C1139, C114, C1140, C1141, C1142, C1143, C1144, C1145, C1146, C1147, C1148, C1149, C115, C1150, C1151, C1152, C1153, C1154, C1155, C1156, C1157, C1158, C1159, C116, C1160, C1161, C1162, C1163, C1164, C1165, C1166, C1167, C1168, C1169, C117, C1170, C1171, C1172, C1173, C1174, C1175, C1176, C1177, C1178, C1179, C118, C1180, C1181, C1182, C1183, C1184, C1185, C1186, C1187, C1188, C1189, C119, C1190, C1191, C1192, C1193, C1194, C1195, C1196, C1197, C1198, C1199, C12, C120, C1200, C121, C122, C123, C124, C125, C126, C127, C128, C129, C13, C130, C131, C132, C133, C134, C135, C136, C137, C138, C139, C14, C140, C141, C142, C143, C144, C145, C146, C147, C148, C149, C15, C150, C151, C152, C153, C154, C155, C156, C157, C158, C159, C16, C160, C161, C162, C163, C164, C165, C166, C167, C168, C169, C17, C170, C171, C172, C173, C174, C175, C176, C177, C178, C179, C18, C180, C181, C182, C183, C184, C185, C186, C187, C188, C189, C19, C190, C191, C192, C193, C194, C195, C196, C197, C198, C199, C2, C20, C200, C201, C202, C203, C204, C205, C206, C207, C208, C209, C21, C210, C211, C212, C213, C214, C215, C216, C217, C218, C219, C22, C220, C221, C222, C223, C224, C225, C226, C227, C228, C229, C23, C230, C231, C232, C233, C234, C235, C236, C237, C238, C239, C24, C240, C241, C242, C243, C244, C245, C246, C247, C248, C249, C25, C250, C251, C252, C253, C254, C255, C256, C257, C258, C259, C26, C260, C261, C262, C263, C264, C265, C266, C267, C268, C269, C27, C270, C271, C272, C273, C274, C275, C276, C277, C278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: footprint MyLibrary:Capacitor_SMD_0402_1005Metric -> TomoshibiLibrary:Capacitor_SMD_0402_1005Metric
