File: circuits/Wireless/1stLayer/1stLayer.kicad_sch (KiCad schematic)
At the start: 4 parts, among them J1 Conn_01x14_Pin, J2 Conn_01x14_Pin, J3 Conn_01x14_Pin, J5 Conn_01x10_Socket

Commit message: シンボル・フットプリントMyLib->TomoshibiLib置き換え
Parts:
- J1, J2, J3: footprint MyLibrary:BoxHeader_2x07_P1.27mm_Horizontal -> TomoshibiLibrary:BoxHeader_2x07_P1.27mm_Horizontal
Changed lines of the file:
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@@
       (effects (font (size 1.27 1.27)))
     )
-    (property "Footprint" "MyLibrary:BoxHeader_2x07_P1.27mm_Horizontal" (at 144.78 88.9 0)
+    (property "Footprint" "TomoshibiLibrary:BoxHeader_2x07_P1.27mm_Horizontal" (at 144.78 88.9 0)
       (effects (font (size 1.27 1.27)) hide)
     )
@@
       (effects (font (size 1.27 1.27)))
     )
-    (property "Footprint" "MyLibrary:BoxHeader_2x07_P1.27mm_Horizontal" (at 119.38 144.78 0)
+    (property "Footprint" "TomoshibiLibrary:BoxHeader_2x07_P1.27mm_Horizontal" (at 119.38 144.78 0)
       (effects (font (size 1.27 1.27)) hide)
     )
@@
       (effects (font (size 1.27 1.27)))
     )
-    (property "Footprint" "MyLibrary:BoxHeader_2x07_P1.27mm_Horizontal" (at 119.38 88.9 0)
+    (property "Footprint" "TomoshibiLibrary:BoxHeader_2x07_P1.27mm_Horizontal" (at 119.38 88.9 0)
       (effects (font (size 1.27 1.27)) hide)
     )
