File: circuits/Power/Power.kicad_sch (KiCad schematic)
At the start: 0 parts

Commit message: PDFプロット
Parts:
- added C3: 1uF, Capacitor_SMD:C_0402_1005Metric, symbol Device:C
- added C4: 470uF, Capacitor_SMD:C_Elec_8x10.2, symbol Device:C_Polarized
- added D2: 1N5819WS, Diode_SMD:D_SOD-323_HandSoldering, symbol Device:D_Schottky
- added D3: Green, LED_SMD:LED_0603_1608Metric_Pad1.05x0.95mm_HandSolder, symbol Device:LED
- added F2: Fuse, Fuse:Fuseholder_Blade_Mini_Keystone_3568, symbol Device:Fuse
- added J4: Conn_01x02_Male, Connector_AMASS:AMASS_XT30U-M_1x02_P5.0mm_Vertical, symbol Connector:Conn_01x02_Male
- added J5, J6: Conn_01x02_Male, Connector_Molex:Molex_SPOX_5267-02A_1x02_P2.50mm_Vertical, symbol Connector:Conn_01x02_Male
- added Q4, Q6: SQS141ELNW, MyLibrary:Package_TSON-Advance, symbol Transistor_FET:AON6411
- added Q5: BSS138, Package_TO_SOT_SMD:SOT-23, symbol Device:Q_NMOS_GSD
- added R10, R5, R6, R7, R8, R9: 10k, Resistor_SMD:R_0402_1005Metric, symbol Device:R
- added R11: 20k, Resistor_SMD:R_0402_1005Metric, symbol Device:R
- added SW2: SW_SPDT, MyLibrary:SW_Slide_3P_SPDT, symbol Switch:SW_SPDT
- added TP1, TP2: TestPoint, TestPoint:TestPoint_THTPad_D2.0mm_Drill1.0mm, symbol Connector:TestPoint
Connections:
- new net: C3.2, Q6.4 (G), R10.1, R9.2
- new net: D3.2 (A), R11.1
- new net: Q5.3 (D), R10.2
- new net: R5.1, SW2.1 (A)
- new net: Q4.4 (G), R7.1, R8.2
- new net: F2.2, Q4.5 (D)
- new net +BATT: F2.1, J4.2 (Pin_2)
- new net GND: C4.2, D2.2 (A), D3.1 (K), J4.1 (Pin_1), J5.1 (Pin_1), J6.1 (Pin_1), Q5.2 (S), R6.2, R7.2, TP2.1
- new net PowerSW: Q5.1 (G), R5.2, R6.1
- new net S-S: C3.1, Q4.1 (S), Q4.2 (S), Q4.3 (S), Q6.1 (S), Q6.2 (S), Q6.3 (S), R8.1, R9.1, SW2.2 (B)
- new net VDD: C4.1, D2.1 (K), J5.2 (Pin_2), J6.2 (Pin_2), Q6.5 (D), R11.2, TP1.1
- no-connect marks 0 -> 1
Other:
- note added: "Capacitor"
- note added: "Conn to Battery"
- note added: "Conn\"
- note added: "PowerModule"
- note added: "TestPoint"
- note added: "インジケーターLED"
- note added: "主電源スイッチ"
- note added: "保護回路・スイッチ"

Commit message: シンボル・フットプリントMyLib->TomoshibiLib置き換え
Parts:
- Q4, Q6: footprint MyLibrary:Package_TSON-Advance -> TomoshibiLibrary:Package_TSON-Advance
- SW2: footprint MyLibrary:SW_Slide_3P_SPDT -> TomoshibiLibrary:SW_Slide_3P_SPDT
Changed lines of the file:
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@@
       (effects (font (size 1.27 1.27)) (justify left))
     )
-    (property "Footprint" "MyLibrary:SW_Slide_3P_SPDT" (at 68.58 93.98 0)
+    (property "Footprint" "TomoshibiLibrary:SW_Slide_3P_SPDT" (at 68.58 93.98 0)
       (effects (font (size 1.27 1.27)) hide)
     )
@@
       (effects (font (size 1.27 1.27)))
     )
-    (property "Footprint" "MyLibrary:Package_TSON-Advance" (at 121.285 73.66 0)
+    (property "Footprint" "TomoshibiLibrary:Package_TSON-Advance" (at 121.285 73.66 0)
       (effects (font (size 1.27 1.27)) (justify left) hide)
     )
@@
       (effects (font (size 1.27 1.27)))
     )
-    (property "Footprint" "MyLibrary:Package_TSON-Advance" (at 147.955 73.66 0)
+    (property "Footprint" "TomoshibiLibrary:Package_TSON-Advance" (at 147.955 73.66 0)
       (effects (font (size 1.27 1.27)) (justify left) hide)
     )

Commit message: 配線
Parts:
- added H1, H2: MountingHole_Pad, MountingHole:MountingHole_3.2mm_M3_Pad_Via, symbol Mechanical:MountingHole_Pad
Connections:
- net GND: now also H1.1
- net VDD: now also H2.1
Changed lines of the file:
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@@
   (symbol (lib_id "Connector:Conn_01x02_Male") (at 193.04 66.04 0) (mirror y) (unit 1)
     (in_bom yes) (on_board yes) (dnp no)
-    (property "Reference" "J5" (at 180.34 71.12 0)
-      (effects (font (size 1.27 1.27)))
-    )
-    (property "Value" "Conn_01x02_Male" (at 187.96 73.66 0)
+    (property "Reference" "J5" (at 177.8 71.12 0)
+      (effects (font (size 1.27 1.27)))
+    )
+    (property "Value" "Conn_01x02_Male" (at 185.42 73.66 0)
       (effects (font (size 1.27 1.27)))
     )
@@
     )
   )
+  (symbol (lib_id "Mechanical:MountingHole_Pad") (at 205.74 63.5 0) (unit 1)
+    (in_bom yes) (on_board yes) (dnp no)
+    (property "Reference" "H1" (at 195.58 55.88 0)
+      (effects (font (size 1.27 1.27)) (justify left))
+    )
+    (property "Value" "MountingHole_Pad" (at 195.58 58.42 0)
+      (effects (font (size 1.27 1.27)) (justify left))
+    )
+    (property "Footprint" "MountingHole:MountingHole_3.2mm_M3_Pad_Via" (at 205.74 63.5 0)
+      (effects (font (size 1.27 1.27)) hide)
+    )
+    (property "Datasheet" "~" (at 205.74 63.5 0)
+      (effects (font (size 1.27 1.27)) hide)
+    )
+    (pin "1")
+    (instances
+      (project "Power"
+        (path "/599e2e4a-5379-461e-b684-22a177410a52"
+          (reference "H1") (unit 1)
+        )
+      )
+    )
+  )
   (symbol (lib_id "Device:C") (at 134.62 81.28 0) (unit 1)
     (in_bom yes) (on_board yes) (dnp no)
@@
         (path "/599e2e4a-5379-461e-b684-22a177410a52"
           (reference "F2") (unit 1)
+        )
+      )
+    )
+  )
+  (symbol (lib_id "Mechanical:MountingHole_Pad") (at 205.74 71.12 180) (unit 1)
+    (in_bom yes) (on_board yes) (dnp no)
+    (property "Reference" "H2" (at 195.58 73.66 0)
+      (effects (font (size 1.27 1.27)) (justify right))
+    )
+    (property "Value" "MountingHole_Pad" (at 195.58 76.2 0)
+      (effects (font (size 1.27 1.27)) (justify right))
+    )
+    (property "Footprint" "MountingHole:MountingHole_3.2mm_M3_Pad_Via" (at 205.74 71.12 0)
+      (effects (font (size 1.27 1.27)) hide)
+    )
+    (property "Datasheet" "~" (at 205.74 71.12 0)
+      (effects (font (size 1.27 1.27)) hide)
+    )
+    (pin "1")
+    (instances
+      (project "Power"
+        (path "/599e2e4a-5379-461e-b684-22a177410a52"
+          (reference "H2") (unit 1)
         )
       )
@@
   (symbol (lib_id "Connector:Conn_01x02_Male") (at 193.04 81.28 0) (mirror y) (unit 1)
     (in_bom yes) (on_board yes) (dnp no)
-    (property "Reference" "J6" (at 180.34 86.36 0)
-      (effects (font (size 1.27 1.27)))
-    )
-    (property "Value" "Conn_01x02_Male" (at 187.96 88.9 0)
-      (effects (font (size 1.27 1.27)))
-    )
+    (property "Reference" "J6" (at 177.8 86.36 0)
+      (effects (font (size 1.27 1.27)))
+    )
+    (property "Value" "Conn_01x02_Male" (at 185.42 88.9 0)
+      (effects (font (size 1.27 1.27)))
+    )
