File: circuits/Power/Power.kicad_pcb (KiCad board)
At the start: 2 copper layers, 21 parts, among them J4 Conn_01x02_Male, J5 Conn_01x02_Male, J6 Conn_01x02_Male, Q4 SQS141ELNW, Q5 BSS138, Q6 SQS141ELNW, SW2 SW_SPDT

Commit message: 配線
Parts:
- added H1: MountingHole_Pad, MountingHole:MountingHole_3.2mm_M3_Pad_Via, F.Cu at (15.4, -4.68)
- added H2: MountingHole_Pad, MountingHole:MountingHole_3.2mm_M3_Pad_Via, F.Cu at (23.7, -4.93)
- SW2: moved to B.Cu
- moved TP1 102.0 mm to (26.9, -55.2)
- moved TP2 102.0 mm to (26.9, -51.1)
- moved Q6 101.9 mm to (9.17, -40.9)
- moved Q4 101.9 mm to (4.49, -40.9)
- moved D3 94.1 mm to (9.26, -36.4)
- moved C3 89.9 mm to (8.47, -34.2)
- moved D2 87.6 mm to (22.1, -34.4)
- moved J6 86.6 mm to (5.62, -46.1)
- moved J5 86.6 mm to (5.62, -53.1)
- moved C4 81.1 mm to (16.4, -46.0)
- moved Q5 79.0 mm to (4.59, -35.3)
- moved R10 73.6 mm to (29.2, -36.4)
- moved R11 73.6 mm to (29.2, -34.4)
- moved R5 73.6 mm to (29.2, -46.4)
- moved R6 73.6 mm to (29.2, -44.4)
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Other:
- board outline added: 38 x 31 mm

Commit message: 配線おけ
Parts:
- Q4, Q6: moved to B.Cu
- moved Q4 55.6 mm to (52.6, -13.0), turned to 180 degrees
- moved J5 54.4 mm to (34.0, -6.71), turned to -90 degrees
- moved Q6 47.8 mm to (47.9, -13.0), turned to 180 degrees
- moved C4 40.0 mm to (53.7, -31.7), turned to 180 degrees
- moved J6 39.2 mm to (4.43, -6.93), turned to -90 degrees
- moved J4 14.2 mm to (17.5, -16.6), turned to 0 degrees
- moved H2 13.1 mm to (29.1, -16.8)
- moved H1 12.7 mm to (11.1, -16.7)
- moved F2 10.5 mm to (14.9, -6.86)

Commit message: 更新
Parts:
- moved Q4 65.0 mm to (-7.20, 12.4), turned to 0 degrees
- moved Q6 58.6 mm to (-7.18, 6.85)
- moved H2 40.3 mm to (-7.40, 0.20)
- moved J5 26.1 mm to (13.5, 9.50)
- moved J6 22.9 mm to (-11.2, 9.75)
- moved F2 21.3 mm to (6.46, 12.7), turned to 180 degrees
- moved J4 19.3 mm to (4.50, -2.25), turned to 180 degrees
- moved H1 17.1 mm to (12.4, 0.40)
Other:
- board outline removed
