File: circuits/RasPi/RasPi.kicad_pcb (KiCad board)
At the start: 2 copper layers, 132 parts, among them IC1 DCDC_MPM3620A, J1 Conn_01x14_Pin, J2 Conn_01x06_MountingPin, J3 Conn_01x06_MountingPin, J6 USB_C_Receptacle_USB2.0, Q1 S8550, Q10 BSS138, Q11 SSM3J332R, Q12 SSM6J808R, Q13 BSS138, Q14 SSM6J808R, Q15 S8550, Q16 SSM3J332R, Q17 S8550, Q2 S8550, Q6 SSM3J332R, Q7 S8550, Q8 SSM3J332R, Q9 S8550, SW1 SW_SPST, SW2 SW_DIP_x04, SW3 SW_SPDT, SW4 SW_SPDT_White, U1 STM32F446RETx, U2 MAX3485, U3 MAX3485, U4 MAX3485, U5 MAX3485, U6 SBC_RPi-CM4, U7 FPGA_TangPrimer25K_Core, Y1 16MHz

Commit message: PDFプロット
Parts:
- removed JP1, JP2, JP3, JP4: Jumper_2_Open, Connector_PinHeader_2.54mm:PinHeader_1x02_P2.54mm_Vertical
- added C15: 0.1uF, Capacitor_SMD:C_0402_1005Metric, F.Cu at (214.0, 31.9)
- added C16: 0.1uF, Capacitor_SMD:C_0402_1005Metric, F.Cu at (214.0, 33.8)
- added C17: 0.1uF, Capacitor_SMD:C_0402_1005Metric, F.Cu at (214.0, 35.8)
- added C18: 0.1uF, Capacitor_SMD:C_0402_1005Metric, F.Cu at (214.0, 37.8)
- added C26: 0.1uF, Capacitor_SMD:C_0402_1005Metric, F.Cu at (214.0, 39.7)
- added C28: 0.1uF, Capacitor_SMD:C_0402_1005Metric, F.Cu at (202.6, 30.3)
- added C31: 0.1uF, Capacitor_SMD:C_0402_1005Metric, F.Cu at (202.6, 32.2)
- added C33: 0.1uF, Capacitor_SMD:C_0402_1005Metric, F.Cu at (202.6, 34.2)
- added C35: 0.1uF, Capacitor_SMD:C_0402_1005Metric, F.Cu at (202.6, 36.2)
- added C36: 0.1uF, Capacitor_SMD:C_0402_1005Metric, F.Cu at (202.6, 38.1)
- added C38: 0.1uF, Capacitor_SMD:C_0402_1005Metric, F.Cu at (217.1, 57.7)
- added D12: Red, LED_SMD:LED_0603_1608Metric_Pad1.05x0.95mm_HandSolder, F.Cu at (218.3, 18.6)
- added D13: Red, LED_SMD:LED_0603_1608Metric_Pad1.05x0.95mm_HandSolder, F.Cu at (218.3, 21.2)
- added D14: Red, LED_SMD:LED_0603_1608Metric_Pad1.05x0.95mm_HandSolder, F.Cu at (218.3, 23.8)
- added D15: Red, LED_SMD:LED_0603_1608Metric_Pad1.05x0.95mm_HandSolder, F.Cu at (218.3, 26.4)
- added J5: Conn_01x05_Pin, Connector_PinHeader_2.54mm:PinHeader_1x05_P2.54mm_Vertical, F.Cu at (210.2, 33.2)
- added Q18: S8550, Package_TO_SOT_SMD:SOT-23, F.Cu at (194.7, 33.6)
- added Q19: S8550, Package_TO_SOT_SMD:SOT-23, F.Cu at (194.7, 38.2)
- added Q21: BSS138, Package_TO_SOT_SMD:SOT-23, F.Cu at (219.8, 33.3)
- added Q22: S8550, Package_TO_SOT_SMD:SOT-23, F.Cu at (213.2, 56.6)
- added Q3: S8550, Package_TO_SOT_SMD:SOT-23, F.Cu at (194.7, 19.7)
- added Q4: S8550, Package_TO_SOT_SMD:SOT-23, F.Cu at (194.7, 24.4)
- added Q5: S8550, Package_TO_SOT_SMD:SOT-23, F.Cu at (194.7, 29.0)
- added R29: 5.1k, Resistor_SMD:R_0402_1005Metric, F.Cu at (189.0, 79.5)
- added R30: 7.5k, Resistor_SMD:R_0603_1608Metric, F.Cu at (199.1, 30.5)
- added R31: 20k, Resistor_SMD:R_0402_1005Metric, F.Cu at (198.6, 18.3)
- added R32: 2.2k, Resistor_SMD:R_0402_1005Metric, F.Cu at (198.6, 20.3)
- added R33: 2.2k, Resistor_SMD:R_0402_1005Metric, F.Cu at (198.6, 22.3)
- added R34: 20k, Resistor_SMD:R_0402_1005Metric, F.Cu at (198.6, 24.3)
- added R35: 2.2k, Resistor_SMD:R_0402_1005Metric, F.Cu at (198.6, 26.3)
- added R36: 2.2k, Resistor_SMD:R_0402_1005Metric, F.Cu at (198.6, 28.3)
- added R37: 7.5k, Resistor_SMD:R_0603_1608Metric, F.Cu at (199.1, 33.0)
- added R38: 20k, Resistor_SMD:R_0402_1005Metric, F.Cu at (201.5, 18.3)
- added R39: 2.2k, Resistor_SMD:R_0402_1005Metric, F.Cu at (201.5, 20.3)
- added R40: 2.2k, Resistor_SMD:R_0402_1005Metric, F.Cu at (201.5, 22.3)
- added R41: 7.5k, Resistor_SMD:R_0603_1608Metric, F.Cu at (199.1, 35.5)
- added R74: 20k, Resistor_SMD:R_0402_1005Metric, F.Cu at (201.5, 24.3)
- added R75: 2.2k, Resistor_SMD:R_0402_1005Metric, F.Cu at (201.5, 26.3)
- added R76: 2.2k, Resistor_SMD:R_0402_1005Metric, F.Cu at (201.5, 28.3)
- added R77: 7.5k, Resistor_SMD:R_0603_1608Metric, F.Cu at (199.1, 38.1)
- added R78: 20k, Resistor_SMD:R_0402_1005Metric, F.Cu at (204.4, 18.3)
- added R79: 2.2k, Resistor_SMD:R_0402_1005Metric, F.Cu at (204.4, 20.3)
- added R80: 1k, Resistor_SMD:R_0402_1005Metric, F.Cu at (221.9, 18.3)
- added R81: 1k, Resistor_SMD:R_0402_1005Metric, F.Cu at (221.9, 20.3)
- added R82: 1k, Resistor_SMD:R_0402_1005Metric, F.Cu at (221.9, 22.3)
- added R83: 1k, Resistor_SMD:R_0402_1005Metric, F.Cu at (221.9, 24.3)
- added R84: 10k, Resistor_SMD:R_0402_1005Metric, F.Cu at (221.9, 26.3)
- added R85: 5.1k, Resistor_SMD:R_0402_1005Metric, F.Cu at (189.0, 81.5)
- added R86: 5.1k, Resistor_SMD:R_0402_1005Metric, F.Cu at (189.0, 83.5)
- added R87: 2.2k, Resistor_SMD:R_0402_1005Metric, F.Cu at (204.4, 22.3)
- added R89: 10k, Resistor_SMD:R_0402_1005Metric, F.Cu at (218.8, 36.5)
- added R90: 7.5k, Resistor_SMD:R_0603_1608Metric, F.Cu at (217.7, 55.5)
- added R95: 20k, Resistor_SMD:R_0402_1005Metric, F.Cu at (209.3, 48.7)
- added R96: 2.2k, Resistor_SMD:R_0402_1005Metric, F.Cu at (209.3, 50.6)
- added R97: 2.2k, Resistor_SMD:R_0402_1005Metric, F.Cu at (209.3, 52.6)
- added R98: 120, Resistor_SMD:R_0402_1005Metric, F.Cu at (209.3, 54.6)
- added SW6: SW_SPDT, MyLibrary:SW_Slide_3P_SPDT, F.Cu at (212.0, 24.0)
- added U10: MAX3485, Package_SO:SOP-8_3.9x4.9mm_P1.27mm, F.Cu at (188.0, 33.9)
- added U11: MAX3485, Package_SO:SOP-8_3.9x4.9mm_P1.27mm, F.Cu at (188.0, 40.4)
- added U12: MAX3485, Package_SO:SOP-8_3.9x4.9mm_P1.27mm, F.Cu at (188.0, 47.0)
- added U14: MAX3485, Package_SO:SOP-8_3.9x4.9mm_P1.27mm, F.Cu at (215.0, 51.0)
- added U8: MAX3485, Package_SO:SOP-8_3.9x4.9mm_P1.27mm, F.Cu at (188.0, 20.7)
- added U9: MAX3485, Package_SO:SOP-8_3.9x4.9mm_P1.27mm, F.Cu at (188.0, 27.3)
- R13, R22: value 10k -> 2.2k
- R15, R23: value 2.2k -> 120
- R16: value 2.2k -> 10k
- R18, R27: value 120 -> 2.2k
- R20: value 7.5k -> 10k; footprint Resistor_SMD:R_0603_1608Metric -> Resistor_SMD:R_0402_1005Metric
- R21: value 20k -> 2.2k
- R24: value 2.2k -> 7.5k; footprint Resistor_SMD:R_0402_1005Metric -> Resistor_SMD:R_0603_1608Metric
- R25: value 2.2k -> 20k
- R28: value 120 -> 7.5k; footprint Resistor_SMD:R_0402_1005Metric -> Resistor_SMD:R_0603_1608Metric
- R4, R5, R71, R72, R73: value 2k -> 1k
- moved U6 101.0 mm to (155.5, 62.2), turned to -90 degrees
- moved U7 25.0 mm to (119.0, 73.0)
Connections:
- R13 pad 1: Net-(U3-DE) -> +3.3V
- R13 pad 2: GND -> /RingNW/RS485_RingNW/RS485X_TA
- R14 pad 1: +3.3V -> /RingNW/RS485_RingNW/RS485X_TB
- R14 pad 2: /RingNW/RS485_RingNW/RS485X_TA -> GND
- R15 pad 1: /RingNW/RS485_RingNW/RS485X_TB -> /RingNW/RS485_RingNW/RS485X_TA
- R15 pad 2: GND -> /RingNW/RS485_RingNW/RS485X_TB
- R16 pad 1: +3.3V -> Net-(U3-DE)
- R16 pad 2: /RingNW/RS485_RingNW/RS485X_RA -> GND
- R17 pad 1: /RingNW/RS485_RingNW/RS485X_RB -> +3.3V
- R17 pad 2: GND -> /RingNW/RS485_RingNW/RS485X_RA
- R18 pad 1: Net-(JP1-B) -> /RingNW/RS485_RingNW/RS485X_RB
- R18 pad 2: /RingNW/RS485_RingNW/RS485X_TB -> GND
- R19 pad 1: Net-(JP2-B) -> /RingNW/RS485_RingNW/RS485X_RA
- R20 pad 1: Net-(Q2-B) -> Net-(U4-DE)
- R20 pad 2: /RingNW/F446TXx_RS485YRX -> GND
- R21 pad 1: Net-(Q2-C) -> +3.3V
- R21 pad 2: GND -> /RingNW/RS485_RingNW/RS485Y_RA
- R22 pad 1: Net-(U5-DE) -> /RingNW/RS485_RingNW/RS485Y_RB
- R23 pad 1: +3.3V -> /RingNW/RS485_RingNW/RS485Y_RA
- R23 pad 2: /RingNW/RS485_RingNW/RS485Y_TA -> /RingNW/RS485_RingNW/RS485Y_RB
- R24 pad 1: /RingNW/RS485_RingNW/RS485Y_TB -> Net-(Q2-B)
- R24 pad 2: GND -> /FPGA_TangPrimerCore/TangPrimerTXx_Panel0RX
- R25 pad 1: +3.3V -> Net-(Q2-C)
- R25 pad 2: /RingNW/RS485_RingNW/RS485Y_RA -> GND
- R26 pad 1: /RingNW/RS485_RingNW/RS485Y_RB -> +3.3V
- R26 pad 2: GND -> Net-(U5-B)
- R27 pad 1: Net-(JP3-B) -> Net-(U5-B)
- R27 pad 2: /RingNW/RS485_RingNW/RS485Y_TB -> GND
- R28 pad 2: /RingNW/RS485_RingNW/RS485Y_RB -> /FPGA_TangPrimerCore/TangPrimerTXx_Panel2RX
- U4 pad 1: unconnected-(U4-RO-Pad1) -> /RingNW/F446RXx_RS485YTX
- U4 pad 2: Net-(Q2-C) -> Net-(U4-DE)
- U4 pad 3: Net-(Q2-C) -> Net-(U4-DE)
- U4 pad 4: /RingNW/F446TXx_RS485YRX -> unconnected-(U4-DI-Pad4)
- U4 pad 6: /RingNW/RS485_RingNW/RS485Y_TA -> /RingNW/RS485_RingNW/RS485Y_RA
- U4 pad 7: /RingNW/RS485_RingNW/RS485Y_TB -> /RingNW/RS485_RingNW/RS485Y_RB
- U5 pad 1: /RingNW/F446RXx_RS485YTX -> /FPGA_TangPrimerCore/TangPrimerRXx_Panel0TX
- U5 pad 2: Net-(U5-DE) -> Net-(Q2-C)
- U5 pad 3: Net-(U5-DE) -> Net-(Q2-C)
- U5 pad 4: unconnected-(U5-DI-Pad4) -> /FPGA_TangPrimerCore/TangPrimerTXx_Panel0RX
- U5 pad 6: /RingNW/RS485_RingNW/RS485Y_RA -> /FPGA_TangPrimerCore/RS485_Panel/RS485_Panel0
- U5 pad 7: /RingNW/RS485_RingNW/RS485Y_RB -> Net-(U5-B)
- U6 pad 79: unconnected-(U6A-+5V(INPUT)__1-Pad79) -> +5V(INPUT)__1
- U6 pad 81: unconnected-(U6A-+5V(INPUT)__2-Pad81) -> +5V(INPUT)__2
- U6 pad 83: unconnected-(U6A-+5V(INPUT)__3-Pad83) -> +5V(INPUT)__3
- U6 pad 84: unconnected-(U6A-CM4_3.3V(OUTPUT)-Pad84) -> CM4_3.3V(OUTPUT)__1
- U6 pad 85: unconnected-(U6A-+5V(INPUT)__4-Pad85) -> +5V(INPUT)__4
- U6 pad 86: unconnected-(U6A-CM4_3.3V(OUTPUT)__1-Pad86) -> CM4_3.3V(OUTPUT)__1
- U6 pad 87: unconnected-(U6A-+5V(INPUT)__5-Pad87) -> +5V(INPUT)__5
- U6 pad 88: unconnected-(U6A-CM4_1.8V(OUTPUT)-Pad88) -> CM4_1.8V(OUTPUT)__1
- U6 pad 90: unconnected-(U6A-CM4_1.8V(OUTPUT)__1-Pad90) -> CM4_1.8V(OUTPUT)__1
- U7 pad A1: unconnected-(U7-GND-PadA1) -> GND
- U7 pad A13: unconnected-(U7-D8_RECONFIG-PadA13) -> /RST_FPGA
- U7 pad A19: unconnected-(U7-GND-PadA19) -> GND
- U7 pad A2: unconnected-(U7-VCCIO2/3-PadA2) -> /FPGA_TangPrimerCore/3.3V_TangPrimer
- U7 pad A21: unconnected-(U7-C1_TCK-PadA21) -> /FPGA_TangPrimerCore/TCK
- U7 pad A23: unconnected-(U7-B1_TMS-PadA23) -> /FPGA_TangPrimerCore/TMS
- U7 pad A25: unconnected-(U7-A2_TDO-PadA25) -> /FPGA_TangPrimerCore/TDO
- U7 pad A27: unconnected-(U7-A3_TDI-PadA27) -> /FPGA_TangPrimerCore/TDI
- U7 pad A29: unconnected-(U7-GND-PadA29) -> GND
- U7 pad A31: unconnected-(U7-M0_D3_P-PadA31) -> /FPGA_TangPrimerCore/MIPI_D3_P
- U7 pad A33: unconnected-(U7-M0_D3_N-PadA33) -> /FPGA_TangPrimerCore/MIPI_D3_N
- U7 pad A35: unconnected-(U7-GND-PadA35) -> GND
- U7 pad A37: unconnected-(U7-M0_D2_P-PadA37) -> /FPGA_TangPrimerCore/MIPI_D2_P
- U7 pad A39: unconnected-(U7-M0_D2_N-PadA39) -> /FPGA_TangPrimerCore/MIPI_D2_N
- U7 pad A4: unconnected-(U7-VCCIO2/3-PadA4) -> /FPGA_TangPrimerCore/3.3V_TangPrimer
- U7 pad A41: unconnected-(U7-GND-PadA41) -> GND
- U7 pad A43: unconnected-(U7-M0_CK_P-PadA43) -> /FPGA_TangPrimerCore/MIPI_CK_P
- U7 pad A45: unconnected-(U7-M0_CK_N-PadA45) -> /FPGA_TangPrimerCore/MIPI_CK_N
- U7 pad A46: unconnected-(U7-VDD_3V3-PadA46) -> /FPGA_TangPrimerCore/3.3V_TangPrimer
- U7 pad A47: unconnected-(U7-GND-PadA47) -> GND
- U7 pad A48: unconnected-(U7-VDD_3V3-PadA48) -> /FPGA_TangPrimerCore/3.3V_TangPrimer
- U7 pad A49: unconnected-(U7-M0_D1_P-PadA49) -> /FPGA_TangPrimerCore/MIPI_D1_P
- U7 pad A50: unconnected-(U7-VDD_3V3-PadA50) -> /FPGA_TangPrimerCore/3.3V_TangPrimer
- U7 pad A51: unconnected-(U7-M0_D1_N-PadA51) -> /FPGA_TangPrimerCore/MIPI_D1_N
- U7 pad A52: unconnected-(U7-VDD_5V-PadA52) -> +5V
- U7 pad A53: unconnected-(U7-GND-PadA53) -> GND
- U7 pad A54: unconnected-(U7-VDD_5V-PadA54) -> +5V
- U7 pad A55: unconnected-(U7-M0_D0_P-PadA55) -> /FPGA_TangPrimerCore/MIPI_D0_P
- U7 pad A56: unconnected-(U7-VDD_5V-PadA56) -> +5V
- U7 pad A57: unconnected-(U7-M0_D0_N-PadA57) -> /FPGA_TangPrimerCore/MIPI_D0_N
- U7 pad A58: unconnected-(U7-VDD_5V-PadA58) -> +5V
- U7 pad A59: unconnected-(U7-GND-PadA59) -> GND
- U7 pad A60: unconnected-(U7-VDD_5V-PadA60) -> +5V
- U7 pad B1: unconnected-(U7-GND-PadB1) -> GND
- U7 pad B15: unconnected-(U7-GND-PadB15) -> GND
- U7 pad B17: unconnected-(U7-E8_READY-PadB17) -> Net-(U7-E8_READY)
- U7 pad B2: unconnected-(U7-GND-PadB2) -> GND
- U7 pad B24: unconnected-(U7-VCCIO0/1-PadB24) -> /FPGA_TangPrimerCore/3.3V_TangPrimer
- U7 pad B25: unconnected-(U7-D7_DONE-PadB25) -> Net-(U7-D7_DONE)
- U7 pad B26: unconnected-(U7-VCCIO0/1-PadB26) -> /FPGA_TangPrimerCore/3.3V_TangPrimer
- U7 pad B27: unconnected-(U7-GND-PadB27) -> GND
- U7 pad B28: unconnected-(U7-GND-PadB28) -> GND
- U7 pad B29: unconnected-(U7-VCCIO6/7-PadB29) -> /FPGA_TangPrimerCore/3.3V_TangPrimer
- U7 pad B31: unconnected-(U7-VCCIO6/7-PadB31) -> /FPGA_TangPrimerCore/3.3V_TangPrimer
- U7 pad B45: unconnected-(U7-GND-PadB45) -> GND
- U7 pad B50: unconnected-(U7-GND-PadB50) -> GND
- U7 pad B59: unconnected-(U7-GND-PadB59) -> GND
- U7 pad B60: unconnected-(U7-GND-PadB60) -> GND

Commit message: panelフットプリント配置
Parts:
- removed IC1: DCDC_MPM3620A, MyLibrary:DCDC_MPM3620A
- removed Q11: SSM3J332R, Package_TO_SOT_SMD:SOT-23W
- removed R51: 12k, Resistor_SMD:R_0402_1005Metric
- removed R52: 2.2k, Resistor_SMD:R_0402_1005Metric
- added C37: 0.1uF, Capacitor_SMD:C_0402_1005Metric, F.Cu at (237.8, -9.62)
- added C39: 0.1uF, Capacitor_SMD:C_0402_1005Metric, F.Cu at (237.8, -7.66)
- added C40: 0.1uF, Capacitor_SMD:C_0402_1005Metric, F.Cu at (237.8, -5.68)
- added C41: 0.1uF, Capacitor_SMD:C_0402_1005Metric, F.Cu at (237.8, -3.71)
- added C42: 0.1uF, Capacitor_SMD:C_0402_1005Metric, F.Cu at (237.8, -1.75)
- added C43: 0.1uF, Capacitor_SMD:C_0402_1005Metric, F.Cu at (237.8, 0.23)
- added C44: 0.1uF, Capacitor_SMD:C_0402_1005Metric, F.Cu at (237.8, 2.19)
- added C45: 10uF, Capacitor_SMD:C_0805_2012Metric, F.Cu at (284.0, 16.4)
- added C46: 0.1uF, Capacitor_SMD:C_0402_1005Metric, F.Cu at (266.5, 15.0)
- added C47: 4700pF, Capacitor_SMD:C_0603_1608Metric, F.Cu at (246.9, -19.8)
- added C49: 100uF, Capacitor_SMD:C_0805_2012Metric, F.Cu at (238.6, -23.1)
- added C50: 47uF, Capacitor_SMD:C_0805_2012Metric, F.Cu at (238.6, -20.1)
- added C51: 0.1uF, Capacitor_SMD:C_0603_1608Metric, F.Cu at (246.9, -17.3)
- added C52: 0.1uF, Capacitor_SMD:C_0402_1005Metric, F.Cu at (258.4, -25.0)
- added C53: 47uF, Capacitor_SMD:C_0805_2012Metric, F.Cu at (274.9, -9.23)
- added C54: 0.1uF, Capacitor_SMD:C_0603_1608Metric, F.Cu at (274.6, -6.47)
- added C55: 47uF, Capacitor_SMD:C_0805_2012Metric, F.Cu at (238.6, -17.1)
- added C56: 1uF, Capacitor_SMD:C_0603_1608Metric, F.Cu at (246.9, -14.8)
- added C57: 47uF, Capacitor_SMD:C_0805_2012Metric, F.Cu at (238.6, -14.1)
- added D16: D_Zener, Diode_SMD:D_SOD-323_HandSoldering, F.Cu at (257.2, -19.6)
- added D17: SS2040FL, Diode_SMD:D_SOD-123, F.Cu at (251.8, -19.4)
- added D18: D_Zener, Diode_SMD:D_SOD-323_HandSoldering, F.Cu at (257.2, -16.6)
- added D20: Red, LED_SMD:LED_0603_1608Metric_Pad1.05x0.95mm_HandSolder, F.Cu at (284.9, -31.9)
- added D21: LightGreen, LED_SMD:LED_0603_1608Metric_Pad1.05x0.95mm_HandSolder, F.Cu at (284.9, -29.3)
- added D22: Yellow, LED_SMD:LED_0603_1608Metric_Pad1.05x0.95mm_HandSolder, F.Cu at (284.9, -26.7)
- added D23: Green, LED_SMD:LED_0603_1608Metric_Pad1.05x0.95mm_HandSolder, F.Cu at (288.2, -16.0)
- added D24: LightGreen, LED_SMD:LED_0603_1608Metric_Pad1.05x0.95mm_HandSolder, F.Cu at (288.2, -13.4)
- added D25: Yellow, LED_SMD:LED_0603_1608Metric_Pad1.05x0.95mm_HandSolder, F.Cu at (288.2, -10.8)
- added D26: LightGreen, LED_SMD:LED_0603_1608Metric_Pad1.05x0.95mm_HandSolder, F.Cu at (288.2, -8.26)
- added D27: SS2040FL, Diode_SMD:D_SOD-123, F.Cu at (251.8, -16.0)
- added D29: Red, LED_SMD:LED_0603_1608Metric_Pad1.05x0.95mm_HandSolder, F.Cu at (288.2, -5.67)
- added J10: Conn_01x03_MountingPin, Connector_Molex:Molex_PicoBlade_53261-0371_1x03-1MP_P1.25mm_Horizontal, F.Cu at (245.2, 1.47)
- added J12: Conn_01x02_MountingPin, Connector_Molex:Molex_PicoBlade_53261-0271_1x02-1MP_P1.25mm_Horizontal, F.Cu at (267.4, -13.1)
- added J13: Conn_01x03_MountingPin, Connector_Molex:Molex_PicoBlade_53398-0371_1x03-1MP_P1.25mm_Vertical, F.Cu at (268.0, 3.31)
- added J14: Conn_01x02_MountingPin, Connector_Molex:Molex_PicoBlade_53261-0271_1x02-1MP_P1.25mm_Horizontal, F.Cu at (267.4, -5.25)
- added J8: Conn_01x07_MountingPin, Connector_Molex:Molex_PicoBlade_53261-0771_1x07-1MP_P1.25mm_Horizontal, F.Cu at (285.3, 4.61)
- added J9: Conn_01x04_MountingPin, Connector_Molex:Molex_PicoBlade_53261-0471_1x04-1MP_P1.25mm_Horizontal, F.Cu at (245.8, -6.38)
- added L2: 2.2uH, MyLibrary:Inductor_CDPH4D19F, F.Cu at (248.1, -33.5)
- added L4: 2.2uH, MyLibrary:Inductor_CDPH4D19F, F.Cu at (254.6, -33.5)
- added Q20: BSS138, Package_TO_SOT_SMD:SOT-23, F.Cu at (290.7, 12.6)
- added Q23: BSS138, Package_TO_SOT_SMD:SOT-23, F.Cu at (290.7, 17.3)
- added Q25: BSS138, Package_TO_SOT_SMD:SOT-23, F.Cu at (269.6, 9.73)
- added Q26: SSM3J332R, Package_TO_SOT_SMD:SOT-23W, F.Cu at (264.6, 9.78)
- added Q27: BSS138, Package_TO_SOT_SMD:SOT-23, F.Cu at (279.4, 17.3)
- added Q28: SSM3J332R, Package_TO_SOT_SMD:SOT-23W, F.Cu at (279.4, 12.7)
- added Q29: BSS138, Package_TO_SOT_SMD:SOT-23, F.Cu at (285.1, -35.4)
- added Q30: BSS138, Package_TO_SOT_SMD:SOT-23, F.Cu at (292.8, -14.9)
- added Q33: BSS138, Package_TO_SOT_SMD:SOT-23, F.Cu at (292.8, -10.3)
- added R100: 10k, Resistor_SMD:R_0402_1005Metric, F.Cu at (242.3, -21.7)
- added R102: 10k, Resistor_SMD:R_0402_1005Metric, F.Cu at (273.4, 8.32)
- added R103: 10k, Resistor_SMD:R_0402_1005Metric, F.Cu at (273.4, 10.3)
- added R104: 10k, Resistor_SMD:R_0402_1005Metric, F.Cu at (283.3, 11.2)
- added R105: 10k, Resistor_SMD:R_0402_1005Metric, F.Cu at (288.5, -32.2)
- added R106: 10k, Resistor_SMD:R_0402_1005Metric, F.Cu at (283.3, 13.2)
- added R107: 1k, Resistor_SMD:R_0402_1005Metric, F.Cu at (288.5, -30.2)
- added R108: 1k, Resistor_SMD:R_0402_1005Metric, F.Cu at (288.5, -28.2)
- added R109: 1k, Resistor_SMD:R_0402_1005Metric, F.Cu at (288.5, -26.2)
- added R110: 10k, Resistor_SMD:R_0402_1005Metric, F.Cu at (284.6, -16.3)
- added R111: 1k, Resistor_SMD:R_0402_1005Metric, F.Cu at (284.6, -14.3)
- added R112: 1k, Resistor_SMD:R_0402_1005Metric, F.Cu at (284.6, -12.3)
- added R113: 1k, Resistor_SMD:R_0402_1005Metric, F.Cu at (284.6, -10.4)
- added R114: 1k, Resistor_SMD:R_0402_1005Metric, F.Cu at (284.6, -8.37)
- added R117: 10k, Resistor_SMD:R_0402_1005Metric, F.Cu at (284.6, -6.38)
- added R119: 200k, Resistor_SMD:R_0402_1005Metric, F.Cu at (242.3, -19.7)
- added R120: 1k, Resistor_SMD:R_0402_1005Metric, F.Cu at (284.6, -4.38)
- added R121: 53.6k, Resistor_SMD:R_0402_1005Metric, F.Cu at (242.3, -17.7)
- added R122: 10k, Resistor_SMD:R_0402_1005Metric, F.Cu at (242.3, -15.7)
- added R88: 10k, Resistor_SMD:R_0402_1005Metric, F.Cu at (294.6, 11.2)
- added R91: 10k, Resistor_SMD:R_0402_1005Metric, F.Cu at (294.6, 13.2)
- added R92: 10k, Resistor_SMD:R_0402_1005Metric, F.Cu at (252.5, 9.77)
- added R93: 470, Resistor_SMD:R_0402_1005Metric, F.Cu at (263.6, 15.0)
- added R94: 470, Resistor_SMD:R_0402_1005Metric, F.Cu at (263.6, 17.0)
- added R99: 53.6k, Resistor_SMD:R_0402_1005Metric, F.Cu at (242.3, -23.7)
- added SW5: SW_SPDT, MyLibrary:SW_Slide_3P_SPDT, F.Cu at (255.1, 3.90)
- added SW7: SW_SPST, Button_Switch_SMD:SW_SPST_Omron_B3FS-100xP, F.Cu at (244.9, 9.02)
- added U13: TPS54560BDDA, Package_SO:Texas_R-PDSO-G8_EP2.95x4.9mm_Mask2.4x3.1mm_ThermalVias, F.Cu at (240.6, -34.5)
- added U15: STM32H723VGTx, Package_QFP:LQFP-100_14x14mm_P0.5mm, F.Cu at (271.4, -28.6)
- added U16: AZ1084CD-3.3, Package_TO_SOT_SMD:TO-252-2, F.Cu at (251.8, -25.1)
- added U17: M51957B, Package_SO:SOP-8_3.9x4.9mm_P1.27mm, F.Cu at (240.6, -27.9)
- added U18: DAC_PT8211S, Package_SO:SOP-8_3.9x4.9mm_P1.27mm, F.Cu at (276.9, -14.0)
- added U19: DCDC_TPS61023, MyLibrary:DCDC_TPS61023, F.Cu at (258.6, -27.6)
- C20: value 10uF -> 4.7uF; footprint Capacitor_SMD:C_1206_3216Metric -> Capacitor_SMD:C_0603_1608Metric
- C22: value 22uF -> 1uF; footprint Capacitor_SMD:C_0805_2012Metric -> Capacitor_SMD:C_0402_1005Metric
- D12, D13, D14, D15, D2, D3: value Red -> Blue
- R45: value 200k -> 10k
- R50: value 100k -> 10k
- R54: value 10k -> 75k; footprint Resistor_SMD:R_0402_1005Metric -> Resistor_SMD:R_0603_1608Metric
- R57: value 10k -> 5.1k; footprint Resistor_SMD:R_0402_1005Metric -> Resistor_SMD:R_0603_1608Metric
- moved U6 167.4 mm to (0.00, 0.00)
- moved U7 165.8 mm to (-30.7, 1.80)
- moved C28 112.6 mm to (246.2, -73.5)
- moved C15 112.6 mm to (257.6, -71.9)
- moved C16 112.6 mm to (257.6, -70.0)
- moved C17 112.6 mm to (257.6, -68.0)
- moved C18 112.6 mm to (257.6, -66.0)
- moved C26 112.6 mm to (257.6, -64.1)
- moved C31 112.6 mm to (246.2, -71.6)
- moved C33 112.6 mm to (246.2, -69.6)
- moved C35 112.6 mm to (246.2, -67.6)
- moved C36 112.6 mm to (246.2, -65.6)
- moved C38 112.6 mm to (260.7, -46.0)
- moved D12 112.6 mm to (261.9, -85.2)
- moved D13 112.6 mm to (261.9, -82.6)
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Connections:
- net /FPGA_TangPrimerCore/LED0 renamed /FPGA_TangPrimerCore/LED_B0
- net /FPGA_TangPrimerCore/LED1 renamed /FPGA_TangPrimerCore/LED_B1
- net /FPGA_TangPrimerCore/LED2 renamed /FPGA_TangPrimerCore/LED_B2
- net /FPGA_TangPrimerCore/LED3 renamed /FPGA_TangPrimerCore/LED_B3
- net /Power/PG renamed Net-(D16-K)
- net /RasPi->RST_FPGA renamed /RasPi->RST_TangPrimer
- net /RingNW/LED0 renamed /RingNW/LED_B0
- net /RingNW/LED1 renamed /RingNW/LED_B1
- net V_Meas. renamed /V_Meas.
- C15 pad 1: +3.3V -> +5V
- C16 pad 1: +3.3V -> +5V
- C17 pad 1: +3.3V -> +5V
- C18 pad 1: +3.3V -> +5V
- C20 pad 1: VCC -> Net-(C20-Pad1)
- C22 pad 1: /Power/Vout -> GND
- C22 pad 2: GND -> +3.3V
- C26 pad 1: +3.3V -> +5V
- D4 pad 2: /Power/Vout -> /Power/VSYS
- Q10 pad 2: GND -> Net-(Q10-S)
- Q10 pad 3: Net-(Q10-D) -> /Power/VSYS
- Q21 pad 3: /RST_FPGA -> /RST_TangPrimer
- R45 pad 1: Net-(IC1-EN) -> Net-(Q10-S)
- R45 pad 2: VCC -> /Power/Cap
- R50 pad 2: Net-(IC1-VCC) -> /Power/VSYS
- R54 pad 1: /Power/Vout -> Net-(U17-IN)
- R54 pad 2: Net-(Q10-D) -> VDD
- R57 pad 1: GND -> Net-(U17-IN)
- R57 pad 2: /Power/VSYS -> GND
- U6 pad 1: unconnected-(U6A-GND-Pad1) -> GND
- U6 pad 107: unconnected-(U6A-GND__21-Pad107) -> GND
- U6 pad 108: unconnected-(U6A-GND__22-Pad108) -> GND
- U6 pad 113: unconnected-(U6A-GND__23-Pad113) -> GND
- U6 pad 114: unconnected-(U6A-GND__24-Pad114) -> GND
- U6 pad 119: unconnected-(U6A-GND__25-Pad119) -> GND
- U6 pad 120: unconnected-(U6A-GND__26-Pad120) -> GND
- U6 pad 125: unconnected-(U6A-GND__27-Pad125) -> GND
- U6 pad 126: unconnected-(U6A-GND__28-Pad126) -> GND
- U6 pad 13: unconnected-(U6A-GND__4-Pad13) -> GND
- U6 pad 131: unconnected-(U6A-GND__29-Pad131) -> GND
- U6 pad 132: unconnected-(U6A-GND__30-Pad132) -> GND
- U6 pad 137: unconnected-(U6A-GND__31-Pad137) -> GND
- U6 pad 138: unconnected-(U6A-GND__32-Pad138) -> GND
- U6 pad 14: unconnected-(U6A-GND__5-Pad14) -> GND
- U6 pad 144: unconnected-(U6A-GND__33-Pad144) -> GND
- U6 pad 150: unconnected-(U6A-GND__34-Pad150) -> GND
- U6 pad 155: unconnected-(U6A-GND__35-Pad155) -> GND
- U6 pad 156: unconnected-(U6A-GND__36-Pad156) -> GND
- U6 pad 161: unconnected-(U6A-GND__37-Pad161) -> GND
- U6 pad 162: unconnected-(U6A-GND__38-Pad162) -> GND
- U6 pad 167: unconnected-(U6A-GND__39-Pad167) -> GND
- U6 pad 168: unconnected-(U6A-GND__40-Pad168) -> GND
- U6 pad 173: unconnected-(U6A-GND__41-Pad173) -> GND
- U6 pad 174: unconnected-(U6A-GND__42-Pad174) -> GND
- U6 pad 175: unconnected-(U6B-DSI1_D0_N-Pad175) -> /DSI_D0_N
- U6 pad 177: unconnected-(U6B-DSI1_D0_P-Pad177) -> /DSI_D0_P
- U6 pad 179: unconnected-(U6A-GND__43-Pad179) -> GND
- U6 pad 180: unconnected-(U6A-GND__44-Pad180) -> GND
- U6 pad 181: unconnected-(U6B-DSI1_D1_N-Pad181) -> /DSI_D1_N
- U6 pad 183: unconnected-(U6B-DSI1_D1_P-Pad183) -> /DSI_D1_P
- U6 pad 185: unconnected-(U6A-GND__45-Pad185) -> GND
- U6 pad 186: unconnected-(U6A-GND__46-Pad186) -> GND
- U6 pad 187: unconnected-(U6B-DSI1_C_N-Pad187) -> /DSI_CK_P
- U6 pad 189: unconnected-(U6B-DSI1_C_P-Pad189) -> /DSI_CK_N
- U6 pad 191: unconnected-(U6A-GND__47-Pad191) -> GND
- U6 pad 192: unconnected-(U6A-GND__48-Pad192) -> GND
- U6 pad 193: unconnected-(U6B-DSI1_D2_N-Pad193) -> /DSI_D2_N
- U6 pad 194: unconnected-(U6B-DSI1_D3_N-Pad194) -> /DSI_D3_N
- U6 pad 195: unconnected-(U6B-DSI1_D2_P-Pad195) -> /DSI_D2_P
- U6 pad 196: unconnected-(U6B-DSI1_D3_P-Pad196) -> /DSI_D3_P
- U6 pad 197: unconnected-(U6A-GND__49-Pad197) -> GND
- U6 pad 198: unconnected-(U6A-GND__50-Pad198) -> GND
- U6 pad 2: unconnected-(U6A-GND__1-Pad2) -> GND
- U6 pad 21: unconnected-(U6A-PI_~{LED}_ACTIVITY-Pad21) -> /RasPi_CM4/LED_nACT
- U6 pad 22: unconnected-(U6A-GND__6-Pad22) -> GND
- U6 pad 23: unconnected-(U6A-GND__7-Pad23) -> GND
- U6 pad 25: unconnected-(U6A-GPIO21-Pad25) -> /PCM_DOUT
- U6 pad 26: unconnected-(U6A-GPIO19-Pad26) -> /PCM_FS
- U6 pad 27: unconnected-(U6A-GPIO20-Pad27) -> /PCM_DIN
- U6 pad 32: unconnected-(U6A-GND__8-Pad32) -> GND
- U6 pad 33: unconnected-(U6A-GND__9-Pad33) -> GND
- U6 pad 42: unconnected-(U6A-GND__10-Pad42) -> GND
- U6 pad 43: unconnected-(U6A-GND__11-Pad43) -> GND
- U6 pad 49: unconnected-(U6A-GPIO18-Pad49) -> /PCM_CLK
- U6 pad 52: unconnected-(U6A-GND__12-Pad52) -> GND
- U6 pad 53: unconnected-(U6A-GND__13-Pad53) -> GND
- U6 pad 56: unconnected-(U6A-GPIO3-Pad56) -> /RasPi_GPIO3
- U6 pad 57: unconnected-(U6A-SD_CLK-Pad57) -> /RasPi_CM4/SD_CLK
- U6 pad 59: unconnected-(U6A-GND__14-Pad59) -> GND
- U6 pad 60: unconnected-(U6A-GND__15-Pad60) -> GND
- U6 pad 61: unconnected-(U6A-SD_DAT3-Pad61) -> /RasPi_CM4/SD_DAT3
- U6 pad 62: unconnected-(U6A-SD_CMD-Pad62) -> /RasPi_CM4/SD_CMD
- U6 pad 63: unconnected-(U6A-SD_DAT0-Pad63) -> /RasPi_CM4/SD_DAT0
- U6 pad 65: unconnected-(U6A-GND__16-Pad65) -> GND
- U6 pad 66: unconnected-(U6A-GND__17-Pad66) -> GND
- U6 pad 67: unconnected-(U6A-SD_DAT1-Pad67) -> /RasPi_CM4/SD_DAT1
- U6 pad 69: unconnected-(U6A-SD_DAT2-Pad69) -> /RasPi_CM4/SD_DAT2
- U6 pad 7: unconnected-(U6A-GND__2-Pad7) -> GND
- U6 pad 71: unconnected-(U6A-GND__18-Pad71) -> GND
- U6 pad 74: unconnected-(U6A-GND__19-Pad74) -> GND
- U6 pad 75: unconnected-(U6A-SD_PWR_ON-Pad75) -> /RasPi_CM4/SD_PWR_ON
- U6 pad 77: unconnected-(U6A-+5V(INPUT)-Pad77) -> +5V
- U6 pad 78: unconnected-(U6A-GPIO_VREF-Pad78) -> CM4_3.3V(OUTPUT)__1
- U6 pad 79: +5V(INPUT)__1 -> +5V
- U6 pad 8: unconnected-(U6A-GND__3-Pad8) -> GND
- U6 pad 81: +5V(INPUT)__2 -> +5V
- U6 pad 83: +5V(INPUT)__3 -> +5V
- U6 pad 85: +5V(INPUT)__4 -> +5V
- U6 pad 87: +5V(INPUT)__5 -> +5V
- U6 pad 95: unconnected-(U6A-PI_LED_~{PWR}-Pad95) -> /RasPi_CM4/LED_nPWR
- U6 pad 98: unconnected-(U6A-GND__20-Pad98) -> GND
- U6 pad 99: unconnected-(U6A-GLOBAL_EN-Pad99) -> /RasPi_CM4/GLOBAL_EN
- U7 pad A31: /FPGA_TangPrimerCore/MIPI_D3_P -> /DSI_D3_P
- U7 pad A33: /FPGA_TangPrimerCore/MIPI_D3_N -> /DSI_D3_N
- U7 pad A37: /FPGA_TangPrimerCore/MIPI_D2_P -> /DSI_D2_P
- U7 pad A39: /FPGA_TangPrimerCore/MIPI_D2_N -> /DSI_D2_N
- U7 pad A43: /FPGA_TangPrimerCore/MIPI_CK_P -> /DSI_CK_P
- U7 pad A45: /FPGA_TangPrimerCore/MIPI_CK_N -> /DSI_CK_N
- U7 pad A49: /FPGA_TangPrimerCore/MIPI_D1_P -> /DSI_D1_P
- U7 pad A51: /FPGA_TangPrimerCore/MIPI_D1_N -> /DSI_D1_N
- U7 pad A55: /FPGA_TangPrimerCore/MIPI_D0_P -> /DSI_D0_P
- U7 pad A57: /FPGA_TangPrimerCore/MIPI_D0_N -> /DSI_D0_N
Other:
- board outline added: 90 x 57 mm
- board text added: "たて"
- board text added: "よこ"

Commit message: シンボル・フットプリントMyLib->TomoshibiLib置き換え
Parts:
- removed C19: 10uF, Capacitor_SMD:C_0805_2012Metric
- removed J10: Conn_01x03_MountingPin, Connector_Molex:Molex_PicoBlade_53261-0371_1x03-1MP_P1.25mm_Horizontal
- removed R42, R43: 5.1k, Resistor_SMD:R_0402_1005Metric
- added C48: 10uF, Capacitor_SMD:C_0805_2012Metric, F.Cu at (24.7, 71.9)
- added C58: 47pF, Capacitor_SMD:C_0603_1608Metric, F.Cu at (28.3, 61.5)
- added C59: 47pF, Capacitor_SMD:C_0603_1608Metric, F.Cu at (28.3, 64.0)
- added C60: 0.1uF, Capacitor_SMD:C_0402_1005Metric, F.Cu at (26.9, 74.3)
- added C61: 0.1uF, Capacitor_SMD:C_0402_1005Metric, F.Cu at (26.9, 76.3)
- added J15: USB_C_Receptacle_USB2.0, Connector_USB:USB_C_Receptacle_G-Switch_GT-USB-7010ASV, F.Cu at (20.4, 65.7)
- added J7: RJ45_Hanrun_HR911105A_Horizontal, TomoshibiLibrary:Connector_RJ45_LPJK7001AGNL, F.Cu at (25.1, 48.1)
- added R101: 33, Resistor_SMD:R_0603_1608Metric, F.Cu at (28.3, 66.5)
- added R115: 33, Resistor_SMD:R_0603_1608Metric, F.Cu at (28.3, 69.1)
- added R51: 5.1k, Resistor_SMD:R_0402_1005Metric, F.Cu at (24.0, 74.4)
- added R52: 5.1k, Resistor_SMD:R_0402_1005Metric, F.Cu at (24.0, 76.3)
- added U20: FT231XS, Package_SO:SSOP-20_3.9x8.7mm_P0.635mm, F.Cu at (18.5, 75.5)
- J1: footprint MyLibrary:BoxHeader_2x07_P1.27mm_Horizontal -> TomoshibiLibrary:BoxHeader_2x07_P1.27mm_Horizontal
- J6: value USB_C_Receptacle_USB2.0 -> Conn_01x03_MountingPin; footprint Connector_USB:USB_C_Receptacle_G-Switch_GT-USB-7010ASV -> Connector_Molex:Molex_PicoBlade_53261-0371_1x03-1MP_P1.25mm_Horizontal
- L1: footprint MyLibrary:Inductor_CDPH4D19F -> TomoshibiLibrary:Inductor_CDPH4D19F
- Q12, Q14: footprint MyLibrary:Package_TSOP6F -> TomoshibiLibrary:Package_TSOP6F
- SW3, SW5, SW6: footprint MyLibrary:SW_Slide_3P_SPDT -> TomoshibiLibrary:SW_Slide_3P_SPDT
- SW4: footprint MyLibrary:SW_Slide_SPDT_White -> TomoshibiLibrary:SW_Slide_SPDT_White
- U16: value AZ1084CD-3.3 -> AZ1117CH-3.3; footprint Package_TO_SOT_SMD:TO-252-2 -> Package_TO_SOT_SMD:SOT-223-3_TabPin2
- U19: footprint MyLibrary:DCDC_TPS61023 -> TomoshibiLibrary:DCDC_TPS61023
- U7: footprint MyLibrary:FPGA_TangPrimer25K_Core -> TomoshibiLibrary:FPGA_TangPrimer25K_Core
Connections:
- C33 pad 1: Net-(Q5-E) -> +3.3V
- Q5 pad 2: Net-(Q5-E) -> +3.3V
- R39 pad 1: Net-(Q5-E) -> +3.3V
- U10 pad 8: Net-(Q5-E) -> +3.3V
- U6 pad 51: unconnected-(U6A-GPIO15-Pad51) -> /RasPi_CM4/RasPiRX0_SerialTX
- U6 pad 55: unconnected-(U6A-GPIO14-Pad55) -> /RasPi_CM4/RasPiTX0_SerialRX

Commit message: 配線
Parts:
- moved J1 0.20 mm to (37.9, -20.9)
- moved U7 0.13 mm to (-30.6, 1.92)

Commit message: 配線おけ
Parts:
- moved J12 243.0 mm to (24.7, -23.9), turned to 180 degrees
- moved J3 106.1 mm to (42.4, -2.49), turned to 90 degrees
Changed lines of the file:
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@@
   )
   (footprint "Connector_Molex:Molex_PicoBlade_53261-0671_1x06-1MP_P1.25mm_Horizontal" (layer "F.Cu")
-    (at 135.8175 47.825)
+    (at 42.388383 -2.493045 90)
     (descr "Molex PicoBlade series connector, 53261-0671 (http://www.molex.com/pdm_docs/sd/532610271_sd.pdf), generated with kicad-footprint-generator")
     (tags "connector Molex PicoBlade top entry")
@@
     (property "ki_keywords" "connector")
     (attr smd)
-    (fp_text reference "J3" (at 0 -4.4) (layer "F.SilkS")
+    (fp_text reference "J3" (at 0 -4.4 90) (layer "F.SilkS")
         (effects (font (size 1 1) (thickness 0.15)))
     )
-    (fp_text value "Conn_01x06_MountingPin" (at 0 3.8) (layer "F.Fab")
+    (fp_text value "Conn_01x06_MountingPin" (at 0 3.8 90) (layer "F.Fab")
         (effects (font (size 1 1) (thickness 0.15)))
     )
-    (fp_text user "${REFERENCE}" (at 0 1.9) (layer "F.Fab")
+    (fp_text user "${REFERENCE}" (at 0 1.9 90) (layer "F.Fab")
         (effects (font (size 1 1) (thickness 0.15)))
     )
@@
     (fp_line (start 6.325 1.4) (end 6.125 1.6)
       (stroke (width 0.1) (type solid)) (layer "F.Fab"))
-    (pad "1" smd roundrect (at -3.125 -2.4) (size 0.8 1.6) (layers "F.Cu" "F.Paste" "F.Mask") (roundrect_rratio 0.25)
+    (pad "1" smd roundrect (at -3.125 -2.4 90) (size 0.8 1.6) (layers "F.Cu" "F.Paste" "F.Mask") (roundrect_rratio 0.25)
       (net 2 "GND") (pinfunction "Pin_1") (pintype "passive"))
-    (pad "2" smd roundrect (at -1.875 -2.4) (size 0.8 1.6) (layers "F.Cu" "F.Paste" "F.Mask") (roundrect_rratio 0.25)
+    (pad "2" smd roundrect (at -1.875 -2.4 90) (size 0.8 1.6) (layers "F.Cu" "F.Paste" "F.Mask") (roundrect_rratio 0.25)
       (net 40 "+BATT") (pinfunction "Pin_2") (pintype "passive"))
-    (pad "3" smd roundrect (at -0.625 -2.4) (size 0.8 1.6) (layers "F.Cu" "F.Paste" "F.Mask") (roundrect_rratio 0.25)
+    (pad "3" smd roundrect (at -0.625 -2.4 90) (size 0.8 1.6) (layers "F.Cu" "F.Paste" "F.Mask") (roundrect_rratio 0.25)
       (net 45 "/RingNW/RS485_RingNW/RS485Y_TA") (pinfunction "Pin_3") (pintype "passive"))
-    (pad "4" smd roundrect (at 0.625 -2.4) (size 0.8 1.6) (layers "F.Cu" "F.Paste" "F.Mask") (roundrect_rratio 0.25)
+    (pad "4" smd roundrect (at 0.625 -2.4 90) (size 0.8 1.6) (layers "F.Cu" "F.Paste" "F.Mask") (roundrect_rratio 0.25)
       (net 46 "/RingNW/RS485_RingNW/RS485Y_TB") (pinfunction "Pin_4") (pintype "passive"))
-    (pad "5" smd roundrect (at 1.875 -2.4) (size 0.8 1.6) (layers "F.Cu" "F.Paste" "F.Mask") (roundrect_rratio 0.25)
+    (pad "5" smd roundrect (at 1.875 -2.4 90) (size 0.8 1.6) (layers "F.Cu" "F.Paste" "F.Mask") (roundrect_rratio 0.25)
       (net 47 "/RingNW/RS485_RingNW/RS485Y_RA") (pinfunction "Pin_5") (pintype "passive"))
-    (pad "6" smd roundrect (at 3.125 -2.4) (size 0.8 1.6) (layers "F.Cu" "F.Paste" "F.Mask") (roundrect_rratio 0.25)
+    (pad "6" smd roundrect (at 3.125 -2.4 90) (size 0.8 1.6) (layers "F.Cu" "F.Paste" "F.Mask") (roundrect_rratio 0.25)
       (net 48 "/RingNW/RS485_RingNW/RS485Y_RB") (pinfunction "Pin_6") (pintype "passive"))
-    (pad "MP" smd roundrect (at -5.675 0.5) (size 2.1 3) (layers "F.Cu" "F.Paste" "F.Mask") (roundrect_rratio 0.119048)
+    (pad "MP" smd roundrect (at -5.675 0.5 90) (size 2.1 3) (layers "F.Cu" "F.Paste" "F.Mask") (roundrect_rratio 0.119048)
       (net 2 "GND") (pinfunction "MountPin") (pintype "passive"))
-    (pad "MP" smd roundrect (at 5.675 0.5) (size 2.1 3) (layers "F.Cu" "F.Paste" "F.Mask") (roundrect_rratio 0.119048)
+    (pad "MP" smd roundrect (at 5.675 0.5 90) (size 2.1 3) (layers "F.Cu" "F.Paste" "F.Mask") (roundrect_rratio 0.119048)
       (net 2 "GND") (pinfunction "MountPin") (pintype "passive"))
     (model "${KICAD6_3DMODEL_DIR}/Connector_Molex.3dshapes/Molex_PicoBlade_53261-0671_1x06-1MP_P1.25mm_Horizontal.wrl"
@@
   )
   (footprint "Connector_Molex:Molex_PicoBlade_53261-0271_1x02-1MP_P1.25mm_Horizontal" (layer "F.Cu")
-    (at 267.4 -13.095)
+    (at 24.689951 -23.904691 180)
     (descr "Molex PicoBlade series connector, 53261-0271 (http://www.molex.com/pdm_docs/sd/532610271_sd.pdf), generated with kicad-footprint-generator")
     (tags "connector Molex PicoBlade top entry")
@@
     (fp_line (start 3.825 1.4) (end 3.625 1.6)
       (stroke (width 0.1) (type solid)) (layer "F.Fab"))
-    (pad "1" smd roundrect (at -0.625 -2.4) (size 0.8 1.6) (layers "F.Cu" "F.Paste" "F.Mask") (roundrect_rratio 0.25)
+    (pad "1" smd roundrect (at -0.625 -2.4 180) (size 0.8 1.6) (layers "F.Cu" "F.Paste" "F.Mask") (roundrect_rratio 0.25)
       (net 2 "GND") (pinfunction "Pin_1") (pintype "passive"))
-    (pad "2" smd roundrect (at 0.625 -2.4) (size 0.8 1.6) (layers "F.Cu" "F.Paste" "F.Mask") (roundrect_rratio 0.25)
+    (pad "2" smd roundrect (at 0.625 -2.4 180) (size 0.8 1.6) (layers "F.Cu" "F.Paste" "F.Mask") (roundrect_rratio 0.25)
       (net 157 "/FPGA_TangPrimerCore/DAC/LCH_OUT") (pinfunction "Pin_2") (pintype "passive"))
-    (pad "MP" smd roundrect (at -3.175 0.5) (size 2.1 3) (layers "F.Cu" "F.Paste" "F.Mask") (roundrect_rratio 0.119048)
+    (pad "MP" smd roundrect (at -3.175 0.5 180) (size 2.1 3) (layers "F.Cu" "F.Paste" "F.Mask") (roundrect_rratio 0.119048)
       (net 2 "GND") (pinfunction "MountPin") (pintype "passive"))
-    (pad "MP" smd roundrect (at 3.175 0.5) (size 2.1 3) (layers "F.Cu" "F.Paste" "F.Mask") (roundrect_rratio 0.119048)
+    (pad "MP" smd roundrect (at 3.175 0.5 180) (size 2.1 3) (layers "F.Cu" "F.Paste" "F.Mask") (roundrect_rratio 0.119048)
       (net 2 "GND") (pinfunction "MountPin") (pintype "passive"))
     (model "${KICAD6_3DMODEL_DIR}/Connector_Molex.3dshapes/Molex_PicoBlade_53261-0271_1x02-1MP_P1.25mm_Horizontal.wrl"
