File: circuits/RasPi/Power.kicad_sch (KiCad schematic)
At the start: 126 parts, among them J4 Conn_01x02_Pin, Q11 2N7002, Q12 SSM6J808R, Q14 SSM6J808R, Q15 S8550, Q16 SSM3J332R, Q17 S8550, Q29 SSM6J808R, Q30 S8550, Q31 MTP4835I3, Q32 S8550, Q33 SSM3J332R, Q34 2N7002, Q35 SSM3J332R, Q36 S8550, Q37 S8550, Q38 2N7002, Q6 SSM3J332R, Q7 S8550, Q8 SSM3J332R, Q9 S8550, SW4 SW_SPDT, U13 TPS54560BDDA, U16 AZ1117CH-3.3, U17 M51957B, U19 DCDC_TPS61023, U20 M51957B, U21 74AHC1G02, U22 NJM2732

Commit message: 発注第2弾
RasPi発注
Parts:
- removed C18: 100uF, Capacitor_SMD:C_1206_3216Metric, symbol Device:C
- removed C27, C32, C34: 470uF, symbol Device:C_Polarized
- removed D27: 1N5819WS, Diode_SMD:D_SOD-323_HandSoldering, symbol Device:D_Schottky
- removed Q29: SSM6J808R, TomoshibiLibrary:Package_TSOP6F, symbol Transistor_FET:PMN48XP
- removed Q33: SSM3J332R, Package_TO_SOT_SMD:SOT-23W, symbol Device:Q_PMOS_GSD
- removed TP2, TP3: TestPoint, TestPoint:TestPoint_THTPad_D2.0mm_Drill1.0mm, symbol Connector:TestPoint
- removed U17, U20: M51957B, Package_SO:SOP-8_3.9x4.9mm_P1.27mm, symbol TomoshibiLibrary:Power_Supervisor_M51957B
- removed U21: 74AHC1G02, Package_TO_SOT_SMD:SOT-23-5, symbol 74xGxx:74AHC1G02
- added C18: 220uF, Capacitor_Tantalum_SMD:CP_EIA-7343-20_Kemet-V, symbol Device:C_Polarized
- added C27: 10uF_50V, Capacitor_SMD:C_0805_2012Metric, symbol Device:C
- added C32, C34, C73, C74, C75: 100uF, Capacitor_SMD:C_1206_3216Metric, symbol Device:C
- added C72: 0.1uF, Capacitor_SMD:C_0402_1005Metric, symbol Device:C
- added D5: 1N5819WS, TomoshibiLibrary:Diode_SOD-323, symbol Device:D_Schottky
- added Q29: SSM3J332R, Package_TO_SOT_SMD:SOT-23W, symbol Device:Q_PMOS_GSD
- added Q33: SSM3K344R, Package_TO_SOT_SMD:SOT-23W, symbol Device:Q_NMOS_GSD
- added Q39: MTP4835I3, Package_TO_SOT_SMD:TO-252-2, symbol Device:Q_PMOS_GDS
- added Q40: 2N7002, Package_TO_SOT_SMD:SC-59, symbol Transistor_FET:2N7002
- added R136, R137, R144, R153: 5.1k, Resistor_SMD:R_0402_1005Metric, symbol Device:R
- added R138, R148, R154, R155: 10k, Resistor_SMD:R_0402_1005Metric, symbol Device:R
- added R139, R143: R, Resistor_SMD:R_0603_1608Metric, symbol Device:R
- added R140: 0.1, Resistor_SMD:R_0805_2012Metric, symbol Device:R
- added R141: 100k, Resistor_SMD:R_0402_1005Metric, symbol Device:R
- added R142: 100, Resistor_SMD:R_0603_1608Metric, symbol Device:R
- added R145, R156: 2k, Resistor_SMD:R_0402_1005Metric, symbol Device:R
- added R146, R147, R150: 1M, Resistor_SMD:R_0402_1005Metric, symbol Device:R
- added R149: 5, Resistor_SMD:R_2512_6332Metric, symbol Device:R
- added R151: 1M, Resistor_SMD:R_0603_1608Metric, symbol Device:R
- added R91: 1k, Resistor_SMD:R_0402_1005Metric, symbol Device:R
- added U17: NJU7109, Package_TO_SOT_SMD:SOT-23-5, symbol Comparator:LM397
- added U23: NJM2380, Package_TO_SOT_SMD:SOT-23-5, symbol Reference_Voltage:TL432DBV
- added U24: NJU77242, Package_SO:TSSOP-8_3x3mm_P0.65mm, symbol Comparator:LM2903
- added U25: 74AHC1G00, Package_TO_SOT_SMD:SOT-23-5, symbol 74xGxx:74AHC1G00
- C10, C16, C17: value 10uF -> 10uF_50V; footprint Capacitor_SMD:C_1206_3216Metric -> Capacitor_SMD:C_0805_2012Metric
- C26: value 100uF -> C; footprint Capacitor_SMD:C_1206_3216Metric -> Resistor_SMD:R_0603_1608Metric
- C29: value 470uF -> 47uF; footprint (none) -> Capacitor_SMD:CP_Elec_6.3x5.4
- C47: value 0.1uF -> 1uF
- C49: value 100uF -> 1uF; footprint Capacitor_SMD:C_1206_3216Metric -> Capacitor_SMD:C_0402_1005Metric
- C52: value 0.1uF -> 22uF; footprint Capacitor_SMD:C_0402_1005Metric -> Capacitor_SMD:C_0805_2012Metric
- C56, C70: value 15pF -> 100uF; footprint Capacitor_SMD:C_0402_1005Metric -> Capacitor_SMD:C_1206_3216Metric
- C9: value 100uF -> 4.7uF; footprint Capacitor_SMD:C_1206_3216Metric -> Capacitor_SMD:C_0603_1608Metric
- D16, D18, D4, D6, D8: footprint Diode_SMD:D_SOD-323_HandSoldering -> TomoshibiLibrary:Diode_SOD-323
- JP1: value SolderJumper_3_Bridged12 -> VBUS/VDD
- Q11, Q17, Q30, Q37, Q7, Q9: footprint Package_TO_SOT_SMD:SOT-23 -> Package_TO_SOT_SMD:SC-59
- R123: value 10k -> 510
- R124: value 100k -> 10k
- R125: footprint Resistor_SMD:R_1210_3225Metric -> Resistor_SMD:R_0805_2012Metric
- R128: value 200 -> 100; footprint Resistor_SMD:R_0402_1005Metric -> Resistor_SMD:R_0603_1608Metric
- R134: value 100k -> 3.3k; footprint Resistor_SMD:R_0603_1608Metric -> Resistor_SMD:R_0402_1005Metric
- R135: value 7.5k -> 2k; footprint Resistor_SMD:R_0603_1608Metric -> Resistor_SMD:R_0402_1005Metric
- R54: value 100k -> 2k; footprint Resistor_SMD:R_0603_1608Metric -> Resistor_SMD:R_0402_1005Metric
- R55: value 10k -> 22k
- R57: value 7.5k -> 2.2k; footprint Resistor_SMD:R_0603_1608Metric -> Resistor_SMD:R_0402_1005Metric
- R64, R66: value 10k -> 20k
- SW6: renamed from SW4; footprint TomoshibiLibrary:SW_Slide_SPDT_IS-1235-G -> TomoshibiLibrary:SW_Slide_SPDT_SSSS213202
- U22: footprint (none) -> TomoshibiLibrary:Package_TSSOP-8_4.4x3.5mm_P0.65mm
- renumbered J4 to J5
Connections:
- net +3.3V: now also C34.1
- net +5V: now also C47.1, C49.1, C56.1, C70.1, C71.2, Q35.2 (S), Q37.2 (E), R123.2, U22.8 (V+), C32.1, C72.2, C73.1, C74.1, C75.1, R136.2, R137.2, R138.2, R151.2, R153.2, U17.5 (V+), U24.8 (V+), U25.5 (VCC); no longer C47.2, C52.2, D18.1 (K), R55.2, TP1.1
- net CC: now also Q32.2 (E), Q29.2 (S), R140.1, R142.2
- net Cap: now also Q39.2 (D), R149.2, R91.2
- net GND: now also C47.2, C52.2, C9.1, R134.2, TP1.1, C18.2, C27.2, C32.2, C34.2, C72.1, C73.2, C74.2, C75.2, Q33.2 (S), Q40.2 (S), R138.1, R144.1, R148.1, R154.2, R155.1, U17.2 (V-), U23.2 (A), U24.4 (V-), U25.3 (GND); no longer C26.2, C47.1, C52.1, C9.2, R135.2, R55.1, U22.5 (+), U22.6 (-)
- net UV_SHDN: now also Q40.1 (G), R148.2, U25.4; no longer Q34.1 (G)
- net VBUS: now also R54.2
- net VDD: now also R55.2, C27.1; no longer R134.2, R54.2
- net VSYS: now also C9.2, D4.2 (A), L2.2, Q30.2 (E), R121.2, C18.1, D5.2 (A), Q29.3 (D); no longer C71.2, Q32.2 (E), Q35.2 (S), Q37.2 (E), R123.1, R46.1, R47.1, U22.8 (V+)
- net at Q34.3 (D): now also Q33.1 (G), R91.1; no longer R123.2
- net at R54.1, R57.1: now also U24.6 (-); no longer D18.2 (A)
- net at R134.1: now also R55.1, U24.2 (-); no longer R135.1
- net VCAP: now reaches C57.1, C66.1, C67.1, D16.1 (K), Q35.3 (D), Q36.2 (E), R99.2, U19.6 (VOUT)
- net VCAP: now also D18.2 (A)
- net at Q32.3 (C), R50.2: now also Q29.1 (G)
- net at U22.7: now also C26.1, R143.2
- net VBUS_UV: now reaches JP1.1 (A)
- net VBUS_UV: now also R137.1, R146.1, U24.7
- net at JP1.2 (C): now also U25.2
- net VDD_UV: now reaches JP1.3 (B)
- net VDD_UV: now also R136.1, R147.1, U24.1, U25.1
- net V_Meas. renamed V_Meas
- new net: C52.1, Q40.3 (D), R151.1, U17.1 (-)
- new net: R142.1, R144.2, U22.5 (+)
- new net: Q39.3 (S), R139.1, R140.2, R141.1
- new net: C26.2, R139.2, U22.6 (-)
- new net: Q39.1 (G), R141.2, R143.1
- new net: R145.1, R146.2, U24.5 (+)
- new net: D18.1 (K), D5.1 (K), R46.1, R47.1
- new net: R135.1, R147.2, U24.3 (+)
- new net: R123.1, R135.2, R145.2, U23.4 (K), U23.5 (REF)
- new net: Q34.1 (G), R150.1, R155.2, U17.4
- new net: R150.2, R156.1, U17.3 (+)
- new net: U23.1, U23.3
- new net: Q33.3 (D), R149.1
- new net: R153.1, R154.1, R156.2
- no-connect marks 3 -> 2
Other:
- note added: "24V系には20k!!!!"
- note added: "VDD-VBUS NAND"
- note added: "VDD/VBUS電圧監視"
- note added: "このダイオードは要検討・要実験 ダイオード着けるならR46いらない説ある"
- note added: "ゲート抵抗は大きめのほうがいいかも"
- note added: "放電回路"
- note added: "理想ダイオード/キャパシタ"
- note removed: "キャパシタ充電スイッチ"
- note removed: "電圧監視"
- note removed: "電源"
- moved on the sheet: C10, C16, C17, C21, C23, C24, C25, C29, C30, C50, C51, C55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
