File: circuits/RasPi/RasPi.kicad_sch (KiCad schematic)
At the start: 0 parts

Commit message: ラズパイ基板とか
Parts:
- added Q21: BSS138, Package_TO_SOT_SMD:SOT-23, symbol Device:Q_NMOS_GSD
- added R89: 10k, Resistor_SMD:R_0402_1005Metric, symbol Device:R
- added U6: SBC_RPi-CM4, MyLibrary:SBC_RPi-CM4, symbol MyLibrary:SBC_RPi-CM4
Connections:
- new net GNDD: Q21.2 (S), R89.2
- new net RST_FPGA: Q21.3 (D)
- new net RasPi->RST_FPGA: Q21.1 (G), R89.1
Other:
- sheet FPGA_TangPrimerCore ports: added CS, MIPI_CK_N, MIPI_CK_P, MIPI_D0_N, MIPI_D0_P, MIPI_D1_N, MIPI_D1_P, MIPI_D2_N, MIPI_D2_P, MIPI_D3_N, MIPI_D3_P, MISO, MOSI, SCLK, nRECONFIG; removed none
- sheet RingNW ports: added CSx_RasPi, F446RE->RasPi_GPIO3, MISOx, MOSIx, SCLKx, V_Meas.; removed none
- note added: "RasPi to TangPrimer Reset"

Commit message: PDFプロット
Parts:
- removed U6: SBC_RPi-CM4, MyLibrary:SBC_RPi-CM4, symbol MyLibrary:SBC_RPi-CM4
- added Q20, Q23: BSS138, Package_TO_SOT_SMD:SOT-23, symbol Device:Q_NMOS_GSD
- added R88, R91: 10k, Resistor_SMD:R_0402_1005Metric, symbol Device:R
Connections:
- net GNDD: now also Q20.2 (S), Q23.2 (S), R88.2, R91.2
- net RST_FPGA: no longer Q21.3 (D)
- net RasPi->RST_FPGA: no longer Q21.1 (G), R89.1
- new net F446RE->RasPi_GPIO3: Q20.1 (G), R88.1
- new net RST_TangPrimer: Q21.3 (D)
- new net RasPi->RST_TangPrimer: Q21.1 (G), R89.1
- new net RasPi_GPIO3: Q20.3 (D)
- new net RasPi_SHDN: Q23.3 (D)
- new net ResetIC->RasPi_SHDN: Q23.1 (G), R91.1
Other:
- sheet FPGA_TangPrimerCore ports: added PCM_CLK, PCM_DIN, PCM_DOUT, PCM_FS; removed none
- sheet Power ports: added UV_SHDN; removed none
- sheet RasPi_CM4 ports: added CSx_F446RE, CSy_FPGA, DSI1_CK_N, DSI1_CK_P, DSI1_D0_N, DSI1_D0_P, DSI1_D1_N, DSI1_D1_P, DSI1_D2_N, DSI1_D2_P, DSI1_D3_N, DSI1_D3_P, MISOx, MISOy, MOSIx, MOSIy, PCM_CLK, PCM_DIN, PCM_DOUT, PCM_FS, RasPi->RST_FPGA, SCLKx, SCLKy, SHDN/BOOT, V_SHDN; removed none
- sheet RingNW ports: added CSx; removed CSx_RasPi
- note added: "F446RE to RasPi Reset"
- note added: "GLOBAL_EN SHDN/BOOT(GPIO3) V_SHDN(電圧監視SHDN)"
- note added: "Reset IC to RasPi SHDN"
- note removed: "マイコン側のラベルと階層シート側のラベルをそれぞれ対応するように書き換える 電解コンの耐圧注意"
- moved on the sheet: Q21, R89

Commit message: 更新
Parts:
- removed Q20, Q21, Q23: BSS138, Package_TO_SOT_SMD:SOT-23, symbol Device:Q_NMOS_GSD
- added Q13, Q20, Q21: 2N7002, Package_TO_SOT_SMD:SOT-23, symbol Transistor_FET:2N7002
Connections:
- net F446RE->RasPi_GPIO3: now also Q13.1 (G)
- net GNDD: now also Q13.2 (S), Q20.2 (S), Q21.2 (S)
- net RST_TangPrimer: now also Q21.3 (D)
- net RasPi->RST_TangPrimer: now also Q21.1 (G)
- net RasPi_GPIO3: now also Q13.3 (D)
- net RasPi_SHDN: now also Q20.3 (D)
- net ResetIC->RasPi_SHDN: now also Q20.1 (G)
Changed lines of the file:
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@@
 (kicad_sch (version 20230121) (generator eeschema)
   (paper "A4")
+  (junction (at 152.4 137.16) (diameter 0) (color 0 0 0 0)
+  )
   (junction (at 160.02 185.42) (diameter 0) (color 0 0 0 0)
   )
   (junction (at 160.02 147.32) (diameter 0) (color 0 0 0 0)
   )
+  (junction (at 152.4 175.26) (diameter 0) (color 0 0 0 0)
+  )
+  (junction (at 233.68 137.16) (diameter 0) (color 0 0 0 0)
+  )
   (junction (at 241.3 147.32) (diameter 0) (color 0 0 0 0)
-  )
-  (junction (at 152.4 175.26) (diameter 0) (color 0 0 0 0)
-  )
-  (junction (at 233.68 137.16) (diameter 0) (color 0 0 0 0)
-  )
-  (junction (at 152.4 137.16) (diameter 0) (color 0 0 0 0)
   )
   (wire (pts (xy 81.28 73.66) (xy 83.82 73.66))
@@
     (effects (font (size 1.27 1.27) (thickness 0.254) bold italic) (justify right bottom))
   )
+  (symbol (lib_id "Transistor_FET:2N7002") (at 157.48 137.16 0) (unit 1)
+    (in_bom yes) (on_board yes) (dnp no)
+    (property "Reference" "Q13" (at 149.86 129.54 0)
+      (effects (font (size 1.27 1.27)) (justify left))
+    )
+    (property "Value" "2N7002" (at 149.86 132.08 0)
+      (effects (font (size 1.27 1.27)) (justify left))
+    )
+    (property "Footprint" "Package_TO_SOT_SMD:SOT-23" (at 162.56 139.065 0)
+      (effects (font (size 1.27 1.27) italic) (justify left) hide)
+    )
+    (property "Datasheet" "https://www.onsemi.com/pub/Collateral/NDS7002A-D.PDF" (at 162.56 140.97 0)
+      (effects (font (size 1.27 1.27)) (justify left) hide)
+    )
+    (pin "3")
+    (pin "1")
+    (pin "2")
+    (instances
+      (project "RasPi"
+        (path "/689a9e74-f202-4ea4-bfbb-4341f2549250"
+          (reference "Q13") (unit 1)
+        )
+      )
+    )
+  )
   (symbol (lib_id "Device:R") (at 152.4 180.34 0) (mirror y) (unit 1)
     (in_bom yes) (on_board yes) (dnp no)
@@
     )
   )
-  (symbol (lib_name "Q_NMOS_GSD_1") (lib_id "Device:Q_NMOS_GSD") (at 157.48 175.26 0) (unit 1)
-    (in_bom yes) (on_board yes) (dnp no)
-    (property "Reference" "Q23" (at 149.86 167.64 0)
-      (effects (font (size 1.27 1.27)) (justify left))
-    )
-    (property "Value" "BSS138" (at 149.86 170.18 0)
-      (effects (font (size 1.27 1.27)) (justify left))
-    )
-    (property "Footprint" "Package_TO_SOT_SMD:SOT-23" (at 162.56 172.72 0)
-      (effects (font (size 1.27 1.27)) hide)
-    )
-    (property "Datasheet" "~" (at 157.48 175.26 0)
+  (symbol (lib_id "Device:R") (at 233.68 142.24 0) (mirror y) (unit 1)
+    (in_bom yes) (on_board yes) (dnp no)
+    (property "Reference" "R89" (at 232.41 140.97 0)
+      (effects (font (size 1.27 1.27)) (justify left))
+    )
+    (property "Value" "10k" (at 232.41 143.51 0)
+      (effects (font (size 1.27 1.27)) (justify left))
+    )
+    (property "Footprint" "Resistor_SMD:R_0402_1005Metric" (at 235.458 142.24 90)
+      (effects (font (size 1.27 1.27)) hide)
+    )
+    (property "Datasheet" "~" (at 233.68 142.24 0)
       (effects (font (size 1.27 1.27)) hide)
     )
     (pin "1")
     (pin "2")
+    (instances
+      (project "RasPi"
+        (path "/689a9e74-f202-4ea4-bfbb-4341f2549250"
+          (reference "R89") (unit 1)
+        )
+      )
+    )
+  )
+  (symbol (lib_id "Transistor_FET:2N7002") (at 238.76 137.16 0) (unit 1)
+    (in_bom yes) (on_board yes) (dnp no)
+    (property "Reference" "Q21" (at 231.14 129.54 0)
+      (effects (font (size 1.27 1.27)) (justify left))
+    )
+    (property "Value" "2N7002" (at 231.14 132.08 0)
+      (effects (font (size 1.27 1.27)) (justify left))
+    )
+    (property "Footprint" "Package_TO_SOT_SMD:SOT-23" (at 243.84 139.065 0)
+      (effects (font (size 1.27 1.27) italic) (justify left) hide)
+    )
+    (property "Datasheet" "https://www.onsemi.com/pub/Collateral/NDS7002A-D.PDF" (at 243.84 140.97 0)
+      (effects (font (size 1.27 1.27)) (justify left) hide)
+    )
     (pin "3")
-    (instances
-      (project "RasPi"
-        (path "/689a9e74-f202-4ea4-bfbb-4341f2549250"
-          (reference "Q23") (unit 1)
-        )
-      )
-    )
-  )
-  (symbol (lib_id "Device:R") (at 233.68 142.24 0) (mirror y) (unit 1)
-    (in_bom yes) (on_board yes) (dnp no)
-    (property "Reference" "R89" (at 232.41 140.97 0)
-      (effects (font (size 1.27 1.27)) (justify left))
-    )
-    (property "Value" "10k" (at 232.41 143.51 0)
-      (effects (font (size 1.27 1.27)) (justify left))
-    )
-    (property "Footprint" "Resistor_SMD:R_0402_1005Metric" (at 235.458 142.24 90)
-      (effects (font (size 1.27 1.27)) hide)
-    )
-    (property "Datasheet" "~" (at 233.68 142.24 0)
-      (effects (font (size 1.27 1.27)) hide)
-    )
     (pin "1")
     (pin "2")
@@
       (project "RasPi"
         (path "/689a9e74-f202-4ea4-bfbb-4341f2549250"
-          (reference "R89") (unit 1)
-        )
-      )
-    )
-  )
-  (symbol (lib_name "Q_NMOS_GSD_1") (lib_id "Device:Q_NMOS_GSD") (at 157.48 137.16 0) (unit 1)
-    (in_bom yes) (on_board yes) (dnp no)
-    (property "Reference" "Q20" (at 149.86 129.54 0)
-      (effects (font (size 1.27 1.27)) (justify left))
-    )
-    (property "Value" "BSS138" (at 149.86 132.08 0)
-      (effects (font (size 1.27 1.27)) (justify left))
-    )
-    (property "Footprint" "Package_TO_SOT_SMD:SOT-23" (at 162.56 134.62 0)
-      (effects (font (size 1.27 1.27)) hide)
-    )
-    (property "Datasheet" "~" (at 157.48 137.16 0)
-      (effects (font (size 1.27 1.27)) hide)
-    )
+          (reference "Q21") (unit 1)
+        )
+      )
+    )
+  )
+  (symbol (lib_id "Transistor_FET:2N7002") (at 157.48 175.26 0) (unit 1)
+    (in_bom yes) (on_board yes) (dnp no)
+    (property "Reference" "Q20" (at 149.86 167.64 0)
+      (effects (font (size 1.27 1.27)) (justify left))
+    )
+    (property "Value" "2N7002" (at 149.86 170.18 0)
+      (effects (font (size 1.27 1.27)) (justify left))
+    )
+    (property "Footprint" "Package_TO_SOT_SMD:SOT-23" (at 162.56 177.165 0)
+      (effects (font (size 1.27 1.27) italic) (justify left) hide)
+    )
+    (property "Datasheet" "https://www.onsemi.com/pub/Collateral/NDS7002A-D.PDF" (at 162.56 179.07 0)
+      (effects (font (size 1.27 1.27)) (justify left) hide)
+    )
+    (pin "3")
     (pin "1")
     (pin "2")
-    (pin "3")
     (instances
       (project "RasPi"
@@
         )
       )
-    )
-  )
-  (symbol (lib_name "Q_NMOS_GSD_1") (lib_id "Device:Q_NMOS_GSD") (at 238.76 137.16 0) (unit 1)
-    (in_bom yes) (on_board yes) (dnp no)
-    (property "Reference" "Q21" (at 231.14 129.54 0)
-      (effects (font (size 1.27 1.27)) (justify left))
-    )
-    (property "Value" "BSS138" (at 231.14 132.08 0)
-      (effects (font (size 1.27 1.27)) (justify left))
-    )
-    (property "Footprint" "Package_TO_SOT_SMD:SOT-23" (at 243.84 134.62 0)
-      (effects (font (size 1.27 1.27)) hide)
-    )
-    (property "Datasheet" "~" (at 238.76 137.16 0)
-      (effects (font (size 1.27 1.27)) hide)
-    )
-    (pin "1")
-    (pin "2")
-    (pin "3")
-    (instances
-      (project "RasPi"
-        (path "/689a9e74-f202-4ea4-bfbb-4341f2549250"
-          (reference "Q21") (unit 1)
-        )
-      )

Commit message: raspi基板回路図
Connections:
- net RST_TangPrimer is gone; now on net RST_FPGA: Q21.3 (D)
- net RasPi->RST_TangPrimer is gone; now on net RasPi->RST_FPGA: Q21.1 (G), R89.1
- net F446RE->RasPi_GPIO3 renamed MCU->RasPi_GPIO3
Other:
- sheet RasPi_CM4 ports: added CS0_MCU, CS4_FPGA, MISO0, MISO4, MOSI0, MOSI4, SCLK0, SCLK4; removed CSx_F446RE, CSy_FPGA, MISOx, MISOy, MOSIx, MOSIy, SCLKx, SCLKy
- sheet RingNW ports: added H723VG->RasPi_GPIO3; removed F446RE->RasPi_GPIO3
- note added: "H723VG to RasPi Reset"
- note removed: "F446RE to RasPi Reset"
Changed lines of the file:
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@@
     (stroke (width 0) (type default))
   )
-  (rectangle (start 205.74 119.38) (end 259.08 154.94)
+  (rectangle (start 205.74 119.38) (end 256.54 154.94)
     (stroke (width 0) (type default))
     (fill (type none))
@@
     (fill (type none))
   )
-  (text "F446RE to RasPi Reset" (at 127 124.46 0)
+  (text "H723VG to RasPi Reset" (at 127 124.46 0)
     (effects (font (size 1.27 1.27)) (justify left bottom))
   )
@@
     (effects (font (size 1.27 1.27) (thickness 0.254) bold italic) (justify left bottom))
   )
-  (label "F446RE->RasPi_GPIO3" (at 149.86 137.16 180) (fields_autoplaced)
+  (label "MCU->RasPi_GPIO3" (at 149.86 137.16 180) (fields_autoplaced)
     (effects (font (size 1.27 1.27) (thickness 0.254) bold italic) (justify right bottom))
   )
@@
     (effects (font (size 1.27 1.27) (thickness 0.254) bold italic) (justify left bottom))
   )
-  (label "RasPi->F446RE_CS" (at 132.08 73.66 180) (fields_autoplaced)
+  (label "RasPi->MCU_CS" (at 132.08 73.66 180) (fields_autoplaced)
     (effects (font (size 1.27 1.27) (thickness 0.254) bold italic) (justify right bottom))
   )
@@
     (effects (font (size 1.27 1.27) (thickness 0.254) bold italic) (justify right bottom))
   )
-  (label "RasPi->F446RE_MOSI" (at 83.82 66.04 0) (fields_autoplaced)
-    (effects (font (size 1.27 1.27) (thickness 0.254) bold italic) (justify left bottom))
-  )
   (label "RST_FPGA" (at 215.9 55.88 180) (fields_autoplaced)
     (effects (font (size 1.27 1.27) (thickness 0.254) bold italic) (justify right bottom))
@@
     (effects (font (size 1.27 1.27) (thickness 0.254) bold italic) (justify left bottom))
   )
-  (label "RST_TangPrimer" (at 241.3 129.54 0) (fields_autoplaced)
-    (effects (font (size 1.27 1.27) (thickness 0.254) bold italic) (justify left bottom))
-  )
-  (label "RasPi->F446RE_MISO" (at 132.08 68.58 180) (fields_autoplaced)
+  (label "RST_FPGA" (at 241.3 129.54 0) (fields_autoplaced)
+    (effects (font (size 1.27 1.27) (thickness 0.254) bold italic) (justify left bottom))
+  )
+  (label "RasPi->MCU_MISO" (at 132.08 68.58 180) (fields_autoplaced)
     (effects (font (size 1.27 1.27) (thickness 0.254) bold italic) (justify right bottom))
   )
@@
     (effects (font (size 1.27 1.27) (thickness 0.254) bold italic) (justify right bottom))
   )
-  (label "RasPi->F446RE_SCLK" (at 132.08 71.12 180) (fields_autoplaced)
+  (label "RasPi->MCU_MOSI" (at 83.82 66.04 0) (fields_autoplaced)
+    (effects (font (size 1.27 1.27) (thickness 0.254) bold italic) (justify left bottom))
+  )
+  (label "RasPi->MCU_SCLK" (at 132.08 71.12 180) (fields_autoplaced)
     (effects (font (size 1.27 1.27) (thickness 0.254) bold italic) (justify right bottom))
   )
@@
     (effects (font (size 1.27 1.27) (thickness 0.254) bold italic) (justify left bottom))
   )
-  (label "RasPi->RST_TangPrimer" (at 231.14 137.16 180) (fields_autoplaced)
-    (effects (font (size 1.27 1.27) (thickness 0.254) bold italic) (justify right bottom))
-  )
-  (label "RasPi->F446RE_MISO" (at 83.82 68.58 0) (fields_autoplaced)
-    (effects (font (size 1.27 1.27) (thickness 0.254) bold italic) (justify left bottom))
-  )
-  (label "F446RE->RasPi_GPIO3" (at 83.82 60.96 0) (fields_autoplaced)
+  (label "RasPi->RST_FPGA" (at 231.14 137.16 180) (fields_autoplaced)
+    (effects (font (size 1.27 1.27) (thickness 0.254) bold italic) (justify right bottom))
+  )
+  (label "MCU->RasPi_GPIO3" (at 83.82 60.96 0) (fields_autoplaced)
     (effects (font (size 1.27 1.27) (thickness 0.254) bold italic) (justify left bottom))
   )
@@
     (effects (font (size 1.27 1.27) (thickness 0.254) bold italic) (justify left bottom))
   )
-  (label "RasPi->F446RE_MOSI" (at 132.08 66.04 180) (fields_autoplaced)
-    (effects (font (size 1.27 1.27) (thickness 0.254) bold italic) (justify right bottom))
+  (label "RasPi->MCU_MOSI" (at 132.08 66.04 180) (fields_autoplaced)
+    (effects (font (size 1.27 1.27) (thickness 0.254) bold italic) (justify right bottom))
+  )
+  (label "RasPi->MCU_MISO" (at 83.82 68.58 0) (fields_autoplaced)
+    (effects (font (size 1.27 1.27) (thickness 0.254) bold italic) (justify left bottom))
   )
   (label "RasPi_SHDN" (at 160.02 167.64 0) (fields_autoplaced)
     (effects (font (size 1.27 1.27) (thickness 0.254) bold italic) (justify left bottom))
   )
+  (label "RasPi->MCU_CS" (at 83.82 73.66 0) (fields_autoplaced)
+    (effects (font (size 1.27 1.27) (thickness 0.254) bold italic) (justify left bottom))
+  )
   (label "DSI_D0_N" (at 215.9 81.28 180) (fields_autoplaced)
     (effects (font (size 1.27 1.27) (thickness 0.254) bold italic) (justify right bottom))
@@
     (effects (font (size 1.27 1.27) (thickness 0.254) bold italic) (justify right bottom))
   )
-  (label "RasPi->F446RE_CS" (at 83.82 73.66 0) (fields_autoplaced)
-    (effects (font (size 1.27 1.27) (thickness 0.254) bold italic) (justify left bottom))
-  )
-  (label "RasPi->F446RE_SCLK" (at 83.82 71.12 0) (fields_autoplaced)
+  (label "RasPi->MCU_SCLK" (at 83.82 71.12 0) (fields_autoplaced)
     (effects (font (size 1.27 1.27) (thickness 0.254) bold italic) (justify left bottom))
   )
@@
       (effects (font (size 1.27 1.27)) (justify right))
     )
-    (pin "F446RE->RasPi_GPIO3" input (at 81.28 60.96 0)
-      (effects (font (size 1.27 1.27)) (justify right))
-    )
     (pin "V_Meas." input (at 81.28 55.88 0)
       (effects (font (size 1.27 1.27)) (justify right))
     )
     (pin "CSx" input (at 81.28 73.66 0)
+      (effects (font (size 1.27 1.27)) (justify right))
+    )
+    (pin "H723VG->RasPi_GPIO3" input (at 81.28 60.96 0)
       (effects (font (size 1.27 1.27)) (justify right))
     )
@@
       (effects (font (size 1.27 1.27)) (justify left top))
     )
-    (pin "MOSIx" input (at 134.62 66.04 180)
-      (effects (font (size 1.27 1.27)) (justify left))
-    )
     (pin "RasPi->RST_FPGA" input (at 165.1 55.88 0)
       (effects (font (size 1.27 1.27)) (justify right))
     )
-    (pin "SCLKx" input (at 134.62 71.12 180)
-      (effects (font (size 1.27 1.27)) (justify left))
-    )
-    (pin "MISOx" input (at 134.62 68.58 180)
-      (effects (font (size 1.27 1.27)) (justify left))
-    )
-    (pin "MOSIy" input (at 165.1 60.96 0)
-      (effects (font (size 1.27 1.27)) (justify right))
-    )
-    (pin "CSy_FPGA" input (at 165.1 68.58 0)
-      (effects (font (size 1.27 1.27)) (justify right))
-    )
-    (pin "SCLKy" input (at 165.1 66.04 0)
-      (effects (font (size 1.27 1.27)) (justify right))
-    )
-    (pin "MISOy" input (at 165.1 63.5 0)
-      (effects (font (size 1.27 1.27)) (justify right))
-    )
-    (pin "CSx_F446RE" input (at 134.62 73.66 180)
-      (effects (font (size 1.27 1.27)) (justify left))
-    )
     (pin "SHDN{slash}BOOT" input (at 134.62 60.96 180)
       (effects (font (size 1.27 1.27)) (justify left))
@@
       (effects (font (size 1.27 1.27)) (justify right))
     )
+    (pin "MOSI0" input (at 134.62 66.04 180)
+      (effects (font (size 1.27 1.27)) (justify left))
+    )
+    (pin "SCLK0" input (at 134.62 71.12 180)
+      (effects (font (size 1.27 1.27)) (justify left))
+    )
+    (pin "MISO0" input (at 134.62 68.58 180)
+      (effects (font (size 1.27 1.27)) (justify left))
+    )
+    (pin "CS0_MCU" input (at 134.62 73.66 180)
+      (effects (font (size 1.27 1.27)) (justify left))
+    )
+    (pin "SCLK4" input (at 165.1 66.04 0)
+      (effects (font (size 1.27 1.27)) (justify right))
+    )
+    (pin "MOSI4" input (at 165.1 60.96 0)
+      (effects (font (size 1.27 1.27)) (justify right))
+    )
+    (pin "MISO4" input (at 165.1 63.5 0)
+      (effects (font (size 1.27 1.27)) (justify right))
+    )
+    (pin "CS4_FPGA" input (at 165.1 68.58 0)
+      (effects (font (size 1.27 1.27)) (justify right))
+    )
