File: circuits/DCDC/DCDC.kicad_pcb (KiCad board)
At the start: 2 copper layers, 270 parts

Commit message: 更新
Parts:
- removed C100, C101, C102, C103, C104, C105, C106, C107, C108, C109, C110, C111, C112, C113, C114, C115, C116, C117, C118, C119, C120, C121, C122, C123, C124, C125, C126, C127, C128, C26, C27, C28, C29, C30, C31, C32, C33, C34, C35, C36, C37, C38, C39, C40, C41, C42, C43, C44, C45, C46, C47, C48, C49, C50, C51, C52, C53, C54, C55, C56, C57, C58, C59, C60, C61, C62, C63, C64, C65, C66, C67, C68, C69, C70, C71, C72, C73, C74, C75, C76, C77, C78, C79, C80, C81, C82, C83, C84, C85, C86, C87, C88, C89, C90, C91, C92, C93, C94, C95, C96, C97, C98, C99: 0.1uF, Capacitor_SMD:C_0402_1005Metric
- removed D100, D101, D102, D103, D104, D105, D106, D107, D108, D109, D11, D110, D111, D112, D113, D114, D115, D116, D117, D118, D119, D12, D120, D121, D122, D123, D124, D125, D126, D127, D128, D13, D14, D15, D16, D17, D18, D19, D20, D21, D22, D23, D24, D25, D26, D27, D28, D29, D30, D31, D32, D33, D34, D35, D36, D37, D38, D39, D40, D41, D42, D43, D44, D45, D46, D47, D48, D49, D50, D51, D52, D53, D54, D55, D56, D57, D58, D59, D60, D61, D62, D63, D64, D65, D66, D67, D68, D69, D70, D71, D72, D73, D74, D75, D76, D77, D78, D79, D80, D81, D82, D83, D84, D85, D86, D87, D88, D89, D90, D91, D92, D93, D94, D95, D96, D97, D98, D99: WS2812C-2020-V1, MyLibrary:NeoPixel_WS2812C-2020-V1
- removed H1, H2: MountingHole_Pad, TestPoint:TestPoint_Pad_3.0x3.0mm
- removed H10, H11, H12, H13, H14, H3, H4, H5, H6, H7, H8, H9: MountingHole_Pad, TestPoint:TestPoint_Pad_2.0x2.0mm
- added J1: Conn_01x07_MountingPin, Connector_Molex:Molex_PicoBlade_53261-0771_1x07-1MP_P1.25mm_Horizontal, F.Cu at (109.2, -31.9)
- added J2: Conn_01x02_Male, Connector_AMASS:AMASS_XT30PW-M_1x02_P2.50mm_Horizontal, F.Cu at (99.3, 17.3)
- added J3: Conn_01x02_Female, Connector_AMASS:AMASS_XT30PW-F_1x02_P2.50mm_Horizontal, F.Cu at (83.8, 8.88)
- added Q1: S8550, Package_TO_SOT_SMD:SOT-23, F.Cu at (100.3, -25.5)
- added Q10: MTP4835I3, Package_TO_SOT_SMD:TO-252-2, F.Cu at (80.0, 19.8)
- added Q11: MTP4835I3, Package_TO_SOT_SMD:TO-252-2, F.Cu at (85.7, 25.5)
- added Q12: BSS138, Package_TO_SOT_SMD:SOT-23, F.Cu at (92.7, -11.4)
- added Q2: S8550, Package_TO_SOT_SMD:SOT-23, F.Cu at (103.6, -22.3)
- added Q3: S8550, Package_TO_SOT_SMD:SOT-23, F.Cu at (106.8, -19.0)
- added Q4: S8550, Package_TO_SOT_SMD:SOT-23, F.Cu at (110.1, -15.7)
- added Q5: S8550, Package_TO_SOT_SMD:SOT-23, F.Cu at (113.4, -12.4)
- added Q6: S8550, Package_TO_SOT_SMD:SOT-23, F.Cu at (116.7, -9.17)
- added Q7: 2SC3265, Package_TO_SOT_SMD:SOT-23, F.Cu at (89.5, -14.7)
- added Q8: MTP4835I3, Package_TO_SOT_SMD:TO-252-2, F.Cu at (68.7, 8.43)
- added Q9: MTP4835I3, Package_TO_SOT_SMD:TO-252-2, F.Cu at (74.3, 14.1)
- added R1: 2.2k, Resistor_SMD:R_0402_1005Metric, F.Cu at (110.5, -26.6)
- added R10: 2.2k, Resistor_SMD:R_0402_1005Metric, F.Cu at (118.9, -18.1)
- added R11: 2.2k, Resistor_SMD:R_0402_1005Metric, F.Cu at (112.5, -28.6)
- added R12: 2.2k, Resistor_SMD:R_0402_1005Metric, F.Cu at (113.9, -27.2)
- added R13: 2.2k, Resistor_SMD:R_0402_1005Metric, F.Cu at (115.3, -25.8)
- added R14: 2.2k, Resistor_SMD:R_0402_1005Metric, F.Cu at (116.7, -24.4)
- added R15: 2.2k, Resistor_SMD:R_0402_1005Metric, F.Cu at (118.1, -23.0)
- added R16: 7.5k, Resistor_SMD:R_0603_1608Metric, F.Cu at (113.5, -18.6)
- added R17: 7.5k, Resistor_SMD:R_0603_1608Metric, F.Cu at (115.3, -16.8)
- added R18: 7.5k, Resistor_SMD:R_0603_1608Metric, F.Cu at (117.1, -15.1)
- added R19: 20k, Resistor_SMD:R_0402_1005Metric, F.Cu at (119.5, -21.6)
- added R2: 2.2k, Resistor_SMD:R_0402_1005Metric, F.Cu at (111.9, -25.2)
- added R20: 20k, Resistor_SMD:R_0402_1005Metric, F.Cu at (121.0, -20.2)
- added R21: 20k, Resistor_SMD:R_0402_1005Metric, F.Cu at (114.6, -30.7)
- added R22: 2.2k, Resistor_SMD:R_0402_1005Metric, F.Cu at (116.0, -29.3)
- added R23: 2.2k, Resistor_SMD:R_0402_1005Metric, F.Cu at (117.4, -27.9)
- added R24: 2.2k, Resistor_SMD:R_0402_1005Metric, F.Cu at (118.8, -26.5)
- added R25: 1k, Resistor_SMD:R_0402_1005Metric, F.Cu at (106.9, 9.76)
- added R26: 510, Resistor_SMD:R_0402_1005Metric, F.Cu at (108.3, 11.2)
- added R27: 10k, Resistor_SMD:R_0402_1005Metric, F.Cu at (109.7, 12.6)
- added R28: 10, Resistor_SMD:R_0603_1608Metric, F.Cu at (82.7, -9.50)
- added R29: 10k, Resistor_SMD:R_0402_1005Metric, F.Cu at (111.1, 14.0)
- added R3: 2.2k, Resistor_SMD:R_0402_1005Metric, F.Cu at (113.3, -23.7)
- added R30: R_snub, Resistor_SMD:R_0603_1608Metric, F.Cu at (84.4, -7.73)
- added R31: 1k, Resistor_SMD:R_0402_1005Metric, F.Cu at (112.5, 15.4)
- added R32: 1k, Resistor_SMD:R_0402_1005Metric, F.Cu at (108.9, 7.71)
- added R33: R_snub, Resistor_SMD:R_0603_1608Metric, F.Cu at (86.2, -5.95)
- added R34: R_snub, Resistor_SMD:R_0603_1608Metric, F.Cu at (88.0, -4.18)
- added R35: 5.1k, Resistor_SMD:R_0402_1005Metric, F.Cu at (110.3, 9.11)
- added R36: 5.1k, Resistor_SMD:R_0603_1608Metric, F.Cu at (89.8, -2.40)
- added R37: 7.5k, Resistor_SMD:R_0603_1608Metric, F.Cu at (85.5, -12.3)
- added R38: 1.5k, Resistor_SMD:R_0603_1608Metric, F.Cu at (87.3, -10.6)
- added R39: 10k, Resistor_SMD:R_0402_1005Metric, F.Cu at (111.8, 10.5)
- added R4: 7.5k, Resistor_SMD:R_0603_1608Metric, F.Cu at (108.2, -23.9)
- added R40: 2k, Resistor_SMD:R_0603_1608Metric, F.Cu at (89.1, -8.79)
- added R41: 100k, Resistor_SMD:R_0402_1005Metric, F.Cu at (113.2, 11.9)
- added R42: 10k, Resistor_SMD:R_0402_1005Metric, F.Cu at (114.6, 13.3)
- added R43: 33k, Resistor_SMD:R_0603_1608Metric, F.Cu at (90.8, -7.01)
- added R44: 10k, Resistor_SMD:R_0402_1005Metric, F.Cu at (111.0, 5.65)
- added R45: 10k, Resistor_SMD:R_0603_1608Metric, F.Cu at (92.6, -5.24)
- added R46: 1k, Resistor_SMD:R_0402_1005Metric, F.Cu at (112.4, 7.06)
- added R47: 10k, Resistor_SMD:R_0402_1005Metric, F.Cu at (113.8, 8.46)
- added R48: 10k, Resistor_SMD:R_0402_1005Metric, F.Cu at (115.2, 9.87)
- added R5: 7.5k, Resistor_SMD:R_0603_1608Metric, F.Cu at (110.0, -22.2)
- added R6: 7.5k, Resistor_SMD:R_0603_1608Metric, F.Cu at (111.7, -20.4)
- added R7: 20k, Resistor_SMD:R_0402_1005Metric, F.Cu at (114.7, -22.3)
- added R8: 20k, Resistor_SMD:R_0402_1005Metric, F.Cu at (116.1, -20.9)
- added R9: 20k, Resistor_SMD:R_0402_1005Metric, F.Cu at (117.5, -19.5)
- added TP1: TestPoint, TestPoint:TestPoint_THTPad_D2.0mm_Drill1.0mm, F.Cu at (95.8, 3.65)
- added TP2: TestPoint, TestPoint:TestPoint_THTPad_D2.0mm_Drill1.0mm, F.Cu at (98.7, 6.51)
- added TP3: TestPoint, TestPoint:TestPoint_THTPad_D2.0mm_Drill1.0mm, F.Cu at (101.6, 9.38)
- added TP4: TestPoint, TestPoint:TestPoint_THTPad_D2.0mm_Drill1.0mm, F.Cu at (104.4, 12.2)
- added TP5: TestPoint, TestPoint:TestPoint_THTPad_D2.0mm_Drill1.0mm, F.Cu at (107.3, 15.1)
- added U1: MAX3485, Package_SO:SOP-8_3.9x4.9mm_P1.27mm, F.Cu at (96.3, -20.1)
- added U2: MAX3485, Package_SO:SOP-8_3.9x4.9mm_P1.27mm, F.Cu at (100.9, -15.5)
- added U3: MAX3485, Package_SO:SOP-8_3.9x4.9mm_P1.27mm, F.Cu at (105.6, -10.8)
- added U4: MAX3485, Package_SO:SOP-8_3.9x4.9mm_P1.27mm, F.Cu at (110.2, -6.17)
- added U5: MAX3485, Package_SO:SOP-8_3.9x4.9mm_P1.27mm, F.Cu at (114.9, -1.52)
- added U6: MAX3485, Package_SO:SOP-8_3.9x4.9mm_P1.27mm, F.Cu at (119.5, 3.13)
- added U7: MC34063AD, Package_SO:SOIC-8_3.9x4.9mm_P1.27mm, F.Cu at (101.2, 0.17)
- added U8: AZ1084CD-3.3, Package_TO_SOT_SMD:TO-252-2, F.Cu at (91.4, 31.2)
- added U9: M51957B, Package_SO:SOP-8_3.9x4.9mm_P1.27mm, F.Cu at (105.9, 4.82)
- C11, C15, C16: value 0.1uF -> C_snub; footprint Capacitor_SMD:C_0402_1005Metric -> Capacitor_SMD:C_0603_1608Metric
- C12, C8, C9: value 0.1uF -> 10uF; footprint Capacitor_SMD:C_0402_1005Metric -> Capacitor_SMD:C_0805_2012Metric
- C13: value 0.1uF -> 470uF; footprint Capacitor_SMD:C_0402_1005Metric -> Capacitor_THT:CP_Radial_D10.0mm_P2.50mm_P5.00mm
- C14: value 0.1uF -> 100pF; footprint Capacitor_SMD:C_0402_1005Metric -> Capacitor_SMD:C_0603_1608Metric
- C17, C18, C19, C20: value 0.1uF -> 470uF; footprint Capacitor_SMD:C_0402_1005Metric -> Capacitor_SMD:C_Elec_8x10.2
- C21, C23, C24: value 0.1uF -> 1uF
- C25: value 0.1uF -> 4700pF; footprint Capacitor_SMD:C_0402_1005Metric -> Capacitor_SMD:C_0603_1608Metric
- D1, D6: value WS2812C-2020-V1 -> Green; footprint MyLibrary:NeoPixel_WS2812C-2020-V1 -> LED_SMD:LED_0603_1608Metric_Pad1.05x0.95mm_HandSolder
- D10, D2, D3: value WS2812C-2020-V1 -> SS2040FL; footprint MyLibrary:NeoPixel_WS2812C-2020-V1 -> Diode_SMD:D_SOD-123
- D4, D5, D8, D9: value WS2812C-2020-V1 -> 1N5819WS; footprint MyLibrary:NeoPixel_WS2812C-2020-V1 -> Diode_SMD:D_SOD-323_HandSoldering
- D7: value WS2812C-2020-V1 -> CBD20150VCT; footprint MyLibrary:NeoPixel_WS2812C-2020-V1 -> Package_TO_SOT_THT:TO-220-3_Horizontal_TabDown
- moved C14 81.6 mm to (59.6, 20.6), turned to 45 degrees
- moved C15 80.6 mm to (61.0, 21.9), turned to 45 degrees
- moved C1 80.0 mm to (57.6, 22.6), turned to 45 degrees
- moved C16 79.6 mm to (62.4, 23.3), turned to 45 degrees
- moved C2 78.9 mm to (59.0, 24.0), turned to 45 degrees
- moved C17 78.6 mm to (63.8, 24.7), turned to 45 degrees
- moved C3 77.9 mm to (60.4, 25.4), turned to 45 degrees
- moved C18 77.7 mm to (65.2, 26.1), turned to 45 degrees
- moved C4 76.9 mm to (61.8, 26.8), turned to 45 degrees
- moved C19 76.8 mm to (66.6, 27.5), turned to 45 degrees
- moved C5 76.0 mm to (63.2, 28.2), turned to 45 degrees
- moved C20 75.8 mm to (68.0, 28.9), turned to 45 degrees
- moved C6 75.0 mm to (64.6, 29.5), turned to 45 degrees
- moved C21 74.9 mm to (69.4, 30.3), turned to 45 degrees
- moved C7 74.1 mm to (65.9, 30.9), turned to 45 degrees
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Connections:
- C1 pad 1: VDD -> +3.3V
- C1 pad 2: GND -> GNDD
- C10 pad 1: VDD -> GND
- C10 pad 2: GND -> Net-(D2-K)
- C11 pad 1: VDD -> GND
- C11 pad 2: GND -> Net-(C11-Pad2)
- C12 pad 1: VDD -> Net-(D4-A)
- C13 pad 1: VDD -> Net-(D4-A)
- C14 pad 1: VDD -> GND
- C14 pad 2: GND -> Net-(U7-TC)
- C15 pad 1: VDD -> GND
- C15 pad 2: GND -> Net-(C15-Pad2)
- C16 pad 1: VDD -> GND
- C16 pad 2: GND -> Net-(C16-Pad2)
- C18 pad 1: VDD -> +5V
- C19 pad 1: VDD -> VCC
- C2 pad 1: VDD -> +3.3V
- C2 pad 2: GND -> GNDD
- C20 pad 1: VDD -> +3.3V
- C21 pad 1: VDD -> /Power/S-S
- C21 pad 2: GND -> Net-(Q11-G)
- C22 pad 1: VDD -> GND
- C22 pad 2: GND -> VDD
- C23 pad 1: VDD -> VCC
- C24 pad 1: VDD -> +3.3V
- C25 pad 1: VDD -> GND
- C25 pad 2: GND -> Net-(U9-Cdelay)
- C3 pad 1: VDD -> +3.3V
- C3 pad 2: GND -> GNDD
- C4 pad 1: VDD -> +3.3V
- C4 pad 2: GND -> GNDD
- C5 pad 1: VDD -> +3.3V
- C5 pad 2: GND -> GNDD
- C6 pad 1: VDD -> +3.3V
- C6 pad 2: GND -> GNDD
- C7 pad 1: VDD -> GND
- C7 pad 2: GND -> VDD
- C9 pad 1: VDD -> Net-(D2-K)
- D1 pad 1: Net-(D1-DOUT) -> GND
- D1 pad 2: GND -> Net-(D1-A)
- D10 pad 1: Net-(D10-DOUT) -> VCC
- D10 pad 2: GND -> +5V
- D2 pad 1: Net-(D2-DOUT) -> Net-(D2-K)
- D2 pad 2: GND -> VDD
- D3 pad 1: Net-(D3-DOUT) -> Net-(D3-K)
- D3 pad 2: GND -> Net-(D3-A)
- D4 pad 1: Net-(D4-DOUT) -> VDD
- D4 pad 2: GND -> Net-(D4-A)
- D5 pad 1: Net-(D5-DOUT) -> Net-(D4-A)
- D5 pad 2: GND -> +5V
- D6 pad 1: Net-(D6-DOUT) -> GND
- D6 pad 2: GND -> Net-(D6-A)
- D7 pad 1: Net-(D7-DOUT) -> GND
- D7 pad 2: GND -> Net-(D7-K)
- D7 pad 3: Net-(D6-DOUT) -> GND
- D8 pad 1: Net-(D8-DOUT) -> VCC
- D8 pad 2: GND -> +3.3V
- D9 pad 1: Net-(D10-DIN) -> VDD
Other:
- board outline added: 100 x 100 mm

Commit message: raspi基板回路図
Parts:
- removed C10, C7: 0.1uF, Capacitor_SMD:C_0402_1005Metric
- removed C11, C15, C16: C_snub, Capacitor_SMD:C_0603_1608Metric
- removed C12, C8, C9: 10uF, Capacitor_SMD:C_0805_2012Metric
- removed C13: 470uF, Capacitor_THT:CP_Radial_D10.0mm_P2.50mm_P5.00mm
- removed C14: 100pF, Capacitor_SMD:C_0603_1608Metric
- removed C17, C18, C19, C20: 470uF, Capacitor_SMD:C_Elec_8x10.2
- removed D10, D2, D3: SS2040FL, Diode_SMD:D_SOD-123
- removed D4, D5, D8: 1N5819WS, Diode_SMD:D_SOD-323_HandSoldering
- removed D7: CBD20150VCT, Package_TO_SOT_THT:TO-220-3_Horizontal_TabDown
- removed J3: Conn_01x02_Female, Connector_AMASS:AMASS_XT30PW-F_1x02_P2.50mm_Horizontal
- removed Q8, Q9: MTP4835I3, Package_TO_SOT_SMD:TO-252-2
- removed R27, R39, R47, R48: 10k, Resistor_SMD:R_0402_1005Metric
- removed R28: 10, Resistor_SMD:R_0603_1608Metric
- removed R30, R33, R34: R_snub, Resistor_SMD:R_0603_1608Metric
- removed R32, R46: 1k, Resistor_SMD:R_0402_1005Metric
- removed R35: 5.1k, Resistor_SMD:R_0402_1005Metric
- removed R36: 5.1k, Resistor_SMD:R_0603_1608Metric
- removed R37: 7.5k, Resistor_SMD:R_0603_1608Metric
- removed R38: 1.5k, Resistor_SMD:R_0603_1608Metric
- removed R40: 2k, Resistor_SMD:R_0603_1608Metric
- removed U7: MC34063AD, Package_SO:SOIC-8_3.9x4.9mm_P1.27mm
- removed U8: AZ1084CD-3.3, Package_TO_SOT_SMD:TO-252-2
- added C26: 0.1uF, Capacitor_SMD:C_0402_1005Metric, B.Cu at (-55.8, -62.2)
- added C27: 0.1uF, Capacitor_SMD:C_0402_1005Metric, B.Cu at (-55.8, -60.2)
- added C28: 0.1uF, Capacitor_SMD:C_0402_1005Metric, B.Cu at (-55.8, -58.2)
- added C29: 1uF, Capacitor_SMD:C_0402_1005Metric, B.Cu at (-55.8, -56.3)
- added C30: 1uF, Capacitor_SMD:C_0402_1005Metric, B.Cu at (-55.8, -54.3)
- added C31: 10uF, Capacitor_SMD:C_0805_2012Metric, B.Cu at (-36.0, -34.0)
- added C32: 330uF, Capacitor_THT:CP_Radial_D10.0mm_P2.50mm_P5.00mm, B.Cu at (-38.5, -41.3)
- added C33: C_snub, Capacitor_SMD:C_0603_1608Metric, B.Cu at (-47.9, -48.8)
- added C34: C_snub, Capacitor_SMD:C_0603_1608Metric, B.Cu at (-47.9, -46.2)
- added D11: SS2040FL, Diode_SMD:D_SOD-123, B.Cu at (-55.7, -48.3)
- added D12: SS2040FL, Diode_SMD:D_SOD-123, B.Cu at (-55.7, -45.0)
- added D13: 1N5819WS, Diode_SMD:D_SOD-323_HandSoldering, B.Cu at (-55.4, -38.5)
- added D14: SS2040FL, Diode_SMD:D_SOD-123, B.Cu at (-55.7, -41.6)
- added D15: 1N5819WS, Diode_SMD:D_SOD-323_HandSoldering, B.Cu at (-55.4, -35.5)
- added JP1: Jumper_2_Bridged, Jumper:SolderJumper-2_P1.3mm_Bridged_RoundedPad1.0x1.5mm, B.Cu at (0.35, -53.5)
- added Q15: MTP4835I3, Package_TO_SOT_SMD:TO-252-2, B.Cu at (-40.6, -59.1)
- added R49: 10k, Resistor_SMD:R_0402_1005Metric, B.Cu at (-51.3, -49.0)
- added R50: 10k, Resistor_SMD:R_0402_1005Metric, B.Cu at (-51.3, -47.0)
- added R51: 1k, Resistor_SMD:R_0402_1005Metric, B.Cu at (-51.3, -45.0)
- added R52: 10k, Resistor_SMD:R_0402_1005Metric, B.Cu at (-51.3, -43.0)
- added R53: 10k, Resistor_SMD:R_0402_1005Metric, B.Cu at (-51.3, -41.0)
- added R54: R_snub, Resistor_SMD:R_0603_1608Metric, B.Cu at (-47.9, -43.7)
- added R55: 5.1k, Resistor_SMD:R_0402_1005Metric, B.Cu at (-51.3, -39.1)
- added R56: 5.1k, Resistor_SMD:R_0603_1608Metric, B.Cu at (-47.9, -41.2)
- added R57: 7.5k, Resistor_SMD:R_0603_1608Metric, B.Cu at (-47.9, -38.7)
- added R58: 1.5k, Resistor_SMD:R_0603_1608Metric, B.Cu at (-47.9, -36.2)
- added R59: 10k, Resistor_SMD:R_0402_1005Metric, B.Cu at (-51.3, -37.1)
- added R60: 2k, Resistor_SMD:R_0603_1608Metric, B.Cu at (-47.9, -33.7)
- added U10: RT9624A, Package_SO:SOP-8_3.9x4.9mm_P1.27mm, B.Cu at (-50.1, -59.8)
- added U11: RT8250, Package_SO:SOP-8_3.9x4.9mm_P1.27mm, B.Cu at (-50.1, -53.2)
- added U12: AZ1084CD-12, Package_TO_SOT_SMD:TO-252-2, B.Cu at (-40.6, -51.1)
- C1, C2, C21, C22, C25, C3, C4, C5, C6, D1, D6, D9, Q1, Q10, Q11, Q2, Q3, Q4, Q5, Q6, R1, R10, R11, R12, R13, R14, R15, R16, R17, R18, R19, R2, R20, R21, R22, R23, R24, R25, R29, R3, R31, R4, R41, R42, R44, R5, R6, R7, R8, R9, TP1, TP2, TP3, TP4, TP5, U1, U2, U3, U4, U5, U6, U9: moved to B.Cu
- C23: value 1uF -> 0.1uF; moved to B.Cu
- C24: value 1uF -> 10uF; footprint Capacitor_SMD:C_0402_1005Metric -> Capacitor_SMD:C_0805_2012Metric; moved to B.Cu
- J1: value Conn_01x07_MountingPin -> Conn_01x08_MountingPin; footprint Connector_Molex:Molex_PicoBlade_53261-0771_1x07-1MP_P1.25mm_Horizontal -> Connector_Molex:Molex_PicoBlade_53261-0871_1x08-1MP_P1.25mm_Horizontal; moved to B.Cu
- J2: footprint Connector_AMASS:AMASS_XT30PW-M_1x02_P2.50mm_Horizontal -> Connector_Molex:Molex_SPOX_5268-02A_1x02_P2.50mm_Horizontal; moved to B.Cu
- Q12: value BSS138 -> 2N7002; moved to B.Cu
- Q7: value 2SC3265 -> 2N7002; moved to B.Cu
- R26: value 510 -> 10k; moved to B.Cu
- R43: value 33k -> R_snub; moved to B.Cu
- R45: value 10k -> 1k; footprint Resistor_SMD:R_0603_1608Metric -> Resistor_SMD:R_0402_1005Metric; moved to B.Cu
- moved R42 188.4 mm to (-46.3, -84.8), turned to 90 degrees
- moved R31 186.2 mm to (-46.3, -81.9), turned to 90 degrees
- moved R41 184.8 mm to (-44.3, -84.8), turned to 90 degrees
- moved R29 182.6 mm to (-44.3, -81.9), turned to 90 degrees
- moved TP5 176.5 mm to (-42.4, -78.4), turned to 90 degrees
- moved R44 176.1 mm to (-38.3, -87.7), turned to 90 degrees
- moved R26 175.3 mm to (-40.3, -81.9), turned to 90 degrees
- moved R25 171.7 mm to (-38.3, -81.9), turned to 90 degrees
- moved TP4 169.1 mm to (-38.3, -78.4), turned to 90 degrees
- moved U9 166.1 mm to (-34.1, -84.6), turned to 90 degrees
- moved TP3 161.7 mm to (-34.3, -78.4), turned to 90 degrees
- moved C25 161.3 mm to (-71.2, -32.3), turned to 90 degrees
- moved C24 157.6 mm to (-69.2, -32.4), turned to 90 degrees
- moved TP2 154.4 mm to (-30.2, -78.4), turned to 90 degrees
- moved C23 154.0 mm to (-67.2, -32.3), turned to 90 degrees
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Connections:
- net /Power/12VBAT renamed +BATT
- net 主電源スイッチ renamed /Power/PowerSW
- C23 pad 1: VCC -> GND
- C23 pad 2: GND -> VDD
- C24 pad 1: +3.3V -> VDD
- Q7 pad 1: Net-(D3-K) -> /Panel_PWRCtrl
- Q7 pad 2: Net-(D3-A) -> GNDD
- Q7 pad 3: VDD -> /DCDC_OUTCtrl
- R26 pad 1: VDD -> /Panel_PWRCtrl
- R26 pad 2: Net-(D3-K) -> GNDD
- R31 pad 2: +3.3V -> +5V
- R43 pad 1: VDD -> Net-(C34-Pad2)
- R43 pad 2: V_Measure -> VDD
- R45 pad 1: V_Measure -> VDD
- U9 pad 2: V_Surv. -> /Power/V_Surv.
- U9 pad 6: SHDN_overV -> /DCDC_OUTCtrl
Other:
- outline, holes or cut-outs redrawn

Commit message: 発注第3弾
DCDC、MD追加
Parts:
- removed D11, D12, D14: SS2040FL, Diode_SMD:D_SOD-123
- removed D13, D15, D9: 1N5819WS, Diode_SMD:D_SOD-323_HandSoldering
- removed Q12: 2N7002, Package_TO_SOT_SMD:SOT-23
- removed Q15: MTP4835I3, Package_TO_SOT_SMD:TO-252-2
- removed R13, R14: 2.2k, Resistor_SMD:R_0402_1005Metric
- removed R52, R59: 10k, Resistor_SMD:R_0402_1005Metric
- removed R54: R_snub, Resistor_SMD:R_0603_1608Metric
- removed R55: 5.1k, Resistor_SMD:R_0402_1005Metric
- removed R56: 5.1k, Resistor_SMD:R_0603_1608Metric
- removed R57: 7.5k, Resistor_SMD:R_0603_1608Metric
- removed R58: 1.5k, Resistor_SMD:R_0603_1608Metric
- removed R60: 2k, Resistor_SMD:R_0603_1608Metric
- removed R7, R8: 20k, Resistor_SMD:R_0402_1005Metric
- removed TP2, TP3, TP4, TP5: TestPoint, TestPoint:TestPoint_THTPad_D2.0mm_Drill1.0mm
- removed U12: AZ1084CD-12, Package_TO_SOT_SMD:TO-252-2
- added C10: 1uF, Capacitor_SMD:C_0402_1005Metric, B.Cu at (22.2, -12.3)
- added C11: 1uF_50V, Capacitor_SMD:C_0603_1608Metric, B.Cu at (13.7, -4.81)
- added C12: 10uF_50V, Capacitor_SMD:C_0805_2012Metric, B.Cu at (22.5, 7.48)
- added C13: 10uF_50V, Capacitor_SMD:C_0805_2012Metric, B.Cu at (23.7, 8.75)
- added C14: 10uF_50V, Capacitor_SMD:C_0805_2012Metric, B.Cu at (25.0, 10.0)
- added C15: 10uF_50V, Capacitor_SMD:C_0805_2012Metric, B.Cu at (26.4, 12.4)
- added C16: 1nF, Capacitor_SMD:C_0603_1608Metric, B.Cu at (25.5, 13.5)
- added C17: 1500pF, Capacitor_SMD:C_0603_1608Metric, B.Cu at (14.0, -15.0)
- added C18: 47pF, Capacitor_SMD:C_0603_1608Metric, B.Cu at (10.5, -10.0)
- added C19: 1nF, Capacitor_SMD:C_0603_1608Metric, B.Cu at (24.4, -17.8)
- added C20: 2700pF, Capacitor_SMD:C_0603_1608Metric, B.Cu at (9.26, -10.0)
- added C7: 1uF_50V, Capacitor_SMD:C_0603_1608Metric, B.Cu at (24.6, -13.5)
- added C8: 1uF, Capacitor_SMD:C_0402_1005Metric, B.Cu at (33.6, -2.23)
- added C9: 0.1uF_50V, Capacitor_SMD:C_0402_1005Metric, B.Cu at (24.1, -12.3)
- added D2: 1N5819WS, TomoshibiLibrary:Diode_SOD-323, B.Cu at (23.8, -16.1)
- added D3: 1N5819WS, TomoshibiLibrary:Diode_SOD-323, B.Cu at (29.2, -14.1)
- added D4: SS2040FL, Diode_SMD:D_SOD-123, B.Cu at (27.6, 22.7)
- added D5: SS2040FL, Diode_SMD:D_SOD-123, B.Cu at (19.3, 11.6)
- added D7: 1N5819WS, TomoshibiLibrary:Diode_SOD-323, B.Cu at (6.01, 17.3)
- added D8: Green, LED_SMD:LED_0603_1608Metric_Pad1.05x0.95mm_HandSolder, B.Cu at (16.0, -37.1)
- added FB1: FerriteBead, Inductor_SMD:L_0603_1608Metric, B.Cu at (27.1, -17.1)
- added H1: MountingHole_Pad, MountingHole:MountingHole_2.2mm_M2_Pad, B.Cu at (6.50, -3.75)
- added H10: MountingHole_Pad, MountingHole:MountingHole_3.7mm_Pad_Via, B.Cu at (13.5, -42.9)
- added H11: MountingHole_Pad, MountingHole:MountingHole_3.7mm_Pad_Via, B.Cu at (20.8, -39.9)
- added H12: MountingHole_Pad, MountingHole:MountingHole_3.7mm_Pad_Via, B.Cu at (-20.8, -39.9)
- added H13: MountingHole_Pad, MountingHole:MountingHole_3.7mm_Pad_Via, B.Cu at (-13.5, -42.9)
- added H14: MountingHole_Pad, MountingHole:MountingHole_3.7mm_Pad_Via, B.Cu at (-42.9, -13.5)
- added H15: MountingHole_Pad, MountingHole:MountingHole_3.7mm_Pad_Via, B.Cu at (-39.9, -20.8)
- added H16: MountingHole_Pad, MountingHole:MountingHole_3.7mm_Pad_Via, B.Cu at (-39.9, 20.8)
- added H17: MountingHole_Pad, MountingHole:MountingHole_3.7mm_Pad_Via, B.Cu at (-42.9, 13.5)
- added H18: MountingHole_Pad, MountingHole:MountingHole_3.7mm_Pad_Via, B.Cu at (-13.5, 42.9)
- added H19: MountingHole_Pad, MountingHole:MountingHole_3.7mm_Pad_Via, B.Cu at (-20.8, 39.9)
- added H2: MountingHole_Pad, MountingHole:MountingHole_2.2mm_M2_Pad, B.Cu at (0.00, -7.50)
- added H20: MountingHole_Pad, MountingHole:MountingHole_3.7mm_Pad_Via, B.Cu at (20.8, 39.9)
- added H21: MountingHole_Pad, MountingHole:MountingHole_3.7mm_Pad_Via, B.Cu at (13.5, 42.9)
- added H22: MountingHole_Pad, MountingHole:MountingHole_3.7mm_Pad_Via, B.Cu at (42.9, 13.5)
- added H23: MountingHole_Pad, MountingHole:MountingHole_3.7mm_Pad_Via, B.Cu at (39.9, 20.8)
- added H3: MountingHole_Pad, MountingHole:MountingHole_2.2mm_M2_Pad, B.Cu at (-6.50, -3.75)
- added H4: MountingHole_Pad, MountingHole:MountingHole_2.2mm_M2_Pad, B.Cu at (-6.50, 3.75)
- added H5: MountingHole_Pad, MountingHole:MountingHole_2.2mm_M2_Pad, B.Cu at (0.00, 7.50)
- added H6: MountingHole_Pad, MountingHole:MountingHole_2.2mm_M2_Pad, B.Cu at (6.50, 3.75)
- added H7: MountingHole_Pad, TestPoint:TestPoint_Pad_D1.5mm, B.Cu at (7.84, -20.0)
- added H8: MountingHole_Pad, MountingHole:MountingHole_3.7mm_Pad_Via, B.Cu at (39.9, -20.8)
- added H9: MountingHole_Pad, MountingHole:MountingHole_3.7mm_Pad_Via, B.Cu at (42.9, -13.5)
- added JP2: Jumper_2_Bridged, Jumper:SolderJumper-2_P1.3mm_Bridged_RoundedPad1.0x1.5mm, B.Cu at (-7.92, 25.5)
- added JP3: Jumper_2_Bridged, Jumper:SolderJumper-2_P1.3mm_Bridged_RoundedPad1.0x1.5mm, B.Cu at (-11.8, 21.6)
- added JP4: Jumper_2_Bridged, Jumper:SolderJumper-2_P1.3mm_Bridged_RoundedPad1.0x1.5mm, B.Cu at (-15.7, 17.7)
- added JP5: Jumper_2_Bridged, Jumper:SolderJumper-2_P1.3mm_Bridged_RoundedPad1.0x1.5mm, B.Cu at (-19.6, 13.8)
- added JP6: Jumper_2_Bridged, Jumper:SolderJumper-2_P1.3mm_Bridged_RoundedPad1.0x1.5mm, B.Cu at (-23.2, 10.2)
- added L1: 2.2uH, TomoshibiLibrary:Inductor_ETQ-P4M_KVK, B.Cu at (13.8, 22.3)
- added Q8: TPH11006NL, TomoshibiLibrary:Package_SOP-Advance, B.Cu at (25.1, 19.5)
- added Q9: TPH11006NL, TomoshibiLibrary:Package_SOP-Advance, B.Cu at (21.0, 15.5)
- added R27: 20k, Resistor_SMD:R_0402_1005Metric, B.Cu at (29.7, -15.6)
- added R28: 10k, Resistor_SMD:R_0402_1005Metric, B.Cu at (16.5, -7.00)
- added R30: 1k, Resistor_SMD:R_0402_1005Metric, B.Cu at (16.7, -16.4)
- added R32: 510, Resistor_SMD:R_0402_1005Metric, B.Cu at (11.5, -17.0)
- added R34: 12k, Resistor_SMD:R_0603_1608Metric, B.Cu at (10.3, -7.95)
- added R35: 2.7k, Resistor_SMD:R_0603_1608Metric, B.Cu at (10.6, -12.4)
- added R36: 1k, Resistor_SMD:R_0402_1005Metric, B.Cu at (16.3, -14.9)
- added R38: R_snub, Resistor_SMD:R_0603_1608Metric, B.Cu at (16.3, 17.6)
- added R39: 5.1k, Resistor_SMD:R_0402_1005Metric, B.Cu at (13.3, -3.11)
- added R40: 3.3k, Resistor_SMD:R_0402_1005Metric, B.Cu at (14.2, -3.11)
- added R46: 7.5k, Resistor_SMD:R_0603_1608Metric, B.Cu at (-3.32, 2.49)
- added R47: 2k, Resistor_SMD:R_0603_1608Metric, B.Cu at (-4.72, 0.07)
- added R48: 1k, Resistor_SMD:R_0402_1005Metric, B.Cu at (7.11, 16.3)
- added SW1: SW_SPDT_White, TomoshibiLibrary:SW_Slide_SPDT_IS-1235-G, B.Cu at (44.6, 0.49)
- added U7: NJM78L12S_SOT89, Package_TO_SOT_SMD:SOT-89-3, B.Cu at (23.2, -9.10)
- added U8: UC3843_SOIC8, Package_SO:SOIC-8_3.9x4.9mm_P1.27mm, B.Cu at (16.0, -11.7)
- C22, C27: value 0.1uF -> 1nF; footprint Capacitor_SMD:C_0402_1005Metric -> Capacitor_SMD:C_0603_1608Metric
- C23: value 0.1uF -> C_snub; footprint Capacitor_SMD:C_0402_1005Metric -> Capacitor_SMD:C_0603_1608Metric
- C24: value 10uF -> 0.1uF; footprint Capacitor_SMD:C_0805_2012Metric -> Capacitor_SMD:C_0402_1005Metric
- C25: value 4700pF -> 1nF
- C26: value 0.1uF -> 330uF; footprint Capacitor_SMD:C_0402_1005Metric -> Capacitor_Tantalum_SMD:CP_EIA-7343-20_Kemet-V
- C29: value 1uF -> 1uF_50V; footprint Capacitor_SMD:C_0402_1005Metric -> Capacitor_SMD:C_0603_1608Metric
- C30: value 1uF -> 0.1uF
- C31: value 10uF -> 100uF; footprint Capacitor_SMD:C_0805_2012Metric -> TomoshibiLibrary:Capacitor_Alum_Radial_5.0x11.0mm_Horizontal
- C32: value 330uF -> 100uF; footprint Capacitor_THT:CP_Radial_D10.0mm_P2.50mm_P5.00mm -> TomoshibiLibrary:Capacitor_Alum_Radial_5.0x11.0mm_Horizontal
- C33: value C_snub -> 4700pF
- C34: value C_snub -> 0.1uF; footprint Capacitor_SMD:C_0603_1608Metric -> Capacitor_SMD:C_0402_1005Metric
- D1, D6: value Green -> 1N5819WS; footprint LED_SMD:LED_0603_1608Metric_Pad1.05x0.95mm_HandSolder -> TomoshibiLibrary:Diode_SOD-323
- J2: value Conn_01x02_Male -> Conn_01x02_Pin
- Q1, Q3: value S8550 -> SSM6J808R; footprint Package_TO_SOT_SMD:SOT-23 -> TomoshibiLibrary:Package_TSOP6F
- Q11: value MTP4835I3 -> 2N7002; footprint Package_TO_SOT_SMD:TO-252-2 -> Package_TO_SOT_SMD:SC-59
- Q2: value S8550 -> 2N7002; footprint Package_TO_SOT_SMD:SOT-23 -> Package_TO_SOT_SMD:SC-59
- Q4, Q5, Q6: value S8550 -> SS8550; footprint Package_TO_SOT_SMD:SOT-23 -> Package_TO_SOT_SMD:SC-59
- Q7: value 2N7002 -> SS8050; footprint Package_TO_SOT_SMD:SOT-23 -> Package_TO_SOT_SMD:SC-59
- R1, R2: value 2.2k -> Rg; footprint Resistor_SMD:R_0402_1005Metric -> Resistor_SMD:R_0603_1608Metric
- R16, R17, R18, R4, R5, R6: value 7.5k -> 2.2k; footprint Resistor_SMD:R_0603_1608Metric -> Resistor_SMD:R_0402_1005Metric
- R19, R21: value 20k -> 10k
- R22, R23, R24: value 2.2k -> 10k
- R25: value 1k -> 10k
- R29: value 10k -> 510
- R31: value 1k -> 10M; footprint Resistor_SMD:R_0402_1005Metric -> Resistor_SMD:R_0603_1608Metric
- R41: value 100k -> 20k
- R43: value R_snub -> 16k
- R44: value 10k -> 16k; footprint Resistor_SMD:R_0402_1005Metric -> Resistor_SMD:R_0603_1608Metric
- R45: value 1k -> 620; footprint Resistor_SMD:R_0402_1005Metric -> Resistor_SMD:R_0603_1608Metric
- R9: value 20k -> 2.2k
- U1, U2, U3, U4, U5, U6: value MAX3485 -> MAX485E
- U10: value RT9624A -> NJU77701; footprint Package_SO:SOP-8_3.9x4.9mm_P1.27mm -> Package_TO_SOT_SMD:SOT-23-5
- U11: value RT8250 -> M51957B
- U9: value M51957B -> Driver_FETGate_RT9624A
- moved R25 109.8 mm to (34.6, 0.14)
- moved R42 102.2 mm to (15.1, -3.11), turned to -90 degrees
- moved R41 102.2 mm to (16.5, -2.69), turned to 0 degrees
- moved C26 101.7 mm to (14.9, 11.0), turned to 45 degrees
- moved U9 99.1 mm to (15.1, 1.41), turned to -90 degrees
- moved C25 98.8 mm to (16.3, 13.7), turned to 45 degrees
- moved C23 96.3 mm to (16.5, 15.2), turned to -135 degrees
- moved C28 94.2 mm to (18.3, -0.07), turned to 90 degrees
- moved C22 93.5 mm to (27.3, -19.0), turned to 135 degrees
- moved R26 92.8 mm to (22.2, -13.3), turned to 180 degrees
- moved R31 92.4 mm to (11.8, -10.0)
- moved C24 91.8 mm to (20.2, -11.6)
- moved R44 90.4 mm to (7.99, -10.0)
- moved C29 88.2 mm to (11.7, 0.57), turned to -90 degrees
- moved J1 87.1 mm to (-33.2, 33.2), turned to 135 degrees
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Connections:
- C1 pad 1: +3.3V -> +5V
- C1 pad 2: GNDD -> GND
- C2 pad 1: +3.3V -> +5V
- C2 pad 2: GNDD -> GND
- C21 pad 1: /Power/S-S -> Net-(Q7-C)
- C21 pad 2: Net-(Q11-G) -> GND
- C22 pad 1: GND -> Net-(D1-K)
- C22 pad 2: VDD -> GND
- C23 pad 2: VDD -> Net-(C23-Pad2)
- C24 pad 1: VDD -> +12V
- C25 pad 1: GND -> Net-(D6-A)
- C25 pad 2: Net-(U9-Cdelay) -> GND
- C26 pad 1: Net-(U11-BST) -> Net-(D6-A)
- C26 pad 2: Net-(U11-SW) -> GND
- C27 pad 1: Net-(U10-VB) -> Net-(C27-Pad1)
- C27 pad 2: Net-(D11-A) -> Net-(D6-A)
- C29 pad 1: VCC -> Net-(U9-BT)
- C29 pad 2: GND -> /Power/SW
- C3 pad 1: +3.3V -> +5V
- C3 pad 2: GNDD -> GND
- C30 pad 1: +12V -> GND
- C30 pad 2: GND -> +5V
- C31 pad 1: Net-(D15-K) -> VDD
- C32 pad 1: Net-(D15-K) -> VCC
- C33 pad 2: Net-(C33-Pad2) -> Net-(U11-Cdelay)
- C34 pad 2: Net-(C34-Pad2) -> +12V
- C4 pad 1: +3.3V -> +5V
- C4 pad 2: GNDD -> GND
- C5 pad 1: +3.3V -> +5V
- C5 pad 2: GNDD -> GND
- C6 pad 1: +3.3V -> +5V
- C6 pad 2: GNDD -> GND
- D1 pad 1: GND -> Net-(D1-K)
- D1 pad 2: Net-(D1-A) -> VDD
- D6 pad 1: GND -> VDD
- J1 pad 1: GNDD -> GND
- J1 pad MP: GNDD -> GND
- JP1 pad 1: unconnected-(JP1-A-Pad1) -> Net-(JP1-A)
- JP1 pad 2: unconnected-(JP1-B-Pad2) -> Net-(JP1-B)
- Q1 pad 1: Net-(Q1-B) -> +BATT
- Q1 pad 2: +3.3V -> +BATT
- Q1 pad 3: Net-(Q1-C) -> Net-(Q1-G)
- Q10 pad 1: GND -> /Power/SHDN
- Q10 pad 2: +BATT -> +5V
- Q10 pad 3: /Power/S-S -> Net-(D6-A)
- Q11 pad 1: Net-(Q11-G) -> /Panel_PWRCtrl
- Q11 pad 2: VDD -> Net-(Q11-S)
- Q11 pad 3: /Power/S-S -> /Power/SHDN
- Q2 pad 1: Net-(Q2-B) -> /Power/PowerSW
- Q2 pad 2: +3.3V -> GND
- Q2 pad 3: Net-(Q2-C) -> Net-(Q2-D)
- Q3 pad 1: Net-(Q3-B) -> VDD
- Q3 pad 2: +3.3V -> VDD
- Q3 pad 3: Net-(Q3-C) -> Net-(Q3-G)
- Q4 pad 2: +3.3V -> Net-(Q4-E)
- Q4 pad 3: Net-(Q4-C) -> GND
- Q5 pad 2: +3.3V -> Net-(Q5-E)
- Q5 pad 3: Net-(Q5-C) -> Net-(Q5-B)
- Q6 pad 1: Net-(Q6-B) -> Net-(Q5-B)
- Q6 pad 2: +3.3V -> Net-(Q6-E)
- Q6 pad 3: Net-(Q6-C) -> /Power/CLK
- Q7 pad 1: /Panel_PWRCtrl -> /Power/CLK
- Q7 pad 2: GNDD -> Net-(Q7-E)
- Q7 pad 3: /DCDC_OUTCtrl -> Net-(Q7-C)
- R1 pad 1: +3.3V -> /Power/HG
- R1 pad 2: Net-(U1-B) -> Net-(U9-UG)
- R10 pad 1: Net-(U1-B) -> Net-(U3-B)
- R10 pad 2: GNDD -> GND
- R11 pad 1: Net-(U2-B) -> +5V
- R11 pad 2: GNDD -> Net-(U4-B)
- R12 pad 1: Net-(U3-B) -> Net-(U4-B)
- R12 pad 2: GNDD -> GND
- R15 pad 1: +3.3V -> +5V
- R15 pad 2: Net-(U6-B) -> Net-(U5-B)
- R16 pad 1: Net-(Q4-B) -> Net-(U5-B)
- R16 pad 2: /TangPrimerTXx_Panel1RX -> GND
- R17 pad 1: Net-(Q5-B) -> +5V
- R17 pad 2: /TangPrimerTXx_Panel3RX -> Net-(U6-B)
- R18 pad 1: Net-(Q6-B) -> Net-(U6-B)
- R18 pad 2: /TangPrimerTXx_Panel5RX -> GND
- R19 pad 1: Net-(Q4-C) -> Net-(Q1-G)
- R19 pad 2: GNDD -> GND
- R2 pad 1: +3.3V -> /Power/LG
- R2 pad 2: Net-(U2-B) -> Net-(U9-LG)
- R20 pad 1: Net-(Q5-C) -> VCC
- R20 pad 2: GNDD -> GND
- R21 pad 1: Net-(Q6-C) -> /Power/S-S
- R21 pad 2: GNDD -> Net-(Q1-G)
- R22 pad 1: Net-(U4-B) -> Net-(SW1-A)
- R22 pad 2: GNDD -> /Power/PowerSW
- R23 pad 1: Net-(U5-B) -> /Power/S-S
- R23 pad 2: GNDD -> Net-(Q3-G)
- R24 pad 1: Net-(U6-B) -> Net-(Q3-G)
- R24 pad 2: GNDD -> Net-(Q2-D)
- R25 pad 1: Net-(D1-A) -> /Power/PowerSW
- R25 pad 2: VCC -> GND
- R26 pad 1: /Panel_PWRCtrl -> GND
- R26 pad 2: GNDD -> +12V
- R29 pad 1: /Power/PowerSW -> Net-(Q5-E)
- R29 pad 2: GND -> Net-(Q7-C)
- R3 pad 1: +3.3V -> +5V
- R3 pad 2: Net-(U3-B) -> Net-(U1-B)
- R31 pad 1: Net-(D6-A) -> Net-(Q4-E)
- R31 pad 2: +5V -> /Power/FB
- R4 pad 1: Net-(Q1-B) -> Net-(U1-B)
- R4 pad 2: /TangPrimerTXx_Panel0RX -> GND
- R41 pad 1: /Power/S-S -> Net-(U9-EN)
- R41 pad 2: Net-(Q11-G) -> +12V
- R42 pad 1: /Power/S-S -> GND
- R42 pad 2: GND -> Net-(U9-EN)
- R43 pad 1: Net-(C34-Pad2) -> /Power/FB
- R43 pad 2: VDD -> Net-(D6-A)
- R44 pad 1: Net-(Q11-G) -> GND
- R44 pad 2: Net-(Q12-D) -> /Power/FB
- R45 pad 1: VDD -> /Power/FB
- R45 pad 2: GND -> Net-(C27-Pad1)
- R49 pad 1: Net-(U10-IN) -> Net-(D6-A)
- R49 pad 2: Net-(U11-SW) -> /Power/SHDN
- R5 pad 1: Net-(Q2-B) -> +5V
- R5 pad 2: /TangPrimerTXx_Panel2RX -> Net-(U2-B)
- R50 pad 1: GND -> +5V
- R50 pad 2: Net-(U10-IN) -> GND
- R51 pad 1: VDD -> Net-(D8-A)
- R51 pad 2: GND -> +5V
- R53 pad 1: GND -> /Panel_PWRCtrl
- R53 pad 2: +12V -> GND
- R6 pad 1: Net-(Q3-B) -> Net-(U2-B)
- R6 pad 2: /TangPrimerTXx_Panel4RX -> GND
- R9 pad 1: Net-(Q3-C) -> +5V
- R9 pad 2: GNDD -> Net-(U3-B)
- TP1 pad 1: VDD -> GND
- U1 pad 1: /TangPrimerRXx_Panel0TX -> Net-(JP1-B)
- U1 pad 2: Net-(Q1-C) -> GND
- U1 pad 3: Net-(Q1-C) -> GND
- U1 pad 4: /TangPrimerTXx_Panel0RX -> GND
- U1 pad 5: GNDD -> GND
- U1 pad 8: +3.3V -> +5V
- U10 pad 1: +12V -> Net-(U10--)
- U10 pad 2: Net-(U10-IN) -> GND
- U10 pad 3: unconnected-(U10-~{SD}-Pad3) -> /Power/CLK
- U10 pad 4: GND -> Net-(U10--)
- U10 pad 5: Net-(Q14-G) -> +5V
- U11 pad 1: Net-(U11-BST) -> unconnected-(U11-NC-Pad1)
- U11 pad 2: +12V -> /Power/V_Surv
- U11 pad 3: Net-(U11-SW) -> unconnected-(U11-NC-Pad3)
- U11 pad 5: /Power/fb -> Net-(U11-Cdelay)
- U11 pad 6: unconnected-(U11-COMP-Pad6) -> Net-(Q11-S)
- U11 pad 7: unconnected-(U11-EN-Pad7) -> +12V
- U2 pad 1: /TangPrimerRXx_Panel2TX -> Net-(JP2-B)
- U2 pad 2: Net-(Q2-C) -> GND
- U2 pad 3: Net-(Q2-C) -> GND
- U2 pad 4: /TangPrimerTXx_Panel2RX -> GND
- U2 pad 5: GNDD -> GND
- U2 pad 6: /RS485/RS485_Panel2 -> /RS485/RS485_Panel1
- U2 pad 8: +3.3V -> +5V
- U3 pad 1: /TangPrimerRXx_Panel4TX -> Net-(JP3-B)
- U3 pad 2: Net-(Q3-C) -> GND
- U3 pad 3: Net-(Q3-C) -> GND
- U3 pad 4: /TangPrimerTXx_Panel4RX -> GND
- U3 pad 5: GNDD -> GND
- U3 pad 6: /RS485/RS485_Panel4 -> /RS485/RS485_Panel2
- U3 pad 8: +3.3V -> +5V
- U4 pad 1: /TangPrimerRXx_Panel1TX -> Net-(JP4-B)
- U4 pad 2: Net-(Q4-C) -> GND
- U4 pad 3: Net-(Q4-C) -> GND
- U4 pad 4: /TangPrimerTXx_Panel1RX -> GND
- U4 pad 5: GNDD -> GND
- U4 pad 6: /RS485/RS485_Panel1 -> /RS485/RS485_Panel3
- U4 pad 8: +3.3V -> +5V
- U5 pad 1: /TangPrimerRXx_Panel3TX -> Net-(JP5-B)
- U5 pad 2: Net-(Q5-C) -> GND
- U5 pad 3: Net-(Q5-C) -> GND
- U5 pad 4: /TangPrimerTXx_Panel3RX -> GND
- U5 pad 5: GNDD -> GND
- U5 pad 6: /RS485/RS485_Panel3 -> /RS485/RS485_Panel4
- U5 pad 8: +3.3V -> +5V
- U6 pad 1: /TangPrimerRXx_Panel5TX -> Net-(JP6-B)
- U6 pad 2: Net-(Q6-C) -> GND
- U6 pad 3: Net-(Q6-C) -> GND
- U6 pad 4: /TangPrimerTXx_Panel5RX -> GND
- U6 pad 5: GNDD -> GND
- U6 pad 8: +3.3V -> +5V
- U9 pad 1: unconnected-(U9-NC-Pad1) -> Net-(U9-BT)
- U9 pad 2: /Power/V_Surv. -> Net-(U9-PWM)
- U9 pad 3: unconnected-(U9-NC-Pad3) -> Net-(U9-EN)
- U9 pad 4: GND -> +12V
- U9 pad 5: Net-(U9-Cdelay) -> Net-(U9-LG)
- U9 pad 6: /DCDC_OUTCtrl -> GND
- U9 pad 7: VDD -> /Power/SW
- U9 pad 8: unconnected-(U9-NC-Pad8) -> Net-(U9-UG)
Routing:
- net +5V: track 0.00 -> 81.9 mm
- net /Panel_PWRCtrl: track 0.00 -> 76.2 mm, vias 0 -> 2
- net Net-(JP5-A): track 0.00 -> 57.1 mm, vias 0 -> 1
- net Net-(JP6-A): track 0.00 -> 54.1 mm, vias 0 -> 1
- net Net-(D6-A): track 0.00 -> 45.0 mm
- net +12V: track 0.00 -> 43.5 mm, vias 0 -> 2
- net /Power/S-S: track 0.00 -> 40.1 mm, vias 0 -> 1
- net Net-(JP1-A): track 0.00 -> 38.9 mm, vias 0 -> 1
- net Net-(JP2-A): track 0.00 -> 35.6 mm, vias 0 -> 1
- net GND: track 0.00 -> 31.7 mm, vias 0 -> 1031
- net Net-(JP3-A): track 0.00 -> 29.3 mm, vias 0 -> 1
- net /Power/SW: track 0.00 -> 25.2 mm, vias 0 -> 4
- net /RS485/RS485_Panel0: track 0.00 -> 24.3 mm
- net Net-(Q3-G): track 0.00 -> 23.3 mm, vias 0 -> 2
- net Net-(Q7-C): track 0.00 -> 21.3 mm, vias 0 -> 3
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- added copper zone on B.Cu, net +5V
- added copper zone on B.Cu, net +BATT
- added copper zone on B.Cu, net /Power/CLK
- added copper zone on B.Cu, net /Power/S-S
- added copper zone on B.Cu, net /Power/SW
- added copper zone on B.Cu, net GND
- added copper zone on F.Cu, net GND
- added copper zone on B.Cu, net Net-(D1-K)
- added copper zone on B.Cu, net Net-(D6-A)
- added copper zone on B.Cu, net VCC
- added copper zone on B.Cu, net VDD
Other:
- outline, holes or cut-outs redrawn
- board text added: "5V"
- board text added: "A"
- board text added: "B"
- board text added: "C"
- board text added: "D"
- board text added: "Designed by @cat_nekonekone"
- board text added: "E"
- board text added: "F"
- board text added: "GND"
- board text added: "JLCJLCJLCJLC"
- board text added: "PWR"
- board text added: "Tomoshibi"
- board text added: "燈"
