File: circuits/DCDC/DCDC.kicad_sch (KiCad schematic)
At the start: 0 parts

Commit message: 更新
Other:
- added sheet Power (Power.kicad_sch)
- added sheet RS485 (RS485.kicad_sch)
Changed lines of the file:
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@@
 (kicad_sch (version 20230121) (generator eeschema)
   (paper "A4")
+  (wire (pts (xy 213.36 68.58) (xy 215.9 68.58))
+    (stroke (width 0) (type default))
+  )
+  (wire (pts (xy 213.36 55.88) (xy 215.9 55.88))
+    (stroke (width 0) (type default))
+  )
+  (wire (pts (xy 213.36 63.5) (xy 215.9 63.5))
+    (stroke (width 0) (type default))
+  )
+  (wire (pts (xy 213.36 38.1) (xy 215.9 38.1))
+    (stroke (width 0) (type default))
+  )
+  (wire (pts (xy 213.36 76.2) (xy 215.9 76.2))
+    (stroke (width 0) (type default))
+  )
+  (wire (pts (xy 213.36 71.12) (xy 215.9 71.12))
+    (stroke (width 0) (type default))
+  )
+  (wire (pts (xy 213.36 78.74) (xy 215.9 78.74))
+    (stroke (width 0) (type default))
+  )
+  (wire (pts (xy 213.36 60.96) (xy 215.9 60.96))
+    (stroke (width 0) (type default))
+  )
+  (wire (pts (xy 213.36 53.34) (xy 215.9 53.34))
+    (stroke (width 0) (type default))
+  )
+  (wire (pts (xy 213.36 48.26) (xy 215.9 48.26))
+    (stroke (width 0) (type default))
+  )
+  (wire (pts (xy 213.36 40.64) (xy 215.9 40.64))
+    (stroke (width 0) (type default))
+  )
+  (wire (pts (xy 213.36 45.72) (xy 215.9 45.72))
+    (stroke (width 0) (type default))
+  )
+  (label "TangPrimerRXx_Panel1TX" (at 213.36 48.26 180) (fields_autoplaced)
+    (effects (font (size 1.27 1.27) (thickness 0.254) bold italic) (justify right bottom))
+  )
+  (label "TangPrimerRXx_Panel3TX" (at 213.36 63.5 180) (fields_autoplaced)
+    (effects (font (size 1.27 1.27) (thickness 0.254) bold italic) (justify right bottom))
+  )
+  (label "TangPrimerTXx_Panel2RX" (at 213.36 53.34 180) (fields_autoplaced)
+    (effects (font (size 1.27 1.27) (thickness 0.254) bold italic) (justify right bottom))
+  )
+  (label "TangPrimerTXx_Panel5RX" (at 213.36 76.2 180) (fields_autoplaced)
+    (effects (font (size 1.27 1.27) (thickness 0.254) bold italic) (justify right bottom))
+  )
+  (label "TangPrimerTXx_Panel1RX" (at 213.36 45.72 180) (fields_autoplaced)
+    (effects (font (size 1.27 1.27) (thickness 0.254) bold italic) (justify right bottom))
+  )
+  (label "TangPrimerTXx_Panel3RX" (at 213.36 60.96 180) (fields_autoplaced)
+    (effects (font (size 1.27 1.27) (thickness 0.254) bold italic) (justify right bottom))
+  )
+  (label "TangPrimerRXx_Panel0TX" (at 213.36 40.64 180) (fields_autoplaced)
+    (effects (font (size 1.27 1.27) (thickness 0.254) bold italic) (justify right bottom))
+  )
+  (label "TangPrimerRXx_Panel5TX" (at 213.36 78.74 180) (fields_autoplaced)
+    (effects (font (size 1.27 1.27) (thickness 0.254) bold italic) (justify right bottom))
+  )
+  (label "TangPrimerTXx_Panel4RX" (at 213.36 68.58 180) (fields_autoplaced)
+    (effects (font (size 1.27 1.27) (thickness 0.254) bold italic) (justify right bottom))
+  )
+  (label "TangPrimerTXx_Panel0RX" (at 213.36 38.1 180) (fields_autoplaced)
+    (effects (font (size 1.27 1.27) (thickness 0.254) bold italic) (justify right bottom))
+  )
+  (label "TangPrimerRXx_Panel4TX" (at 213.36 71.12 180) (fields_autoplaced)
+    (effects (font (size 1.27 1.27) (thickness 0.254) bold italic) (justify right bottom))
+  )
+  (label "TangPrimerRXx_Panel2TX" (at 213.36 55.88 180) (fields_autoplaced)
+    (effects (font (size 1.27 1.27) (thickness 0.254) bold italic) (justify right bottom))
+  )
+  (sheet (at 215.9 33.02) (size 25.4 50.8) (fields_autoplaced)
+    (stroke (width 0.1524) (type solid))
+    (fill (color 0 0 0 0.0000))
+    (property "Sheetname" "RS485" (at 215.9 32.3084 0)
+      (effects (font (size 1.27 1.27)) (justify left bottom))
+    )
+    (property "Sheetfile" "RS485.kicad_sch" (at 215.9 84.4046 0)
+      (effects (font (size 1.27 1.27)) (justify left top))
+    )
+    (pin "FPGARX_Panel2TX" input (at 215.9 55.88 180)
+      (effects (font (size 1.27 1.27)) (justify left))
+    )
+    (pin "FPGATX_Panel2RX" input (at 215.9 53.34 180)
+      (effects (font (size 1.27 1.27)) (justify left))
+    )
+    (pin "FPGARX_Panel0TX" input (at 215.9 40.64 180)
+      (effects (font (size 1.27 1.27)) (justify left))
+    )
+    (pin "FPGATX_Panel0RX" input (at 215.9 38.1 180)
+      (effects (font (size 1.27 1.27)) (justify left))
+    )
+    (pin "FPGARX_Panel3TX" input (at 215.9 63.5 180)
+      (effects (font (size 1.27 1.27)) (justify left))
+    )
+    (pin "FPGATX_Panel3RX" input (at 215.9 60.96 180)
+      (effects (font (size 1.27 1.27)) (justify left))
+    )
+    (pin "FPGATX_Panel1RX" input (at 215.9 45.72 180)
+      (effects (font (size 1.27 1.27)) (justify left))
+    )
+    (pin "FPGARX_Panel1TX" input (at 215.9 48.26 180)
+      (effects (font (size 1.27 1.27)) (justify left))
+    )
+    (pin "FPGARX_Panel5TX" input (at 215.9 78.74 180)
+      (effects (font (size 1.27 1.27)) (justify left))
+    )
+    (pin "FPGATX_Panel5RX" input (at 215.9 76.2 180)
+      (effects (font (size 1.27 1.27)) (justify left))
+    )
+    (pin "FPGARX_Panel4TX" input (at 215.9 71.12 180)
+      (effects (font (size 1.27 1.27)) (justify left))
+    )
+    (pin "FPGATX_Panel4RX" input (at 215.9 68.58 180)
+      (effects (font (size 1.27 1.27)) (justify left))
+    )
+    (instances
+      (project "DCDC"
+        (path "/ff041c4b-2038-4373-9ca4-fac09ac6c22f" (page "2"))
+      )
+    )
+  )
+  (sheet (at 25.4 25.4) (size 20.32 15.24) (fields_autoplaced)
+    (stroke (width 0.1524) (type solid))
+    (fill (color 0 0 0 0.0000))
+    (property "Sheetname" "Power" (at 25.4 24.6884 0)
+      (effects (font (size 1.27 1.27)) (justify left bottom))
+    )
+    (property "Sheetfile" "Power.kicad_sch" (at 25.4 41.2246 0)
+      (effects (font (size 1.27 1.27)) (justify left top))
+    )
+    (instances
+      (project "DCDC"
+        (path "/ff041c4b-2038-4373-9ca4-fac09ac6c22f" (page "3"))
+      )
+    )
+  )
   (sheet_instances
     (path "/" (page "1"))

Commit message: raspi基板回路図
Parts:
- added Q7: 2N7002, Package_TO_SOT_SMD:SOT-23, symbol Transistor_FET:2N7002
- added R26: 10k, Resistor_SMD:R_0402_1005Metric, symbol Device:R
Connections:
- new net DCDC_OUTCtrl: Q7.3 (D)
- new net GNDD: Q7.2 (S), R26.2
- new net Panel_PWRCtrl: Q7.1 (G), R26.1
Other:
- sheet Power ports: added SHDN_overV; removed none
- sheet RS485 ports: added Panel_PWRCtrl; removed none
Changed lines of the file:
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@@
 (kicad_sch (version 20230121) (generator eeschema)
   (paper "A4")
+  (junction (at 154.94 58.42) (diameter 0) (color 0 0 0 0)
+  )
+  (junction (at 147.32 68.58) (diameter 0) (color 0 0 0 0)
+  )
   (wire (pts (xy 213.36 68.58) (xy 215.9 68.58))
     (stroke (width 0) (type default))
@@
     (stroke (width 0) (type default))
   )
+  (wire (pts (xy 147.32 68.58) (xy 147.32 63.5))
+    (stroke (width 0) (type default))
+  )
   (wire (pts (xy 213.36 63.5) (xy 215.9 63.5))
     (stroke (width 0) (type default))
@@
     (stroke (width 0) (type default))
   )
+  (wire (pts (xy 147.32 50.8) (xy 147.32 53.34))
+    (stroke (width 0) (type default))
+  )
   (wire (pts (xy 213.36 76.2) (xy 215.9 76.2))
     (stroke (width 0) (type default))
@@
     (stroke (width 0) (type default))
   )
+  (wire (pts (xy 154.94 68.58) (xy 147.32 68.58))
+    (stroke (width 0) (type default))
+  )
   (wire (pts (xy 213.36 78.74) (xy 215.9 78.74))
     (stroke (width 0) (type default))
@@
     (stroke (width 0) (type default))
   )
+  (wire (pts (xy 213.36 83.82) (xy 215.9 83.82))
+    (stroke (width 0) (type default))
+  )
   (wire (pts (xy 213.36 53.34) (xy 215.9 53.34))
     (stroke (width 0) (type default))
@@
     (stroke (width 0) (type default))
   )
+  (wire (pts (xy 104.14 60.96) (xy 109.22 60.96))
+    (stroke (width 0) (type default))
+  )
+  (wire (pts (xy 154.94 67.31) (xy 154.94 68.58))
+    (stroke (width 0) (type default))
+  )
+  (wire (pts (xy 154.94 58.42) (xy 154.94 59.69))
+    (stroke (width 0) (type default))
+  )
+  (wire (pts (xy 157.48 58.42) (xy 154.94 58.42))
+    (stroke (width 0) (type default))
+  )
+  (rectangle (start 124.46 43.18) (end 175.26 78.74)
+    (stroke (width 0) (type default))
+    (fill (type none))
+  )
   (label "TangPrimerRXx_Panel1TX" (at 213.36 48.26 180) (fields_autoplaced)
     (effects (font (size 1.27 1.27) (thickness 0.254) bold italic) (justify right bottom))
   )
+  (label "Panel_PWRCtrl" (at 157.48 58.42 0) (fields_autoplaced)
+    (effects (font (size 1.27 1.27) (thickness 0.254) bold italic) (justify left bottom))
+  )
   (label "TangPrimerRXx_Panel3TX" (at 213.36 63.5 180) (fields_autoplaced)
     (effects (font (size 1.27 1.27) (thickness 0.254) bold italic) (justify right bottom))
@@
     (effects (font (size 1.27 1.27) (thickness 0.254) bold italic) (justify right bottom))
   )
+  (label "DCDC_OUTCtrl" (at 109.22 60.96 0) (fields_autoplaced)
+    (effects (font (size 1.27 1.27) (thickness 0.254) bold italic) (justify left bottom))
+  )
   (label "TangPrimerTXx_Panel0RX" (at 213.36 38.1 180) (fields_autoplaced)
     (effects (font (size 1.27 1.27) (thickness 0.254) bold italic) (justify right bottom))
   )
+  (label "Panel_PWRCtrl" (at 213.36 83.82 180) (fields_autoplaced)
+    (effects (font (size 1.27 1.27) (thickness 0.254) bold italic) (justify right bottom))
+  )
+  (label "DCDC_OUTCtrl" (at 147.32 50.8 180) (fields_autoplaced)
+    (effects (font (size 1.27 1.27) (thickness 0.254) bold italic) (justify right bottom))
+  )
   (label "TangPrimerRXx_Panel4TX" (at 213.36 71.12 180) (fields_autoplaced)
     (effects (font (size 1.27 1.27) (thickness 0.254) bold italic) (justify right bottom))
@@
     (effects (font (size 1.27 1.27) (thickness 0.254) bold italic) (justify right bottom))
   )
-  (sheet (at 215.9 33.02) (size 25.4 50.8) (fields_autoplaced)
+  (symbol (lib_id "Device:R") (at 154.94 63.5 0) (unit 1)
+    (in_bom yes) (on_board yes) (dnp no)
+    (property "Reference" "R26" (at 156.21 62.23 0)
+      (effects (font (size 1.27 1.27)) (justify left))
+    )
+    (property "Value" "10k" (at 156.21 64.77 0)
+      (effects (font (size 1.27 1.27)) (justify left))
+    )
+    (property "Footprint" "Resistor_SMD:R_0402_1005Metric" (at 153.162 63.5 90)
+      (effects (font (size 1.27 1.27)) hide)
+    )
+    (property "Datasheet" "~" (at 154.94 63.5 0)
+      (effects (font (size 1.27 1.27)) hide)
+    )
+    (pin "1")
+    (pin "2")
+    (instances
+      (project "DCDC"
+        (path "/ff041c4b-2038-4373-9ca4-fac09ac6c22f"
+          (reference "R26") (unit 1)
+        )
+      )
+    )
+  )
+  (symbol (lib_id "Transistor_FET:2N7002") (at 149.86 58.42 0) (mirror y) (unit 1)
+    (in_bom yes) (on_board yes) (dnp no)
+    (property "Reference" "Q7" (at 157.48 50.8 0)
+      (effects (font (size 1.27 1.27)) (justify left))
+    )
+    (property "Value" "2N7002" (at 157.48 53.34 0)
+      (effects (font (size 1.27 1.27)) (justify left))
+    )
+    (property "Footprint" "Package_TO_SOT_SMD:SOT-23" (at 144.78 60.325 0)
+      (effects (font (size 1.27 1.27) italic) (justify left) hide)
+    )
+    (property "Datasheet" "https://www.onsemi.com/pub/Collateral/NDS7002A-D.PDF" (at 144.78 62.23 0)
+      (effects (font (size 1.27 1.27)) (justify left) hide)
+    )
+    (pin "3")
+    (pin "1")
+    (pin "2")
+    (instances
+      (project "DCDC"
+        (path "/ff041c4b-2038-4373-9ca4-fac09ac6c22f"
+          (reference "Q7") (unit 1)
+        )
+      )
+    )
+  )
+  (symbol (lib_id "power:GNDD") (at 147.32 68.58 0) (mirror y) (unit 1)
+    (in_bom yes) (on_board yes) (dnp no)
+    (property "Reference" "#PWR029" (at 147.32 74.93 0)
+      (effects (font (size 1.27 1.27)) hide)
+    )
+    (property "Value" "GNDD" (at 147.32 72.39 0)
+      (effects (font (size 1.27 1.27)))
+    )
+    (property "Footprint" "" (at 147.32 68.58 0)
+      (effects (font (size 1.27 1.27)) hide)
+    )
+    (property "Datasheet" "" (at 147.32 68.58 0)
+      (effects (font (size 1.27 1.27)) hide)
+    )
+    (pin "1")
+    (instances
+      (project "DCDC"
+        (path "/ff041c4b-2038-4373-9ca4-fac09ac6c22f"
+          (reference "#PWR029") (unit 1)
+        )
+      )
+    )
+  )
+  (sheet (at 215.9 33.02) (size 25.4 55.88) (fields_autoplaced)
     (stroke (width 0.1524) (type solid))
     (fill (color 0 0 0 0.0000))
@@
       (effects (font (size 1.27 1.27)) (justify left bottom))
     )
-    (property "Sheetfile" "RS485.kicad_sch" (at 215.9 84.4046 0)
+    (property "Sheetfile" "RS485.kicad_sch" (at 215.9 89.4846 0)
       (effects (font (size 1.27 1.27)) (justify left top))
     )
@@
       (effects (font (size 1.27 1.27)) (justify left))
     )
+    (pin "Panel_PWRCtrl" input (at 215.9 83.82 180)
+      (effects (font (size 1.27 1.27)) (justify left))
+    )
     (instances
       (project "DCDC"
@@
     )
   )
-  (sheet (at 25.4 25.4) (size 20.32 15.24) (fields_autoplaced)
+  (sheet (at 83.82 53.34) (size 20.32 15.24) (fields_autoplaced)
     (stroke (width 0.1524) (type solid))
     (fill (color 0 0 0 0.0000))
-    (property "Sheetname" "Power" (at 25.4 24.6884 0)
+    (property "Sheetname" "Power" (at 83.82 52.6284 0)
       (effects (font (size 1.27 1.27)) (justify left bottom))
     )
-    (property "Sheetfile" "Power.kicad_sch" (at 25.4 41.2246 0)
+    (property "Sheetfile" "Power.kicad_sch" (at 83.82 69.1646 0)
       (effects (font (size 1.27 1.27)) (justify left top))
     )
-    (instances
+    (pin "SHDN_overV" input (at 104.14 60.96 0)
+      (effects (font (size 1.27 1.27)) (justify right))
+    )
+    (instances

Commit message: 更新
Other:
- sheet Power ports: added SHDN_OV; removed SHDN_overV
Changed lines of the file:
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@@
       (effects (font (size 1.27 1.27)) (justify left top))
     )
-    (pin "SHDN_overV" input (at 104.14 60.96 0)
+    (pin "SHDN_OV" input (at 104.14 60.96 0)
       (effects (font (size 1.27 1.27)) (justify right))
     )

Commit message: 発注第3弾
DCDC、MD追加
Parts:
- removed Q7: 2N7002, Package_TO_SOT_SMD:SOT-23, symbol Transistor_FET:2N7002
- removed R26: 10k, Resistor_SMD:R_0402_1005Metric, symbol Device:R
Other:
- sheet RS485 ports: added none; removed FPGARX_Panel0TX, FPGARX_Panel1TX, FPGARX_Panel2TX, FPGARX_Panel3TX, FPGARX_Panel4TX, FPGARX_Panel5TX, FPGATX_Panel0RX, FPGATX_Panel1RX, FPGATX_Panel2RX, FPGATX_Panel3RX, FPGATX_Panel4RX, FPGATX_Panel5RX
