File: circuits/DCDC/Power.kicad_sch (KiCad schematic)
At the start: 72 parts, among them J2 Conn_01x02_Male, J3 Conn_01x02_Female, Q10 MTP4835I3, Q11 MTP4835I3, Q12 BSS138, Q7 2SC3265, Q8 MTP4835I3, Q9 MTP4835I3, SW1 SW_SPDT_White, U7 MC34063AD, U8 AZ1084CD-3.3, U9 M51957B

Commit message: raspi基板回路図
Parts:
- removed C10, C7: 0.1uF, Capacitor_SMD:C_0402_1005Metric, symbol Device:C
- removed C11, C15, C16: C_snub, Capacitor_SMD:C_0603_1608Metric, symbol Device:C
- removed C12, C8, C9: 10uF, Capacitor_SMD:C_0805_2012Metric, symbol Device:C
- removed C13: 470uF, Capacitor_THT:CP_Radial_D10.0mm_P2.50mm_P5.00mm, symbol Device:C_Polarized_US
- removed C14: 100pF, Capacitor_SMD:C_0603_1608Metric, symbol Device:C
- removed D10, D2, D3: SS2040FL, Diode_SMD:D_SOD-123, symbol Device:D_Schottky
- removed D4, D5, D8: 1N5819WS, Diode_SMD:D_SOD-323_HandSoldering, symbol Device:D_Schottky
- removed D7: CBD20150VCT, Package_TO_SOT_THT:TO-220-3_Horizontal_TabDown, symbol Device:D_Schottky_AKA
- removed J3: Conn_01x02_Female, Connector_AMASS:AMASS_XT30PW-F_1x02_P2.50mm_Horizontal, symbol Connector:Conn_01x02_Female
- removed L1: 2.2uH, Inductor_Power:ETQ-P4M_KVK, symbol Device:L
- removed Q7: 2SC3265, Package_TO_SOT_SMD:SOT-23, symbol Device:Q_NPN_BEC
- removed Q8, Q9: MTP4835I3, Package_TO_SOT_SMD:TO-252-2, symbol Device:Q_PMOS_GDS
- removed R26: 510, Resistor_SMD:R_0402_1005Metric, symbol Device:R
- removed R27, R39, R47, R48: 10k, Resistor_SMD:R_0402_1005Metric, symbol Device:R
- removed R28: 10, Resistor_SMD:R_0603_1608Metric, symbol Device:R
- removed R30, R33, R34: R_snub, Resistor_SMD:R_0603_1608Metric, symbol Device:R
- removed R32, R46: 1k, Resistor_SMD:R_0402_1005Metric, symbol Device:R
- removed R35: 5.1k, Resistor_SMD:R_0402_1005Metric, symbol Device:R
- removed R36: 5.1k, Resistor_SMD:R_0603_1608Metric, symbol Device:R
- removed R37: 7.5k, Resistor_SMD:R_0603_1608Metric, symbol Device:R
- removed R38: 1.5k, Resistor_SMD:R_0603_1608Metric, symbol Device:R
- removed R40: 2k, Resistor_SMD:R_0603_1608Metric, symbol Device:R
- removed RV1: 470, Potentiometer:PVZ3A, symbol Device:R_Potentiometer
- removed U7: MC34063AD, Package_SO:SOIC-8_3.9x4.9mm_P1.27mm, symbol Regulator_Switching:MC34063AD
- removed U8: AZ1084CD-3.3, Package_TO_SOT_SMD:TO-252-2, symbol Regulator_Linear:AMS1117CD-3.3
- added C26, C27, C28: 0.1uF, Capacitor_SMD:C_0402_1005Metric, symbol Device:C
- added C29, C30: 1uF, Capacitor_SMD:C_0402_1005Metric, symbol Device:C
- added C31: 10uF, Capacitor_SMD:C_0805_2012Metric, symbol Device:C
- added C32: 330uF, Capacitor_THT:CP_Radial_D10.0mm_P2.50mm_P5.00mm, symbol Device:C_Polarized_US
- added C33, C34: C_snub, Capacitor_SMD:C_0603_1608Metric, symbol Device:C
- added D11, D12, D14: SS2040FL, Diode_SMD:D_SOD-123, symbol Device:D_Schottky
- added D13, D15: 1N5819WS, Diode_SMD:D_SOD-323_HandSoldering, symbol Device:D_Schottky
- added L2: 2.2uH, Inductor_Power:ETQ-P4M_KVK, symbol Device:L
- added Q13, Q14: TPN19008QM, MyLibrary:Package_TSON-Advance, symbol Transistor_FET:FDMS8050
- added Q15: MTP4835I3, Package_TO_SOT_SMD:TO-252-2, symbol Device:Q_PMOS_GDS
- added R49, R50, R52, R53, R59: 10k, Resistor_SMD:R_0402_1005Metric, symbol Device:R
- added R51: 1k, Resistor_SMD:R_0402_1005Metric, symbol Device:R
- added R54: R_snub, Resistor_SMD:R_0603_1608Metric, symbol Device:R
- added R55: 5.1k, Resistor_SMD:R_0402_1005Metric, symbol Device:R
- added R56: 5.1k, Resistor_SMD:R_0603_1608Metric, symbol Device:R
- added R57: 7.5k, Resistor_SMD:R_0603_1608Metric, symbol Device:R
- added R58: 1.5k, Resistor_SMD:R_0603_1608Metric, symbol Device:R
- added R60: 2k, Resistor_SMD:R_0603_1608Metric, symbol Device:R
- added RV2: 470, Potentiometer:PVZ3A, symbol Device:R_Potentiometer
- added U10: RT9624A, Package_SO:SOP-8_3.9x4.9mm_P1.27mm, symbol Driver_FET:IR2109
- added U11: RT8250, Package_SO:SOP-8_3.9x4.9mm_P1.27mm, symbol Regulator_Switching:AP6503
- added U12: AZ1084CD-12, Package_TO_SOT_SMD:TO-252-2, symbol Regulator_Linear:AMS1117CD-3.3
- C17, C18, C19, C20: footprint Capacitor_SMD:C_Elec_8x10.2 -> (none)
- C23: value 1uF -> 0.1uF
- C24: value 1uF -> 10uF; footprint Capacitor_SMD:C_0402_1005Metric -> Capacitor_SMD:C_0805_2012Metric
- J2: footprint Connector_AMASS:AMASS_XT30PW-M_1x02_P2.50mm_Horizontal -> Connector_Molex:Molex_SPOX_5268-02A_1x02_P2.50mm_Horizontal
- Q12: value BSS138 -> 2N7002
- R43: value 33k -> R_snub
- R45: value 10k -> 1k; footprint Resistor_SMD:R_0603_1608Metric -> Resistor_SMD:R_0402_1005Metric
Connections:
- net V_Measure is gone; now on net VDD: R43.2, R45.1
- net +3.3V: no longer C24.1, R31.2
- net +5V: now also R31.2, D15.2 (A), Q15.2 (D)
- net GND: now also C23.1, C28.1, C29.2, C30.2, C31.2, C32.2, C33.1, C34.1, D12.2 (A), Q14.1 (S), Q14.2 (S), Q14.3 (S), R50.1, R51.2, R52.2, R53.1, R58.1, R60.2, U10.4 (COM), U11.4 (GND), U11.9 (EP), U12.1 (GND); no longer C23.2
- net SHDN_overV: now also Q15.1 (G), R55.2
- net VCC: now also C29.1, D13.1 (K), D14.1 (K), R52.1, U12.3 (VI); no longer C23.1
- net VDD: now also C23.2, C24.1, D11.1 (K), D14.2 (A), Q13.5 (D), R51.1; no longer R43.1
- net V_Surv.: now also R57.1, R60.1
- net 12VBAT renamed +BATT
- net 主電源スイッチ renamed PowerSW
- new net: C27.2, D11.2 (A), D12.1 (K), L2.1, Q13.1 (S), Q13.2 (S), Q13.3 (S), Q14.5 (D), U10.6 (VS)
- new net: C31.1, C32.1, D15.1 (K), L2.2, Q15.3 (S), R54.2, R55.1, R56.2, R57.2
- new net: Q14.4 (G), U10.5 (LO)
- new net: R49.1, R50.2, U10.2 (IN)
- new net: C26.2, R49.2, U11.3 (SW)
- new net: C26.1, U11.1 (BST)
- new net: C34.2, R43.1
- new net: R58.2, R59.1, RV2.2
- new net: R59.2, RV2.1
- new net: Q13.4 (G), U10.7 (HO)
- new net: C27.1, U10.8 (VB)
- new net: C33.2, R54.1
- new net +12V: C28.2, C30.1, D13.2 (A), R53.2, U10.1 (VCC), U11.2 (IN), U12.2 (VO)
- new net fb: R56.1, RV2.3, U11.5 (FB)
- no-connect marks 1 -> 5

Commit message: 更新
Parts:
- removed C26: 0.1uF, Capacitor_SMD:C_0402_1005Metric, symbol Device:C
- removed D14: SS2040FL, Diode_SMD:D_SOD-123, symbol Device:D_Schottky
- removed R58: 1.5k, Resistor_SMD:R_0603_1608Metric, symbol Device:R
- removed R59: 10k, Resistor_SMD:R_0402_1005Metric, symbol Device:R
- removed RV2: 470, Potentiometer:PVZ3A, symbol Device:R_Potentiometer
- removed U11: RT8250, Package_SO:SOP-8_3.9x4.9mm_P1.27mm, symbol Regulator_Switching:AP6503
- added C10: 2700pF, Capacitor_SMD:C_0402_1005Metric, symbol Device:C
- added C11: 47pF, Capacitor_SMD:C_0402_1005Metric, symbol Device:C
- added C12, C14: 0.1uF, Capacitor_SMD:C_0402_1005Metric, symbol Device:C
- added C13: 1nF, Capacitor_SMD:C_0402_1005Metric, symbol Device:C
- added C7, C9: 1uF, Capacitor_SMD:C_0402_1005Metric, symbol Device:C
- added C8: 1500pF, Capacitor_SMD:C_0402_1005Metric, symbol Device:C
- added D2: 1N5819WS, Diode_SMD:D_SOD-323_HandSoldering, symbol Device:D_Schottky
- added H1: MountingHole_Pad, TestPoint:TestPoint_Pad_D1.5mm, symbol Mechanical:MountingHole_Pad
- added Q16, Q17, Q9: 2SA1037AK, Package_TO_SOT_SMD:SOT-23, symbol Device:Q_PNP_BEC
- added Q8: SS8050, Package_TO_SOT_SMD:SOT-23, symbol Device:Q_NPN_BEC
- added R27, R32: 510, Resistor_SMD:R_0402_1005Metric, symbol Device:R
- added R28, R34: 1k, Resistor_SMD:R_0402_1005Metric, symbol Device:R
- added R30, R46: 10k, Resistor_SMD:R_0402_1005Metric, symbol Device:R
- added R33: 2.7k, Resistor_SMD:R_0402_1005Metric, symbol Device:R
- added R35: 12k, Resistor_SMD:R_0402_1005Metric, symbol Device:R
- added R36: 10M, Resistor_SMD:R_0402_1005Metric, symbol Device:R
- added R37: 16k, Resistor_SMD:R_0603_1608Metric, symbol Device:R
- added R38: 620, Resistor_SMD:R_0603_1608Metric, symbol Device:R
- added R39: 1k, Resistor_SMD:R_0603_1608Metric, symbol Device:R
- added R40: 10k, Resistor_SMD:R_0603_1608Metric, symbol Device:R
- added R47: 20k, Resistor_SMD:R_0402_1005Metric, symbol Device:R
- added U7: UC3843_SOIC8, Package_SO:SOIC-8_3.9x4.9mm_P1.27mm, symbol Regulator_Controller:UC3843_SOIC8
- added U8: NJM2716, Package_TO_SOT_SMD:SOT-23-5, symbol Amplifier_Operational:ADA4610-1xRJ
- C27: value 0.1uF -> 1uF
- R45: value 1k -> 10k
- R49: value 10k -> 1k
- R50: value 10k -> 510
- R56: value 5.1k -> 16k
- U12: value AZ1084CD-12 -> NJM78L12SU3; footprint Package_TO_SOT_SMD:TO-252-2 -> Package_TO_SOT_SMD:SOT-89-3
Connections:
- net +12V: now also C12.1, R47.2, U7.7 (VCC)
- net +5V: now also C14.2, R40.2, U8.5 (V+)
- net GND: now also C12.2, C14.1, C7.2, C8.2, C9.2, Q17.3 (C), R28.1, R34.1, R37.1, R39.1, R40.1, R46.1, U7.5 (GND), U8.2 (V-)
- net SHDN_overV: no longer U9.6 (OUT)
- net VCC: now also D2.1 (K)
- net VDD: now also D2.2 (A)
- net SW: now reaches C27.2, D11.2 (A), D12.1 (K), L2.1, Q13.1 (S), Q13.2 (S), Q13.3 (S), Q14.5 (D), U10.6 (VS)
- net at C31.1, C32.1, D15.1 (K)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: now also C13.2, R39.2
- net LG: now reaches Q14.4 (G), U10.5 (LO)
- net at R49.2: now also U7.6 (OUT)
- net at U10.3 (~{SD}): now also R46.2, R47.1
- net HG: now reaches Q13.4 (G), U10.7 (HO)
- net fb renamed FB
- net FB: now also C10.2, C11.1, R36.2, R37.2, R38.1, U7.2 (FB)
- new net: C9.1, Q17.1 (B), R30.1
- new net: C7.1, Q8.3 (C), R27.2, R30.2, R32.2, U7.8 (VREF)
- new net: C13.1, R38.2
- new net: C10.1, R35.1
- new net: C11.2, Q17.2 (E), R35.2, R36.1, U7.1 (COMP)
- new net: Q16.2 (E), R32.1
- new net: H1.1, U8.1, U8.4 (-)
- new net: Q16.1 (B), Q16.3 (C), Q9.1 (B), R28.2
- new net: Q9.2 (E), R27.1
- new net: Q8.2 (E), R33.2
- new net CLK: C8.1, Q8.1 (B), Q9.3 (C), U7.4 (RC), U8.3 (+)
- new net SHDN_OV: U9.6 (OUT)
- new net Slope: R33.1, R34.2, U7.3 (CS)
- no-connect marks 5 -> 1
Other:
- note added: "12V生成"
- note added: "パワー段"
- note removed: "3.3V生成"
- note removed: "5V生成"
- moved on the sheet: C17, C18, C19, C20, C21, C22, C25, C27, C28, C29, C30, C31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

Commit message: 発注第3弾
DCDC、MD追加
Parts:
- removed C17, C18, C19, C20: 470uF, symbol Device:C_Polarized
- removed C21, C29, C30: 1uF, Capacitor_SMD:C_0402_1005Metric, symbol Device:C
- removed C23: 0.1uF, Capacitor_SMD:C_0402_1005Metric, symbol Device:C
- removed C24, C31: 10uF, Capacitor_SMD:C_0805_2012Metric, symbol Device:C
- removed C32: 330uF, Capacitor_THT:CP_Radial_D10.0mm_P2.50mm_P5.00mm, symbol Device:C_Polarized_US
- removed C34: C_snub, Capacitor_SMD:C_0603_1608Metric, symbol Device:C
- removed D1, D6: Green, LED_SMD:LED_0603_1608Metric_Pad1.05x0.95mm_HandSolder, symbol Device:LED
- removed D9: 1N5819WS, Diode_SMD:D_SOD-323_HandSoldering, symbol Device:D_Schottky
- removed J2: Conn_01x02_Male, Connector_Molex:Molex_SPOX_5268-02A_1x02_P2.50mm_Horizontal, symbol Connector:Conn_01x02_Male
- removed Q10, Q11: MTP4835I3, Package_TO_SOT_SMD:TO-252-2, symbol Device:Q_PMOS_GDS
- removed Q12: 2N7002, Package_TO_SOT_SMD:SOT-23, symbol Device:Q_NMOS_GSD
- removed R29, R42, R44, R45, R52: 10k, Resistor_SMD:R_0402_1005Metric, symbol Device:R
- removed R31: 1k, Resistor_SMD:R_0402_1005Metric, symbol Device:R
- removed R39: 1k, Resistor_SMD:R_0603_1608Metric, symbol Device:R
- removed R40: 10k, Resistor_SMD:R_0603_1608Metric, symbol Device:R
- removed R41: 100k, Resistor_SMD:R_0402_1005Metric, symbol Device:R
- removed R43: R_snub, Resistor_SMD:R_0603_1608Metric, symbol Device:R
- removed R55: 5.1k, Resistor_SMD:R_0402_1005Metric, symbol Device:R
- removed TP2, TP3, TP4, TP5: TestPoint, TestPoint:TestPoint_THTPad_D2.0mm_Drill1.0mm, symbol Connector:TestPoint
- removed U10: RT9624A, Package_SO:SOP-8_3.9x4.9mm_P1.27mm, symbol Driver_FET:IR2109
- removed U12: NJM78L12SU3, Package_TO_SOT_SMD:SOT-89-3, symbol Regulator_Linear:AMS1117CD-3.3
- added C10, C8: 1uF, Capacitor_SMD:C_0402_1005Metric, symbol Device:C
- added C11, C7: 1uF_50V, Capacitor_SMD:C_0603_1608Metric, symbol Device:C
- added C12, C13, C14, C15: 10uF_50V, Capacitor_SMD:C_0805_2012Metric, symbol Device:C
- added C16, C19, C22, C25: 1nF, Capacitor_SMD:C_0603_1608Metric, symbol Device:C
- added C26: 330uF, Capacitor_Tantalum_SMD:CP_EIA-7343-20_Kemet-V, symbol Device:C_Polarized
- added C31, C32: 100uF, TomoshibiLibrary:Capacitor_Alum_Radial_5.0x11.0mm_Horizontal, symbol Device:C_Polarized
- added D3, D6: 1N5819WS, TomoshibiLibrary:Diode_SOD-323, symbol Device:D_Schottky
- added D8: Green, LED_SMD:LED_0603_1608Metric_Pad1.05x0.95mm_HandSolder, symbol Device:LED
- added FB1: FerriteBead, Inductor_SMD:L_0603_1608Metric, symbol Device:FerriteBead
- added H10, H11, H12, H13, H14, H15, H16, H17, H18, H19, H20, H21, H22, H23, H8, H9: MountingHole_Pad, MountingHole:MountingHole_3.7mm_Pad_Via, symbol Mechanical:MountingHole_Pad
- added J2: Conn_01x02_Pin, Connector_Molex:Molex_SPOX_5268-02A_1x02_P2.50mm_Horizontal, symbol Connector:Conn_01x02_Pin
- added Q1, Q3: SSM6J808R, TomoshibiLibrary:Package_TSOP6F, symbol Transistor_FET:PMN48XP
- added Q11, Q2: 2N7002, Package_TO_SOT_SMD:SC-59, symbol Transistor_FET:2N7002
- added R1, R2: Rg, Resistor_SMD:R_0603_1608Metric, symbol Device:R
- added R19, R21, R22, R23, R24, R49, R50, R53: 10k, Resistor_SMD:R_0402_1005Metric, symbol Device:R
- added R20, R27: 20k, Resistor_SMD:R_0402_1005Metric, symbol Device:R
- added R48: 1k, Resistor_SMD:R_0402_1005Metric, symbol Device:R
- added U7: NJM78L12S_SOT89, Package_TO_SOT_SMD:SOT-89-3, symbol Regulator_Linear:L78L12_SOT89
- added U9: Driver_FETGate_RT9624A, Package_SO:SOP-8_3.9x4.9mm_P1.27mm, symbol TomoshibiLibrary:Driver_FETGate_RT9624A
- C17: renamed from C8; footprint Capacitor_SMD:C_0402_1005Metric -> Capacitor_SMD:C_0603_1608Metric
- C18: renamed from C11; footprint Capacitor_SMD:C_0402_1005Metric -> Capacitor_SMD:C_0603_1608Metric
- C20: renamed from C10; footprint Capacitor_SMD:C_0402_1005Metric -> Capacitor_SMD:C_0603_1608Metric
- C27: renamed from C13; footprint Capacitor_SMD:C_0402_1005Metric -> Capacitor_SMD:C_0603_1608Metric
- C29: renamed from C27; value 1uF -> 1uF_50V; footprint Capacitor_SMD:C_0402_1005Metric -> Capacitor_SMD:C_0603_1608Metric
- C9: value 1uF -> 0.1uF_50V
- D1: renamed from D2; footprint Diode_SMD:D_SOD-323_HandSoldering -> TomoshibiLibrary:Diode_SOD-323
- D2: renamed from D13; footprint Diode_SMD:D_SOD-323_HandSoldering -> TomoshibiLibrary:Diode_SOD-323
- D7: renamed from D15; footprint Diode_SMD:D_SOD-323_HandSoldering -> TomoshibiLibrary:Diode_SOD-323
- L1: renamed from L2; footprint Inductor_Power:ETQ-P4M_KVK -> TomoshibiLibrary:Inductor_ETQ-P4M_KVK
- Q4: renamed from Q17; value 2SA1037AK -> SS8550; footprint Package_TO_SOT_SMD:SOT-23 -> Package_TO_SOT_SMD:SC-59
- Q5: renamed from Q16; value 2SA1037AK -> SS8550; footprint Package_TO_SOT_SMD:SOT-23 -> Package_TO_SOT_SMD:SC-59
- Q6: renamed from Q9; value 2SA1037AK -> SS8550; footprint Package_TO_SOT_SMD:SOT-23 -> Package_TO_SOT_SMD:SC-59
- Q7: renamed from Q8; footprint Package_TO_SOT_SMD:SOT-23 -> Package_TO_SOT_SMD:SC-59
- Q8: renamed from Q13; value TPN19008QM -> TPH11006NL; footprint MyLibrary:Package_TSON-Advance -> TomoshibiLibrary:Package_SOP-Advance
- Q9: renamed from Q14; value TPN19008QM -> TPH11006NL; footprint MyLibrary:Package_TSON-Advance -> TomoshibiLibrary:Package_SOP-Advance
- R25: value 1k -> 10k
- R31: renamed from R36; footprint Resistor_SMD:R_0402_1005Metric -> Resistor_SMD:R_0603_1608Metric
- R34: renamed from R35; footprint Resistor_SMD:R_0402_1005Metric -> Resistor_SMD:R_0603_1608Metric
- R35: renamed from R33; footprint Resistor_SMD:R_0402_1005Metric -> Resistor_SMD:R_0603_1608Metric
- R39: renamed from R49; value 1k -> 5.1k
- R40: renamed from R50; value 510 -> 3.3k
- SW1: footprint Slide_Switch:SW_Slide_SPDT_White -> TomoshibiLibrary:SW_Slide_SPDT_IS-1235-G
- U10: renamed from U8; value NJM2716 -> NJU77701
- renumbered C7 to C21, C33 to C23, C12 to C24, C14 to C30, C25 to C33, C22 to C34, D11 to D4, D12 to D5, H1 to H7, Q15 to Q10, R53 to R26, R30 to R28, R32 to R29, R28 to R30, R27 to R32, R34 to R36, R54 to R38, R47 to R41, R46 to R42, R56 to R43, R37 to R44, R38 to R45, R57 to R46, R60 to R47, U9 to U11, U7 to U8
Connections:
- net +12V: now also C34.2, U11.7 (VCC), C10.1, U7.1 (OUT), U9.4 (VCC)
- net +5V: now also R51.2, H10.1, H12.1, H14.1, H16.1, H18.1, H20.1, H22.1, H8.1, R50.1
- net +BATT: now also J2.2 (Pin_2), Q1.1 (D), Q1.2 (D), Q1.5 (D), Q1.6 (D)
- net GND: now also C9.1, R25.2, TP1.1, C10.2, C11.2, C12.2, C13.2, C14.2, C15.2, C16.2, C19.2, C22.2, C25.2, C26.2, C31.2, C32.2, C7.2, D3.2 (A), D8.1 (K), H11.1, H13.1, H15.1, H17.1, H19.1, H21.1, H23.1, H9.1, J2.1 (Pin_1), Q2.2 (S), R19.2, R20.2, R27.2, R48.2, R50.2, R53.2, U7.2 (GND), U9.6 (GND); no longer C9.2, R51.2
- net HG: now also R1.1
- net LG: now also R2.1
- net PowerSW: now also R25.1, Q2.1 (G), R22.2; no longer SW1.1 (A)
- net S-S: now also C8.1, Q1.4 (S), Q3.4 (S), R21.1, R23.1
- net SHDN_OV: now also Q11.1 (G), R53.1; no longer U11.6 (OUT)
- net SW: now also R38.2, U9.7 (PHS)
- net VCC: now also C9.2, C19.1, C32.1, C7.1, FB1.2, R20.1, U7.3 (IN); no longer D1.1 (K), R25.2
- net VDD: now also C12.1, C13.1, C14.1, C15.1, C16.1, C31.1, D3.1 (K), D6.1 (K), Q3.1 (D), Q3.2 (D), Q3.5 (D), Q3.6 (D), R27.1; no longer C34.2, R51.1, TP1.1, U11.7 (VCC)
- net at Q4.1 (B), R28.1: now also C11.1; no longer C9.1
- net at C27.2, D7.1 (K), L1.2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: now also C25.1, C26.1, D6.2 (A), R48.1, R49.1; no longer R38.2
- net at R41.1, R42.2: now also U9.3 (EN)
- net at R39.1, R40.2: now also U9.2 (PWM)
- net at C29.1: now also U9.1 (BT)
- net SHDN_overV renamed SHDN
- net SHDN: now also Q11.3 (D), R49.2
- net V_Surv. renamed V_Surv
- new net: Q11.2 (S), U11.6 (OUT)
- new net: C8.2, Q3.3 (G), R23.2, R24.1
- new net: Q2.3 (D), R24.2
- new net: C22.1, D1.1 (K), FB1.1
- new net: Q1.3 (G), R19.1, R21.2
- new net: D8.2 (A), R51.1
- new net: R2.2, U9.5 (LG)
- new net: R1.2, U9.8 (UG)
- new net: R22.1, SW1.1 (A)
Other:
- note added: "5V surveillance"
- note added: "Clock Buffer"
- note added: "Panelとの接続"
- note added: "制御段"
- note added: "補機電源生成"
- note removed: "12V生成"
- note removed: "5V監視"
- moved on the sheet: C17, C18, C20, C21, C23, C24, C27, C28, C29, C30, C33, C34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
